File: KiCad/batteryless_gaming_device/batteryless_gaming_device.sch (KiCad schematic (older format))
At the start: 41 parts

Commit message: test update
Parts:
- added U?: TPS610995DRV, symbol batteryless_gaming_device-rescue:TPS610995DRV-johns_library
Changed lines of the file:
@@
 	-1   0    0    1
 $EndComp
+$Comp
+L batteryless_gaming_device-rescue:TPS610995DRV-johns_library U?
+U 1 1 61358B6B
+P 9200 1800
+F 0 "U?" H 9150 1815 50  0000 C CNN
+F 1 "TPS610995DRV" H 9150 1724 50  0000 C CNN
+F 2 "" H 9200 1800 50  0001 C CNN
+F 3 "" H 9200 1800 50  0001 C CNN
+	1    9200 1800
+	1    0    0    -1
+$EndComp
 $EndSCHEMATC
