File: KiCad/batteryless_gaming_device/batteryless_gaming_device.sch (KiCad schematic (older format))
At the start: 42 parts

Commit message: updated some stuff in main schematic
Parts:
- removed C?: 47u, symbol Device:CP1_Small
- removed C? (x4): 10u, symbol Device:C_Small
- removed C?: 4.7u, symbol Device:C_Small
- removed C?: 0.01u, symbol Device:C_Small
- removed C?: 0.1u, symbol Device:C_Small
- removed C?: 220m, symbol Device:CP1_Small
- removed D?: DMA40U1800GU, Diode_THT:Diode_Bridge_IXYS_GUFP, symbol Diode_Bridge:DMA40U1800GU
- removed D?: Zener, Diode_SMD:D_MiniMELF, symbol Diode:ZMMxx
- removed D? (x4): D_Schottky, symbol Device:D_Schottky
- removed L?: 2.2u, symbol Device:L
- removed L?: 22u, symbol Device:L
- removed M?: Hand Generator, symbol Motor:Motor_Servo
- removed R?: 6.25M, symbol Device:R_Small_US
- removed R?: 2.5M, symbol Device:R_Small_US
- removed R?: 1.25M, symbol Device:R_Small_US
- removed R?: 1.67M, symbol Device:R_Small_US
- removed R?: 8.33M, symbol Device:R_Small_US
- removed R?: 4.32M, symbol Device:R_Small_US
- removed R?: 5.68M, symbol Device:R_Small_US
- removed R? (x2): 10M, symbol Device:R_Small_US
- removed U?: BQ25504, Package_DFN_QFN:QFN-16-1EP_3x3mm_P0.5mm_EP1.8x1.8mm, symbol Battery_Management:BQ25504
- removed U?: TPS610995DRV, symbol batteryless_gaming_device-rescue:TPS610995DRV-johns_library
- removed U? (x4): Button_Detect, symbol johns_library:Button
- removed U? (x2): VoltageSupervisor, symbol johns_library:VoltageSupervisor
- removed U?: 74LVC1GU04DRL, Package_TO_SOT_SMD:SOT-553, symbol 74xGxx:74LVC1GU04DRL
- added U?: MSP430FR5994, symbol batteryless_gaming_device-rescue:MSP430FR5994
Connections:
- net labels removed: +3.3V, GPIO
- wire segments 166 -> 29
- no-connect marks 1 -> 0
Other:
- moved on the sheet: C?, L?, SupC, U?

Commit message: keep updating schematic
Parts:
- removed U?: MSP430FR5994, symbol batteryless_gaming_device-rescue:MSP430FR5994
- renumbered SupC to SupC?
Changed lines of the file:
@@
 $Descr A 11000 8500
 encoding utf-8
-Sheet 1 4
+Sheet 1 5
 Title "Battery Free Gaming Device"
 Date ""
@@
 F1 "hand_crank_generator.sch" 50
 F2 "Vout" O R 2300 4650 50
+F3 "generator_voltage" O R 2300 5200 50
 $EndSheet
 Wire Wire Line
@@
 	3650 2450 3650 2650
 $Comp
-L Device:C_Small SupC
+L Device:C_Small SupC?
 U 1 1 608710A0
 P 3650 2750
-F 0 "SupC" H 3742 2796 50  0000 L CNN
+F 0 "SupC?" H 3742 2796 50  0000 L CNN
 F 1 "2.2mF" H 3742 2705 50  0000 L CNN
 F 2 "" H 3650 2750 50  0001 C CNN
@@
 	0    -1   -1   0
 $EndComp
-$Comp
-L batteryless_gaming_device-rescue:MSP430FR5994 U?
-U 1 1 61ABD78E
-P 7900 1150
-F 0 "U?" H 7925 1317 50  0000 C CNN
-F 1 "MSP430FR5994" H 7925 1226 50  0000 C CNN
-F 2 "" V 7000 950 354 0001 C CNN
-F 3 "" V 7000 950 354 0001 C CNN
-	1    7900 1150
-	1    0    0    -1
-$EndComp
+$Sheet
+S 6650 2450 1900 3100
+U 61926AE2
+F0 "Microcontroller" 50
+F1 "micro_msp430fr5994.sch" 50
+$EndSheet
 $EndSCHEMATC

Commit message: keep on keeping on
Parts:
- removed C? (x2): 10u, symbol Device:C_Small
- removed L?: 2.2u, symbol Device:L
- removed SupC?: 2.2mF, symbol Device:C_Small
- removed U? (x2): TPS610995DRV, symbol batteryless_gaming_device-rescue:TPS610995DRV-johns_library
- added C? (x3): 10uF, symbol Device:C_Small
- added C?: 1uF, symbol Device:C_Small
- added C? (x2): 0.1uF, symbol Device:C_Small
- added L?: 2.2u, symbol Device:L
- added R? (x2): R_US, symbol Device:R_US
- added U?: TPS61201DRC, Package_SON:Texas_S-PVSON-N10_ThermalVias, symbol Regulator_Switching:TPS61201DRC
Connections:
- net labels removed: +3V8
- wire segments 29 -> 50

Commit message: updated schematic
Parts:
- removed C? (x3): 10uF, symbol Device:C_Small
- removed C?: 1uF, symbol Device:C_Small
- removed C? (x2): 0.1uF, symbol Device:C_Small
- removed L?: 2.2u, symbol Device:L
- removed R? (x2): R_US, symbol Device:R_US
- removed U?: TPS61201DRC, Package_SON:Texas_S-PVSON-N10_ThermalVias, symbol Regulator_Switching:TPS61201DRC
Other:
- note added: "+3.3V"
- note added: "TODO:\nAdd 0 ohms everywhere\nAdd test points\nAdd mounting holes\nAdd E-ink display\nFootprints/bom spec\nFigure out buck converter\n3.3V program in protection"

Commit message: k
Parts:
- added H? (x4): MountingHole_Pad, symbol Mechanical:MountingHole_Pad
- added J?: Voltage Source Select, symbol Connector_Generic:Conn_01x03
- added U?: E-Ink_Display_1.54Inch, symbol batteryless_gaming_device-rescue:E-Ink_Display_1.54Inch
Connections:
- new net +3V3: J?.2 (Pin_2), U?.8 (VCC)
- new net GND: H?.1, H?.1, H?.1, H?.1, U?.7 (GND)
- new net Microcontroller/V_program: J?.1 (Pin_1)
- new net Power Regulation/Vout: J?.3 (Pin_3)
Other:
- note added: "TODO:\nFootprints/bom spec\nFigure out buck converter\nAdd multiplayer connection pins"
- note removed: "TODO:\nAdd 0 ohms everywhere\nAdd test points\nAdd mounting holes\nAdd E-ink display\nFootprints/bom spec\nFigure out buck converter\n3.3V program in protection"
Changed lines of the file:
@@
 $EndSheet
 $Sheet
-S 6600 2450 1900 3100
+S 7050 2450 1900 3100
 U 61926AE2
 F0 "Microcontroller" 50
 F1 "micro_msp430fr5994.sch" 50
-F2 "Button1" I L 6600 2650 50
-F3 "Button2" I L 6600 2750 50
-F4 "Button3" I L 6600 2850 50
-F5 "Button4" I L 6600 2950 50
-F6 "GeneratorVcc" I L 6600 5100 50
-F7 "VBAT_OK" I L 6600 4950 50
+F2 "Button1" I L 7050 2650 50
+F3 "Button2" I L 7050 2750 50
+F4 "Button3" I L 7050 2850 50
+F5 "Button4" I L 7050 2950 50
+F6 "GeneratorVcc" I L 7050 5100 50
+F7 "VBAT_OK" I L 7050 4950 50
+F8 "V_program" O L 7050 4000 50
 $EndSheet
 Wire Wire Line
@@
 F1 "power_regulation.sch" 50
 F2 "Vin" I L 5100 3600 50
+F3 "Vout" O R 6150 4000 50
 $EndSheet
 Wire Wire Line
@@
 	5200 3800 5350 3800
 Wire Wire Line
-	2600 2950 6600 2950
-Wire Wire Line
-	2600 2850 6600 2850
-Wire Wire Line
-	2600 2750 6600 2750
-Wire Wire Line
-	2600 2650 6600 2650
+	2600 2950 7050 2950
+Wire Wire Line
+	2600 2850 7050 2850
+Wire Wire Line
+	2600 2750 7050 2750
+Wire Wire Line
+	2600 2650 7050 2650
 Wire Wire Line
 	2600 4750 2850 4750
@@
 	2850 4750 2850 5100
 Wire Wire Line
-	2850 5100 6600 5100
+	2850 5100 7050 5100
 Wire Wire Line
 	4700 4500 4900 4500
@@
 	4900 4500 4900 4950
 Wire Wire Line
-	4900 4950 6600 4950
-Text Notes 7400 1750 0    79   ~ 0
-TODO:\nAdd 0 ohms everywhere\nAdd test points\nAdd mounting holes\nAdd E-ink display\nFootprints/bom spec\nFigure out buck converter\n3.3V program in protection
-Wire Notes Line
-	7200 650  7200 1950
-Wire Notes Line
-	7200 1950 9250 1950
-Wire Notes Line
-	9250 1950 9250 650
-Wire Notes Line
-	7200 650  9250 650
+	4900 4950 7050 4950
+Text Notes 6850 1750 0    79   ~ 0
+TODO:\nFootprints/bom spec\nFigure out buck converter\nAdd multiplayer connection pins
+Wire Notes Line
+	6650 650  6650 1950
+Wire Notes Line
+	6650 1950 8700 1950
+Wire Notes Line
+	8700 1950 8700 650
+Wire Notes Line
+	6650 650  8700 650
+$Comp
+L Connector_Generic:Conn_01x03 J?
+U 1 1 61979531
+P 6550 4300
+F 0 "J?" V 6750 4350 50  0000 R CNN
+F 1 "Voltage Source Select" V 6650 4700 50  0000 R CNN
+F 2 "" H 6550 4300 50  0001 C CNN
+F 3 "~" H 6550 4300 50  0001 C CNN
+	1    6550 4300
+	0    1    1    0
+$EndComp
+Wire Wire Line
+	6150 4000 6450 4000
+Wire Wire Line
+	6450 4000 6450 4100
+Wire Wire Line
+	7050 4000 6650 4000
+Wire Wire Line
+	6650 4000 6650 4100
+Wire Wire Line
+	6550 4100 6550 3900
+$Comp
+L power:+3.3V #PWR?
+U 1 1 61980457
+P 6550 3900
+AR Path="/61926AE2/61980457" Ref="#PWR?"  Part="1"
+AR Path="/61980457" Ref="#PWR?"  Part="1"
+F 0 "#PWR?" H 6550 3750 50  0001 C CNN
+F 1 "+3.3V" H 6565 4073 50  0000 C CNN
+F 2 "" H 6550 3900 50  0001 C CNN
+F 3 "" H 6550 3900 50  0001 C CNN
+	1    6550 3900
+	1    0    0    -1
+$EndComp
+$Comp
+L batteryless_gaming_device-rescue:E-Ink_Display_1.54Inch U?
+U 1 1 61986176
+P 9550 3650
+F 0 "U?" H 9800 3800 50  0000 L CNN
+F 1 "E-Ink_Display_1.54Inch" H 9600 3700 50  0000 L CNN
+F 2 "" H 9550 4150 50  0001 C CNN
+F 3 "" H 9550 4150 50  0001 C CNN
+	1    9550 3650
+	1    0    0    -1
+$EndComp
+$Comp
+L power:GND #PWR?
+U 1 1 61988A0E
+P 9600 4400
+AR Path="/61926AE2/61988A0E" Ref="#PWR?"  Part="1"
+AR Path="/61988A0E" Ref="#PWR?"  Part="1"
+F 0 "#PWR?" H 9600 4150 50  0001 C CNN
+F 1 "GND" H 9605 4227 50  0000 C CNN
+F 2 "" H 9600 4400 50  0001 C CNN
+F 3 "" H 9600 4400 50  0001 C CNN
+	1    9600 4400
+	1    0    0    -1
+$EndComp
+Wire Wire Line
+	9600 4400 9600 4350
+$Comp
+L power:+3.3V #PWR?
+U 1 1 6198A1ED
+P 9600 3500
+AR Path="/61926AE2/6198A1ED" Ref="#PWR?"  Part="1"
+AR Path="/6198A1ED" Ref="#PWR?"  Part="1"
+F 0 "#PWR?" H 9600 3350 50  0001 C CNN
+F 1 "+3.3V" H 9615 3673 50  0000 C CNN
+F 2 "" H 9600 3500 50  0001 C CNN
+F 3 "" H 9600 3500 50  0001 C CNN
+	1    9600 3500
+	1    0    0    -1
+$EndComp
+Wire Wire Line
+	9600 3500 9600 3550
+$Comp
+L Mechanical:MountingHole_Pad H?
+U 1 1 6198BDFD
+P 9350 850
+F 0 "H?" H 9450 899 50  0000 L CNN
+F 1 "MountingHole_Pad" H 9350 1100 50  0000 L CNN
+F 2 "" H 9350 850 50  0001 C CNN
+F 3 "~" H 9350 850 50  0001 C CNN
+	1    9350 850
+	1    0    0    -1
+$EndComp
+$Comp
+L Mechanical:MountingHole_Pad H?
+U 1 1 6198CE4F
+P 9950 850
+F 0 "H?" H 10050 899 50  0000 L CNN
+F 1 "MountingHole_Pad" H 9350 1100 50  0000 L CNN
+F 2 "" H 9950 850 50  0001 C CNN
+F 3 "~" H 9950 850 50  0001 C CNN
+	1    9950 850
+	1    0    0    -1
+$EndComp
+$Comp
+L Mechanical:MountingHole_Pad H?
+U 1 1 6198D15F
+P 9350 1350
+F 0 "H?" H 9450 1399 50  0000 L CNN
+F 1 "MountingHole_Pad" H 9350 2100 50  0000 L CNN
+F 2 "" H 9350 1350 50  0001 C CNN
+F 3 "~" H 9350 1350 50  0001 C CNN
+	1    9350 1350
+	1    0    0    -1
+$EndComp
+$Comp
+L Mechanical:MountingHole_Pad H?
+U 1 1 6198D37A
+P 9950 1350
+F 0 "H?" H 10050 1399 50  0000 L CNN
+F 1 "MountingHole_Pad" H 9350 2100 50  0000 L CNN
+F 2 "" H 9950 1350 50  0001 C CNN
+F 3 "~" H 9950 1350 50  0001 C CNN
+	1    9950 1350
+	1    0    0    -1
+$EndComp
+$Comp
+L power:GND #PWR?
+U 1 1 6198DDE0
+P 9350 1450
+AR Path="/61926AE2/6198DDE0" Ref="#PWR?"  Part="1"
+AR Path="/6198DDE0" Ref="#PWR?"  Part="1"
+F 0 "#PWR?" H 9350 1200 50  0001 C CNN
+F 1 "GND" H 9355 1277 50  0000 C CNN
+F 2 "" H 9350 1450 50  0001 C CNN
+F 3 "" H 9350 1450 50  0001 C CNN
+	1    9350 1450
+	1    0    0    -1
+$EndComp
+$Comp
+L power:GND #PWR?
+U 1 1 6198E313
+P 9950 1450
+AR Path="/61926AE2/6198E313" Ref="#PWR?"  Part="1"
+AR Path="/6198E313" Ref="#PWR?"  Part="1"
+F 0 "#PWR?" H 9950 1200 50  0001 C CNN
+F 1 "GND" H 9955 1277 50  0000 C CNN
+F 2 "" H 9950 1450 50  0001 C CNN
+F 3 "" H 9950 1450 50  0001 C CNN
+	1    9950 1450
+	1    0    0    -1
+$EndComp
+$Comp
+L power:GND #PWR?
+U 1 1 6198E5F3
+P 9350 950
+AR Path="/61926AE2/6198E5F3" Ref="#PWR?"  Part="1"
+AR Path="/6198E5F3" Ref="#PWR?"  Part="1"
+F 0 "#PWR?" H 9350 700 50  0001 C CNN
+F 1 "GND" H 9355 777 50  0000 C CNN
+F 2 "" H 9350 950 50  0001 C CNN
+F 3 "" H 9350 950 50  0001 C CNN
+	1    9350 950
+	1    0    0    -1
+$EndComp
+$Comp
+L power:GND #PWR?
+U 1 1 6198E95A
+P 9950 950
+AR Path="/61926AE2/6198E95A" Ref="#PWR?"  Part="1"
+AR Path="/6198E95A" Ref="#PWR?"  Part="1"
+F 0 "#PWR?" H 9950 700 50  0001 C CNN
+F 1 "GND" H 9955 777 50  0000 C CNN
+F 2 "" H 9950 950 50  0001 C CNN
+F 3 "" H 9950 950 50  0001 C CNN
+	1    9950 950
+	1    0    0    -1
+$EndComp
+Wire Notes Line
+	9100 500  9100 1700
+Wire Notes Line
+	9100 1700 10500 1700
 $EndSCHEMATC

Commit message: k
Parts:
- gave numbers to parts that had none: 6
Connections:
- net Microcontroller/P4.1: now reaches U1.1 (BUSY)
- net Microcontroller/P4.2: now reaches U1.2 (RST)
- net Microcontroller/P4.3: now reaches U1.3 (DC)
- net Microcontroller/P2.5: now reaches U1.4 (CS)
- net Microcontroller/P5.2: now reaches U1.5 (CLK)
- net Microcontroller/P5.0: now reaches U1.6 (DIN)
Changed lines of the file:
@@
 F7 "VBAT_OK" I L 7050 4950 50
 F8 "V_program" O L 7050 4000 50
+F9 "P4.1" O R 8950 3700 50
+F10 "P4.2" O R 8950 3800 50
+F11 "P4.3" O R 8950 3900 50
+F12 "P2.5" O R 8950 4000 50
+F13 "P5.2" O R 8950 4100 50
+F14 "P5.0" O R 8950 4200 50
 $EndSheet
 Wire Wire Line
@@
 	6650 650  8700 650
 $Comp
-L Connector_Generic:Conn_01x03 J?
+L Connector_Generic:Conn_01x03 J1
 U 1 1 61979531
 P 6550 4300
-F 0 "J?" V 6750 4350 50  0000 R CNN
+F 0 "J1" V 6750 4350 50  0000 R CNN
 F 1 "Voltage Source Select" V 6650 4700 50  0000 R CNN
 F 2 "" H 6550 4300 50  0001 C CNN
@@
 P 6550 3900
 AR Path="/61926AE2/61980457" Ref="#PWR?"  Part="1"
-AR Path="/61980457" Ref="#PWR?"  Part="1"
-F 0 "#PWR?" H 6550 3750 50  0001 C CNN
+AR Path="/61980457" Ref="#PWR01"  Part="1"
+F 0 "#PWR01" H 6550 3750 50  0001 C CNN
 F 1 "+3.3V" H 6565 4073 50  0000 C CNN
 F 2 "" H 6550 3900 50  0001 C CNN
@@
 $EndComp
 $Comp
-L batteryless_gaming_device-rescue:E-Ink_Display_1.54Inch U?
+L batteryless_gaming_device-rescue:E-Ink_Display_1.54Inch U1
 U 1 1 61986176
 P 9550 3650
-F 0 "U?" H 9800 3800 50  0000 L CNN
+F 0 "U1" H 9800 3800 50  0000 L CNN
 F 1 "E-Ink_Display_1.54Inch" H 9600 3700 50  0000 L CNN
 F 2 "" H 9550 4150 50  0001 C CNN
@@
 P 9600 4400
 AR Path="/61926AE2/61988A0E" Ref="#PWR?"  Part="1"
-AR Path="/61988A0E" Ref="#PWR?"  Part="1"
-F 0 "#PWR?" H 9600 4150 50  0001 C CNN
+AR Path="/61988A0E" Ref="#PWR05"  Part="1"
+F 0 "#PWR05" H 9600 4150 50  0001 C CNN
 F 1 "GND" H 9605 4227 50  0000 C CNN
 F 2 "" H 9600 4400 50  0001 C CNN
@@
 P 9600 3500
 AR Path="/61926AE2/6198A1ED" Ref="#PWR?"  Part="1"
-AR Path="/6198A1ED" Ref="#PWR?"  Part="1"
-F 0 "#PWR?" H 9600 3350 50  0001 C CNN
+AR Path="/6198A1ED" Ref="#PWR04"  Part="1"
+F 0 "#PWR04" H 9600 3350 50  0001 C CNN
 F 1 "+3.3V" H 9615 3673 50  0000 C CNN
 F 2 "" H 9600 3500 50  0001 C CNN
@@
 	9600 3500 9600 3550
 $Comp
-L Mechanical:MountingHole_Pad H?
+L Mechanical:MountingHole_Pad H1
 U 1 1 6198BDFD
 P 9350 850
-F 0 "H?" H 9450 899 50  0000 L CNN
+F 0 "H1" H 9450 899 50  0000 L CNN
 F 1 "MountingHole_Pad" H 9350 1100 50  0000 L CNN
 F 2 "" H 9350 850 50  0001 C CNN
@@
 $EndComp
 $Comp
-L Mechanical:MountingHole_Pad H?
+L Mechanical:MountingHole_Pad H3
 U 1 1 6198CE4F
 P 9950 850
-F 0 "H?" H 10050 899 50  0000 L CNN
+F 0 "H3" H 10050 899 50  0000 L CNN
 F 1 "MountingHole_Pad" H 9350 1100 50  0000 L CNN
 F 2 "" H 9950 850 50  0001 C CNN
@@
 $EndComp
 $Comp
-L Mechanical:MountingHole_Pad H?
+L Mechanical:MountingHole_Pad H2
 U 1 1 6198D15F
 P 9350 1350
-F 0 "H?" H 9450 1399 50  0000 L CNN
+F 0 "H2" H 9450 1399 50  0000 L CNN
 F 1 "MountingHole_Pad" H 9350 2100 50  0000 L CNN
 F 2 "" H 9350 1350 50  0001 C CNN
@@
 $EndComp
 $Comp
-L Mechanical:MountingHole_Pad H?
+L Mechanical:MountingHole_Pad H4
 U 1 1 6198D37A
 P 9950 1350
-F 0 "H?" H 10050 1399 50  0000 L CNN
+F 0 "H4" H 10050 1399 50  0000 L CNN
 F 1 "MountingHole_Pad" H 9350 2100 50  0000 L CNN
 F 2 "" H 9950 1350 50  0001 C CNN
@@
 P 9350 1450
 AR Path="/61926AE2/6198DDE0" Ref="#PWR?"  Part="1"
-AR Path="/6198DDE0" Ref="#PWR?"  Part="1"
-F 0 "#PWR?" H 9350 1200 50  0001 C CNN
+AR Path="/6198DDE0" Ref="#PWR03"  Part="1"
+F 0 "#PWR03" H 9350 1200 50  0001 C CNN
 F 1 "GND" H 9355 1277 50  0000 C CNN
 F 2 "" H 9350 1450 50  0001 C CNN
@@
 P 9950 1450
 AR Path="/61926AE2/6198E313" Ref="#PWR?"  Part="1"
-AR Path="/6198E313" Ref="#PWR?"  Part="1"
-F 0 "#PWR?" H 9950 1200 50  0001 C CNN
+AR Path="/6198E313" Ref="#PWR07"  Part="1"
+F 0 "#PWR07" H 9950 1200 50  0001 C CNN
 F 1 "GND" H 9955 1277 50  0000 C CNN
 F 2 "" H 9950 1450 50  0001 C CNN
@@
 P 9350 950
 AR Path="/61926AE2/6198E5F3" Ref="#PWR?"  Part="1"
-AR Path="/6198E5F3" Ref="#PWR?"  Part="1"
-F 0 "#PWR?" H 9350 700 50  0001 C CNN
+AR Path="/6198E5F3" Ref="#PWR02"  Part="1"
+F 0 "#PWR02" H 9350 700 50  0001 C CNN
 F 1 "GND" H 9355 777 50  0000 C CNN
 F 2 "" H 9350 950 50  0001 C CNN
@@
 P 9950 950
 AR Path="/61926AE2/6198E95A" Ref="#PWR?"  Part="1"
-AR Path="/6198E95A" Ref="#PWR?"  Part="1"
-F 0 "#PWR?" H 9950 700 50  0001 C CNN
+AR Path="/6198E95A" Ref="#PWR06"  Part="1"
+F 0 "#PWR06" H 9950 700 50  0001 C CNN
 F 1 "GND" H 9955 777 50  0000 C CNN
 F 2 "" H 9950 950 50  0001 C CNN
@@
 Wire Notes Line
 	9100 1700 10500 1700
+Wire Wire Line
+	8950 3700 9200 3700
+Wire Wire Line
+	8950 3800 9200 3800
+Wire Wire Line
+	8950 3900 9200 3900
+Wire Wire Line
+	8950 4000 9200 4000
+Wire Wire Line
+	8950 4100 9200 4100
+Wire Wire Line
+	8950 4200 9200 4200
 $EndSCHEMATC
