File: KiCad/batteryless_gaming_device/batteryless_gaming_device.sch (KiCad schematic (older format))
At the start: 6 parts, among them J1 Voltage Source Select, U1 E-Ink_Display_1.54Inch

Commit message: just kinda out here guys ya know what im saying
Parts:
- H100: renamed from H1; footprint (none) -> MountingHole:MountingHole_3.2mm_M3_DIN965_Pad
- H101: renamed from H2; footprint (none) -> MountingHole:MountingHole_3.2mm_M3_DIN965_Pad
- H102: renamed from H3; footprint (none) -> MountingHole:MountingHole_3.2mm_M3_DIN965_Pad
- H103: renamed from H4; footprint (none) -> MountingHole:MountingHole_3.2mm_M3_DIN965_Pad
- J100: renamed from J1; footprint (none) -> Connector_PinHeader_2.54mm:PinHeader_1x03_P2.54mm_Vertical
- U100: renamed from U1; footprint (none) -> Connector_PinHeader_2.54mm:PinHeader_1x06_P2.54mm_Horizontal
Other:
- note added: "TODO:\nFind correct connector for generator"
- note removed: "TODO:\nFootprints/bom spec\nFigure out buck converter\nAdd multiplayer connection pins"
Changed lines of the file:
@@
 Wire Wire Line
 	4900 4950 7050 4950
-Text Notes 6850 1750 0    79   ~ 0
-TODO:\nFootprints/bom spec\nFigure out buck converter\nAdd multiplayer connection pins
-Wire Notes Line
-	6650 650  6650 1950
-Wire Notes Line
-	6650 1950 8700 1950
-Wire Notes Line
-	8700 1950 8700 650
-Wire Notes Line
-	6650 650  8700 650
-$Comp
-L Connector_Generic:Conn_01x03 J1
+Text Notes 6700 850  0    79   ~ 0
+TODO:\nFind correct connector for generator
+Wire Notes Line
+	6650 650  6650 1400
+Wire Notes Line
+	6650 1400 7800 1400
+Wire Notes Line
+	7800 1400 7800 650
+Wire Notes Line
+	6650 650  7800 650
+$Comp
+L Connector_Generic:Conn_01x03 J100
 U 1 1 61979531
 P 6550 4300
-F 0 "J1" V 6750 4350 50  0000 R CNN
+F 0 "J100" V 6750 4350 50  0000 R CNN
 F 1 "Voltage Source Select" V 6650 4700 50  0000 R CNN
-F 2 "" H 6550 4300 50  0001 C CNN
+F 2 "Connector_PinHeader_2.54mm:PinHeader_1x03_P2.54mm_Vertical" H 6550 4300 50  0001 C CNN
 F 3 "~" H 6550 4300 50  0001 C CNN
 	1    6550 4300
@@
 Wire Wire Line
 	6650 4000 6650 4100
-Wire Wire Line
-	6550 4100 6550 3900
 $Comp
 L power:+3.3V #PWR?
@@
 P 6550 3900
 AR Path="/61926AE2/61980457" Ref="#PWR?"  Part="1"
-AR Path="/61980457" Ref="#PWR01"  Part="1"
-F 0 "#PWR01" H 6550 3750 50  0001 C CNN
+AR Path="/61980457" Ref="#PWR0100"  Part="1"
+F 0 "#PWR0100" H 6550 3750 50  0001 C CNN
 F 1 "+3.3V" H 6565 4073 50  0000 C CNN
 F 2 "" H 6550 3900 50  0001 C CNN
@@
 $EndComp
 $Comp
-L batteryless_gaming_device-rescue:E-Ink_Display_1.54Inch U1
+L batteryless_gaming_device-rescue:E-Ink_Display_1.54Inch U100
 U 1 1 61986176
 P 9550 3650
-F 0 "U1" H 9800 3800 50  0000 L CNN
+F 0 "U100" H 9800 3800 50  0000 L CNN
 F 1 "E-Ink_Display_1.54Inch" H 9600 3700 50  0000 L CNN
-F 2 "" H 9550 4150 50  0001 C CNN
+F 2 "Connector_PinHeader_2.54mm:PinHeader_1x06_P2.54mm_Horizontal" H 9550 4150 50  0001 C CNN
 F 3 "" H 9550 4150 50  0001 C CNN
 	1    9550 3650
@@
 P 9600 4400
 AR Path="/61926AE2/61988A0E" Ref="#PWR?"  Part="1"
-AR Path="/61988A0E" Ref="#PWR05"  Part="1"
-F 0 "#PWR05" H 9600 4150 50  0001 C CNN
+AR Path="/61988A0E" Ref="#PWR0104"  Part="1"
+F 0 "#PWR0104" H 9600 4150 50  0001 C CNN
 F 1 "GND" H 9605 4227 50  0000 C CNN
 F 2 "" H 9600 4400 50  0001 C CNN
@@
 P 9600 3500
 AR Path="/61926AE2/6198A1ED" Ref="#PWR?"  Part="1"
-AR Path="/6198A1ED" Ref="#PWR04"  Part="1"
-F 0 "#PWR04" H 9600 3350 50  0001 C CNN
+AR Path="/6198A1ED" Ref="#PWR0103"  Part="1"
+F 0 "#PWR0103" H 9600 3350 50  0001 C CNN
 F 1 "+3.3V" H 9615 3673 50  0000 C CNN
 F 2 "" H 9600 3500 50  0001 C CNN
@@
 	9600 3500 9600 3550
 $Comp
-L Mechanical:MountingHole_Pad H1
+L Mechanical:MountingHole_Pad H100
 U 1 1 6198BDFD
 P 9350 850
-F 0 "H1" H 9450 899 50  0000 L CNN
+F 0 "H100" H 9450 899 50  0000 L CNN
 F 1 "MountingHole_Pad" H 9350 1100 50  0000 L CNN
-F 2 "" H 9350 850 50  0001 C CNN
+F 2 "MountingHole:MountingHole_3.2mm_M3_DIN965_Pad" H 9350 850 50  0001 C CNN
 F 3 "~" H 9350 850 50  0001 C CNN
 	1    9350 850
@@
 $EndComp
 $Comp
-L Mechanical:MountingHole_Pad H3
+L Mechanical:MountingHole_Pad H102
 U 1 1 6198CE4F
 P 9950 850
-F 0 "H3" H 10050 899 50  0000 L CNN
+F 0 "H102" H 10050 899 50  0000 L CNN
 F 1 "MountingHole_Pad" H 9350 1100 50  0000 L CNN
-F 2 "" H 9950 850 50  0001 C CNN
+F 2 "MountingHole:MountingHole_3.2mm_M3_DIN965_Pad" H 9950 850 50  0001 C CNN
 F 3 "~" H 9950 850 50  0001 C CNN
 	1    9950 850
@@
 $EndComp
 $Comp
-L Mechanical:MountingHole_Pad H2
+L Mechanical:MountingHole_Pad H101
 U 1 1 6198D15F
 P 9350 1350
-F 0 "H2" H 9450 1399 50  0000 L CNN
+F 0 "H101" H 9450 1399 50  0000 L CNN
 F 1 "MountingHole_Pad" H 9350 2100 50  0000 L CNN
-F 2 "" H 9350 1350 50  0001 C CNN
+F 2 "MountingHole:MountingHole_3.2mm_M3_DIN965_Pad" H 9350 1350 50  0001 C CNN
 F 3 "~" H 9350 1350 50  0001 C CNN
 	1    9350 1350
@@
 $EndComp
 $Comp
-L Mechanical:MountingHole_Pad H4
+L Mechanical:MountingHole_Pad H103
 U 1 1 6198D37A
 P 9950 1350
-F 0 "H4" H 10050 1399 50  0000 L CNN
+F 0 "H103" H 10050 1399 50  0000 L CNN
 F 1 "MountingHole_Pad" H 9350 2100 50  0000 L CNN
-F 2 "" H 9950 1350 50  0001 C CNN
+F 2 "MountingHole:MountingHole_3.2mm_M3_DIN965_Pad" H 9950 1350 50  0001 C CNN
 F 3 "~" H 9950 1350 50  0001 C CNN
 	1    9950 1350
@@
 P 9350 1450
 AR Path="/61926AE2/6198DDE0" Ref="#PWR?"  Part="1"
-AR Path="/6198DDE0" Ref="#PWR03"  Part="1"
-F 0 "#PWR03" H 9350 1200 50  0001 C CNN
+AR Path="/6198DDE0" Ref="#PWR0102"  Part="1"
+F 0 "#PWR0102" H 9350 1200 50  0001 C CNN
 F 1 "GND" H 9355 1277 50  0000 C CNN
 F 2 "" H 9350 1450 50  0001 C CNN
@@
 P 9950 1450
 AR Path="/61926AE2/6198E313" Ref="#PWR?"  Part="1"
-AR Path="/6198E313" Ref="#PWR07"  Part="1"
-F 0 "#PWR07" H 9950 1200 50  0001 C CNN
+AR Path="/6198E313" Ref="#PWR0106"  Part="1"
+F 0 "#PWR0106" H 9950 1200 50  0001 C CNN
 F 1 "GND" H 9955 1277 50  0000 C CNN
 F 2 "" H 9950 1450 50  0001 C CNN
@@
 P 9350 950
 AR Path="/61926AE2/6198E5F3" Ref="#PWR?"  Part="1"
-AR Path="/6198E5F3" Ref="#PWR02"  Part="1"
-F 0 "#PWR02" H 9350 700 50  0001 C CNN
+AR Path="/6198E5F3" Ref="#PWR0101"  Part="1"
+F 0 "#PWR0101" H 9350 700 50  0001 C CNN
 F 1 "GND" H 9355 777 50  0000 C CNN
 F 2 "" H 9350 950 50  0001 C CNN
@@
 P 9950 950
 AR Path="/61926AE2/6198E95A" Ref="#PWR?"  Part="1"
-AR Path="/6198E95A" Ref="#PWR06"  Part="1"
-F 0 "#PWR06" H 9950 700 50  0001 C CNN
+AR Path="/6198E95A" Ref="#PWR0105"  Part="1"
+F 0 "#PWR0105" H 9950 700 50  0001 C CNN
 F 1 "GND" H 9955 777 50  0000 C CNN
 F 2 "" H 9950 950 50  0001 C CNN
@@
 Wire Wire Line
 	8950 4200 9200 4200
+Wire Wire Line
+	6550 4100 6550 3900
+$Comp
+L power:PWR_FLAG #FLG0101
+U 1 1 61ACAB8C
+P 1450 800
+F 0 "#FLG0101" H 1450 875 50  0001 C CNN
+F 1 "PWR_FLAG" H 1450 973 50  0000 C CNN
+F 2 "" H 1450 800 50  0001 C CNN
+F 3 "~" H 1450 800 50  0001 C CNN
+	1    1450 800
+	1    0    0    -1
+$EndComp
+$Comp
+L power:PWR_FLAG #FLG0102
+U 1 1 61ACB040
+P 1900 950
+F 0 "#FLG0102" H 1900 1025 50  0001 C CNN
+F 1 "PWR_FLAG" H 1900 1123 50  0000 C CNN
+F 2 "" H 1900 950 50  0001 C CNN
+F 3 "~" H 1900 950 50  0001 C CNN
+	1    1900 950
+	-1   0    0    1
+$EndComp
+$Comp
+L power:+3.3V #PWR?
+U 1 1 61ACB2DF
+P 1900 800
+AR Path="/61926AE2/61ACB2DF" Ref="#PWR?"  Part="1"
+AR Path="/61ACB2DF" Ref="#PWR0107"  Part="1"
+F 0 "#PWR0107" H 1900 650 50  0001 C CNN
+F 1 "+3.3V" H 1915 973 50  0000 C CNN
+F 2 "" H 1900 800 50  0001 C CNN
+F 3 "" H 1900 800 50  0001 C CNN
+	1    1900 800
+	1    0    0    -1
+$EndComp
+Wire Wire Line
+	1900 950  1900 800
+$Comp
+L power:GND #PWR0108
+U 1 1 61ACDFF7
+P 1450 950
+F 0 "#PWR0108" H 1450 700 50  0001 C CNN
+F 1 "GND" H 1455 777 50  0000 C CNN
+F 2 "" H 1450 950 50  0001 C CNN
+F 3 "" H 1450 950 50  0001 C CNN
+	1    1450 950
+	1    0    0    -1
+$EndComp
+Wire Wire Line
+	1450 950  1450 800
+$Comp
+L power:PWR_FLAG #FLG0103
+U 1 1 61C1154B
+P 2850 3250
+F 0 "#FLG0103" H 2850 3325 50  0001 C CNN
+F 1 "PWR_FLAG" H 2850 3423 50  0000 C CNN
+F 2 "" H 2850 3250 50  0001 C CNN
+F 3 "~" H 2850 3250 50  0001 C CNN
+	1    2850 3250
+	1    0    0    -1
+$EndComp
+Wire Wire Line
+	2850 3250 2850 3300
+Connection ~ 2850 3300
 $EndSCHEMATC

Commit message: oh ya
Parts:
- added H104: MountingHole_Pad, MountingHole:MountingHole_3.2mm_M3_DIN965_Pad, symbol Mechanical:MountingHole_Pad
- added U101: E-ink_Display_Outline, batteryless_gaming_device:E-Ink_Display_1.54Inch, symbol batteryless_gaming_device-rescue:E-ink_Display_Outline
- U100: footprint Connector_PinHeader_2.54mm:PinHeader_1x06_P2.54mm_Horizontal -> Connector_PinHeader_2.54mm:PinHeader_1x08_P2.54mm_Horizontal
Connections:
- net GND: now also H104.1
Changed lines of the file:
@@
 F 0 "U100" H 9800 3800 50  0000 L CNN
 F 1 "E-Ink_Display_1.54Inch" H 9600 3700 50  0000 L CNN
-F 2 "Connector_PinHeader_2.54mm:PinHeader_1x06_P2.54mm_Horizontal" H 9550 4150 50  0001 C CNN
+F 2 "Connector_PinHeader_2.54mm:PinHeader_1x08_P2.54mm_Horizontal" H 9550 4150 50  0001 C CNN
 F 3 "" H 9550 4150 50  0001 C CNN
 	1    9550 3650
@@
 $EndComp
 Wire Notes Line
-	9100 500  9100 1700
+	9100 500  9100 2250
 Wire Notes Line
-	9100 1700 10500 1700
+	9100 2250 10500 2250
 Wire Wire Line
 	8950 3700 9200 3700
@@
 	2850 3250 2850 3300
 Connection ~ 2850 3300
+$Comp
+L batteryless_gaming_device-rescue:E-ink_Display_Outline U101
+U 1 1 6195AE48
+P 9650 4950
+F 0 "U101" H 9600 5050 50  0000 L CNN
+F 1 "E-ink_Display_Outline" H 9350 4950 50  0000 L CNN
+F 2 "batteryless_gaming_device:E-Ink_Display_1.54Inch" H 9650 4950 50  0001 C CNN
+F 3 "" H 9650 4950 50  0001 C CNN
+	1    9650 4950
+	1    0    0    -1
+$EndComp
+$Comp
+L Mechanical:MountingHole_Pad H104
+U 1 1 61AF7AB7
+P 9950 1900
+F 0 "H104" H 10050 1949 50  0000 L CNN
+F 1 "MountingHole_Pad" H 9350 3200 50  0000 L CNN
+F 2 "MountingHole:MountingHole_3.2mm_M3_DIN965_Pad" H 9950 1900 50  0001 C CNN
+F 3 "~" H 9950 1900 50  0001 C CNN
+	1    9950 1900
+	1    0    0    -1
+$EndComp
+$Comp
+L power:GND #PWR?
+U 1 1 61AF7ABD
+P 9950 2000
+AR Path="/61926AE2/61AF7ABD" Ref="#PWR?"  Part="1"
+AR Path="/61AF7ABD" Ref="#PWR0113"  Part="1"
+F 0 "#PWR0113" H 9950 1750 50  0001 C CNN
+F 1 "GND" H 9955 1827 50  0000 C CNN
+F 2 "" H 9950 2000 50  0001 C CNN
+F 3 "" H 9950 2000 50  0001 C CNN
+	1    9950 2000
+	1    0    0    -1
+$EndComp
 $EndSCHEMATC
