File: KiCad/batteryless_gaming_device/button_generation.sch (KiCad schematic (older format))
At the start: 12 parts

Commit message: updated schematic
Connections:
- net GPIO1 renamed Button1
- net GPIO2 renamed Button2
- net GPIO3 renamed Button3
- net GPIO4 renamed Button4
Changed lines of the file:
@@
 $Descr A4 11693 8268
 encoding utf-8
-Sheet 3 5
+Sheet 6 6
 Title ""
 Date ""
@@
 	3300 6500 3100 6500
 Text HLabel 3100 6500 0    50   Output ~ 0
-GPIO1
+Button1
 Text HLabel 7100 3650 2    50   Output ~ 0
 Vout
@@
 	3300 4950 3100 4950
 Text HLabel 3100 4950 0    50   Output ~ 0
-GPIO2
+Button2
 Wire Wire Line
 	3300 5400 3300 5350
@@
 	3300 3550 3100 3550
 Text HLabel 3100 3550 0    50   Output ~ 0
-GPIO3
+Button3
 Wire Wire Line
 	3300 4000 3300 3950
@@
 	3300 2150 3100 2150
 Text HLabel 3100 2150 0    50   Output ~ 0
-GPIO4
+Button4
 Wire Wire Line
 	3300 2600 3300 2550

Commit message: k
Parts:
- added R? (x4): 0, Resistor_SMD:R_0805_2012Metric_Pad1.20x1.40mm_HandSolder, symbol Device:R_US
Connections:
- net Vout: now also R?.2, R?.2, R?.2, R?.2; no longer D?.1 (+), D?.1 (+), D?.1 (+), D?.1 (+)
- new net: D?.1 (+), R?.1 (x3)
Changed lines of the file:
@@
 	3300 2600 3300 2550
 Wire Wire Line
-	5100 1850 6550 1850
+	6550 3650 7100 3650
+Connection ~ 6550 3650
 Wire Wire Line
 	6550 1850 6550 3250
 Wire Wire Line
-	6550 3650 7100 3650
+	6550 3650 6550 4650
+$Comp
+L Device:R_US R?
+U 1 1 619B6F67
+P 6100 6200
+AR Path="/61926AE2/619B6F67" Ref="R?"  Part="1"
+AR Path="/619B6F67" Ref="R?"  Part="1"
+AR Path="/619E7D55/619B6F67" Ref="R?"  Part="1"
+F 0 "R?" V 6250 6150 50  0000 L CNN
+F 1 "0" V 6168 6155 50  0000 L CNN
+F 2 "Resistor_SMD:R_0805_2012Metric_Pad1.20x1.40mm_HandSolder" V 6140 6190 50  0001 C CNN
+F 3 "~" H 6100 6200 50  0001 C CNN
+F 4 "YAG3755CT-ND" V 6000 6200 39  0000 C CNN "Digikey PN"
+	1    6100 6200
+	0    -1   -1   0
+$EndComp
 Wire Wire Line
-	5100 3250 6550 3250
+	5150 6200 5950 6200
+Wire Wire Line
+	6250 6200 6550 6200
+$Comp
+L Device:R_US R?
+U 1 1 619BB780
+P 6050 4650
+AR Path="/61926AE2/619BB780" Ref="R?"  Part="1"
+AR Path="/619BB780" Ref="R?"  Part="1"
+AR Path="/619E7D55/619BB780" Ref="R?"  Part="1"
+F 0 "R?" V 6200 4600 50  0000 L CNN
+F 1 "0" V 6118 4605 50  0000 L CNN
+F 2 "Resistor_SMD:R_0805_2012Metric_Pad1.20x1.40mm_HandSolder" V 6090 4640 50  0001 C CNN
+F 3 "~" H 6050 4650 50  0001 C CNN
+F 4 "YAG3755CT-ND" V 5950 4650 39  0000 C CNN "Digikey PN"
+	1    6050 4650
+	0    -1   -1   0
+$EndComp
+Wire Wire Line
+	5100 4650 5900 4650
+Wire Wire Line
+	6200 4650 6550 4650
+Connection ~ 6550 4650
+Wire Wire Line
+	6550 4650 6550 6200
+$Comp
+L Device:R_US R?
+U 1 1 619C0235
+P 6050 1850
+AR Path="/61926AE2/619C0235" Ref="R?"  Part="1"
+AR Path="/619C0235" Ref="R?"  Part="1"
+AR Path="/619E7D55/619C0235" Ref="R?"  Part="1"
+F 0 "R?" V 6200 1800 50  0000 L CNN
+F 1 "0" V 6118 1805 50  0000 L CNN
+F 2 "Resistor_SMD:R_0805_2012Metric_Pad1.20x1.40mm_HandSolder" V 6090 1840 50  0001 C CNN
+F 3 "~" H 6050 1850 50  0001 C CNN
+F 4 "YAG3755CT-ND" V 5950 1850 39  0000 C CNN "Digikey PN"
+	1    6050 1850
+	0    -1   -1   0
+$EndComp
+Wire Wire Line
+	5100 1850 5900 1850
+Wire Wire Line
+	6200 1850 6550 1850
+$Comp
+L Device:R_US R?
+U 1 1 619C6E50
+P 6100 3250
+AR Path="/61926AE2/619C6E50" Ref="R?"  Part="1"
+AR Path="/619C6E50" Ref="R?"  Part="1"
+AR Path="/619E7D55/619C6E50" Ref="R?"  Part="1"
+F 0 "R?" V 6250 3200 50  0000 L CNN
+F 1 "0" V 6168 3205 50  0000 L CNN
+F 2 "Resistor_SMD:R_0805_2012Metric_Pad1.20x1.40mm_HandSolder" V 6140 3240 50  0001 C CNN
+F 3 "~" H 6100 3250 50  0001 C CNN
+F 4 "YAG3755CT-ND" V 6000 3250 39  0000 C CNN "Digikey PN"
+	1    6100 3250
+	0    -1   -1   0
+$EndComp
+Wire Wire Line
+	5100 3250 5950 3250
+Wire Wire Line
+	6250 3250 6550 3250
 Connection ~ 6550 3250
 Wire Wire Line
 	6550 3250 6550 3650
-Wire Wire Line
-	5100 4650 6550 4650
-Wire Wire Line
-	6550 4650 6550 3650
-Connection ~ 6550 3650
-Wire Wire Line
-	5100 6200 6550 6200
-Wire Wire Line
-	6550 6200 6550 4650
-Connection ~ 6550 4650
 $EndSCHEMATC

Commit message: k
Parts:
- gave numbers to parts that had none: 16
Changed lines of the file:
@@
 $EndDescr
 $Comp
-L batteryless_gaming_device-rescue:EH_switch SW?
+L batteryless_gaming_device-rescue:EH_switch SW5
 U 1 1 61A3608F
 P 3600 6450
-F 0 "SW?" H 3600 6909 50  0000 C CNN
+F 0 "SW5" H 3600 6909 50  0000 C CNN
 F 1 "EH_switch" H 3600 6818 50  0000 C CNN
 F 2 "" H 3800 6150 50  0001 C CNN
@@
 $EndComp
 $Comp
-L Device:D_Bridge_+-AA D?
+L Device:D_Bridge_+-AA D6
 U 1 1 61A43A75
 P 4800 6200
-F 0 "D?" H 5144 6246 50  0000 L CNN
+F 0 "D6" H 5144 6246 50  0000 L CNN
 F 1 "D_Bridge_+-AA" H 5144 6155 50  0000 L CNN
 F 2 "" H 4800 6200 50  0001 C CNN
@@
 	4800 6650 4800 6500
 $Comp
-L power:GND #PWR?
+L power:GND #PWR037
 U 1 1 61A46511
 P 4450 6350
-F 0 "#PWR?" H 4450 6100 50  0001 C CNN
+F 0 "#PWR037" H 4450 6100 50  0001 C CNN
 F 1 "GND" H 4455 6177 50  0000 C CNN
 F 2 "" H 4450 6350 50  0001 C CNN
@@
 	4450 6200 4500 6200
 $Comp
-L Device:R_US R?
+L Device:R_US R21
 U 1 1 61A486D7
 P 3300 6750
-F 0 "R?" H 3368 6796 50  0000 L CNN
+F 0 "R21" H 3368 6796 50  0000 L CNN
 F 1 "1M" H 3368 6705 50  0000 L CNN
 F 2 "" V 3340 6740 50  0001 C CNN
@@
 Connection ~ 3300 6500
 $Comp
-L power:+3.3V #PWR?
+L power:+3.3V #PWR033
 U 1 1 61A50806
 P 3300 6950
-F 0 "#PWR?" H 3300 6800 50  0001 C CNN
+F 0 "#PWR033" H 3300 6800 50  0001 C CNN
 F 1 "+3.3V" H 3315 7123 50  0000 C CNN
 F 2 "" H 3300 6950 50  0001 C CNN
@@
 	3300 6950 3300 6900
 $Comp
-L batteryless_gaming_device-rescue:EH_switch SW?
+L batteryless_gaming_device-rescue:EH_switch SW4
 U 1 1 61A58E70
 P 3600 4900
-F 0 "SW?" H 3600 5359 50  0000 C CNN
+F 0 "SW4" H 3600 5359 50  0000 C CNN
 F 1 "EH_switch" H 3600 5268 50  0000 C CNN
 F 2 "" H 3800 4600 50  0001 C CNN
@@
 $EndComp
 $Comp
-L Device:D_Bridge_+-AA D?
+L Device:D_Bridge_+-AA D5
 U 1 1 61A58E76
 P 4800 4650
-F 0 "D?" H 5144 4696 50  0000 L CNN
+F 0 "D5" H 5144 4696 50  0000 L CNN
 F 1 "D_Bridge_+-AA" H 5144 4605 50  0000 L CNN
 F 2 "" H 4800 4650 50  0001 C CNN
@@
 	4800 5100 4800 4950
 $Comp
-L power:GND #PWR?
+L power:GND #PWR036
 U 1 1 61A58E84
 P 4450 4800
-F 0 "#PWR?" H 4450 4550 50  0001 C CNN
+F 0 "#PWR036" H 4450 4550 50  0001 C CNN
 F 1 "GND" H 4455 4627 50  0000 C CNN
 F 2 "" H 4450 4800 50  0001 C CNN
@@
 	4450 4650 4500 4650
 $Comp
-L Device:R_US R?
+L Device:R_US R20
 U 1 1 61A58E8C
 P 3300 5200
-F 0 "R?" H 3368 5246 50  0000 L CNN
+F 0 "R20" H 3368 5246 50  0000 L CNN
 F 1 "1M" H 3368 5155 50  0000 L CNN
 F 2 "" V 3340 5190 50  0001 C CNN
@@
 Connection ~ 3300 4950
 $Comp
-L power:+3.3V #PWR?
+L power:+3.3V #PWR032
 U 1 1 61A58E97
 P 3300 5400
-F 0 "#PWR?" H 3300 5250 50  0001 C CNN
+F 0 "#PWR032" H 3300 5250 50  0001 C CNN
 F 1 "+3.3V" H 3315 5573 50  0000 C CNN
 F 2 "" H 3300 5400 50  0001 C CNN
@@
 	3300 5400 3300 5350
 $Comp
-L batteryless_gaming_device-rescue:EH_switch SW?
+L batteryless_gaming_device-rescue:EH_switch SW3
 U 1 1 61A5B26C
 P 3600 3500
-F 0 "SW?" H 3600 3959 50  0000 C CNN
+F 0 "SW3" H 3600 3959 50  0000 C CNN
 F 1 "EH_switch" H 3600 3868 50  0000 C CNN
 F 2 "" H 3800 3200 50  0001 C CNN
@@
 $EndComp
 $Comp
-L Device:D_Bridge_+-AA D?
+L Device:D_Bridge_+-AA D4
 U 1 1 61A5B272
 P 4800 3250
-F 0 "D?" H 5144 3296 50  0000 L CNN
+F 0 "D4" H 5144 3296 50  0000 L CNN
 F 1 "D_Bridge_+-AA" H 5144 3205 50  0000 L CNN
 F 2 "" H 4800 3250 50  0001 C CNN
@@
 	4800 3700 4800 3550
 $Comp
-L power:GND #PWR?
+L power:GND #PWR035
 U 1 1 61A5B280
 P 4450 3400
-F 0 "#PWR?" H 4450 3150 50  0001 C CNN
+F 0 "#PWR035" H 4450 3150 50  0001 C CNN
 F 1 "GND" H 4455 3227 50  0000 C CNN
 F 2 "" H 4450 3400 50  0001 C CNN
@@
 	4450 3250 4500 3250
 $Comp
-L Device:R_US R?
+L Device:R_US R19
 U 1 1 61A5B288
 P 3300 3800
-F 0 "R?" H 3368 3846 50  0000 L CNN
+F 0 "R19" H 3368 3846 50  0000 L CNN
 F 1 "1M" H 3368 3755 50  0000 L CNN
 F 2 "" V 3340 3790 50  0001 C CNN
@@
 Connection ~ 3300 3550
 $Comp
-L power:+3.3V #PWR?
+L power:+3.3V #PWR031
 U 1 1 61A5B293
 P 3300 4000
-F 0 "#PWR?" H 3300 3850 50  0001 C CNN
+F 0 "#PWR031" H 3300 3850 50  0001 C CNN
 F 1 "+3.3V" H 3315 4173 50  0000 C CNN
 F 2 "" H 3300 4000 50  0001 C CNN
@@
 	3300 4000 3300 3950
 $Comp
-L batteryless_gaming_device-rescue:EH_switch SW?
+L batteryless_gaming_device-rescue:EH_switch SW2
 U 1 1 61A5E757
 P 3600 2100
-F 0 "SW?" H 3600 2559 50  0000 C CNN
+F 0 "SW2" H 3600 2559 50  0000 C CNN
 F 1 "EH_switch" H 3600 2468 50  0000 C CNN
 F 2 "" H 3800 1800 50  0001 C CNN
@@
 $EndComp
 $Comp
-L Device:D_Bridge_+-AA D?
+L Device:D_Bridge_+-AA D3
 U 1 1 61A5E75D
 P 4800 1850
-F 0 "D?" H 5144 1896 50  0000 L CNN
+F 0 "D3" H 5144 1896 50  0000 L CNN
 F 1 "D_Bridge_+-AA" H 5144 1805 50  0000 L CNN
 F 2 "" H 4800 1850 50  0001 C CNN
@@
 	4800 2300 4800 2150
 $Comp
-L power:GND #PWR?
+L power:GND #PWR034
 U 1 1 61A5E76B
 P 4450 2000
-F 0 "#PWR?" H 4450 1750 50  0001 C CNN
+F 0 "#PWR034" H 4450 1750 50  0001 C CNN
 F 1 "GND" H 4455 1827 50  0000 C CNN
 F 2 "" H 4450 2000 50  0001 C CNN
@@
 	4450 1850 4500 1850
 $Comp
-L Device:R_US R?
+L Device:R_US R18
 U 1 1 61A5E773
 P 3300 2400
-F 0 "R?" H 3368 2446 50  0000 L CNN
+F 0 "R18" H 3368 2446 50  0000 L CNN
 F 1 "1M" H 3368 2355 50  0000 L CNN
 F 2 "" V 3340 2390 50  0001 C CNN
@@
 Connection ~ 3300 2150
 $Comp
-L power:+3.3V #PWR?
+L power:+3.3V #PWR030
 U 1 1 61A5E77E
 P 3300 2600
-F 0 "#PWR?" H 3300 2450 50  0001 C CNN
+F 0 "#PWR030" H 3300 2450 50  0001 C CNN
 F 1 "+3.3V" H 3315 2773 50  0000 C CNN
 F 2 "" H 3300 2600 50  0001 C CNN
@@
 AR Path="/61926AE2/619B6F67" Ref="R?"  Part="1"
 AR Path="/619B6F67" Ref="R?"  Part="1"
-AR Path="/619E7D55/619B6F67" Ref="R?"  Part="1"
-F 0 "R?" V 6250 6150 50  0000 L CNN
+AR Path="/619E7D55/619B6F67" Ref="R25"  Part="1"
+F 0 "R25" V 6250 6150 50  0000 L CNN
 F 1 "0" V 6168 6155 50  0000 L CNN
 F 2 "Resistor_SMD:R_0805_2012Metric_Pad1.20x1.40mm_HandSolder" V 6140 6190 50  0001 C CNN
@@
 AR Path="/61926AE2/619BB780" Ref="R?"  Part="1"
 AR Path="/619BB780" Ref="R?"  Part="1"
-AR Path="/619E7D55/619BB780" Ref="R?"  Part="1"
-F 0 "R?" V 6200 4600 50  0000 L CNN
+AR Path="/619E7D55/619BB780" Ref="R23"  Part="1"
+F 0 "R23" V 6200 4600 50  0000 L CNN
 F 1 "0" V 6118 4605 50  0000 L CNN
 F 2 "Resistor_SMD:R_0805_2012Metric_Pad1.20x1.40mm_HandSolder" V 6090 4640 50  0001 C CNN
@@
 AR Path="/61926AE2/619C0235" Ref="R?"  Part="1"
 AR Path="/619C0235" Ref="R?"  Part="1"
-AR Path="/619E7D55/619C0235" Ref="R?"  Part="1"
-F 0 "R?" V 6200 1800 50  0000 L CNN
+AR Path="/619E7D55/619C0235" Ref="R22"  Part="1"
+F 0 "R22" V 6200 1800 50  0000 L CNN
 F 1 "0" V 6118 1805 50  0000 L CNN
 F 2 "Resistor_SMD:R_0805_2012Metric_Pad1.20x1.40mm_HandSolder" V 6090 1840 50  0001 C CNN
@@
 AR Path="/61926AE2/619C6E50" Ref="R?"  Part="1"
 AR Path="/619C6E50" Ref="R?"  Part="1"
-AR Path="/619E7D55/619C6E50" Ref="R?"  Part="1"
-F 0 "R?" V 6250 3200 50  0000 L CNN
+AR Path="/619E7D55/619C6E50" Ref="R24"  Part="1"
+F 0 "R24" V 6250 3200 50  0000 L CNN
 F 1 "0" V 6168 3205 50  0000 L CNN
 F 2 "Resistor_SMD:R_0805_2012Metric_Pad1.20x1.40mm_HandSolder" V 6140 3240 50  0001 C CNN

Commit message: k
Parts:
- added C24, C25, C26, C27: 1nF, Capacitor_SMD:C_0603_1608Metric_Pad1.08x0.95mm_HandSolder, symbol Device:C
- renumbered R18 to R20, R19 to R21, R20 to R22, R21 to R23, R22 to R24, R23 to R25, R24 to R26, R25 to R27
Connections:
- net +3V3: now also C24.2, C25.2, C26.2, C27.2
- net Button1: now also C27.1
- net Button2: now also C26.1
- net Button3: now also C25.1
- net Button4: now also C24.1
Other:
- note added: "DNU"
Changed lines of the file:
@@
 	4800 6650 4800 6500
 $Comp
-L power:GND #PWR037
+L power:GND #PWR038
 U 1 1 61A46511
 P 4450 6350
-F 0 "#PWR037" H 4450 6100 50  0001 C CNN
+F 0 "#PWR038" H 4450 6100 50  0001 C CNN
 F 1 "GND" H 4455 6177 50  0000 C CNN
 F 2 "" H 4450 6350 50  0001 C CNN
@@
 	4450 6200 4500 6200
 $Comp
-L Device:R_US R21
+L Device:R_US R23
 U 1 1 61A486D7
 P 3300 6750
-F 0 "R21" H 3368 6796 50  0000 L CNN
+F 0 "R23" H 3368 6796 50  0000 L CNN
 F 1 "1M" H 3368 6705 50  0000 L CNN
 F 2 "" V 3340 6740 50  0001 C CNN
@@
 $EndComp
 Wire Wire Line
-	3300 6600 3300 6500
+	3300 6600 3300 6550
 Wire Wire Line
 	3300 6500 3400 6500
@@
 Connection ~ 3300 6500
 $Comp
-L power:+3.3V #PWR033
+L power:+3.3V #PWR034
 U 1 1 61A50806
 P 3300 6950
-F 0 "#PWR033" H 3300 6800 50  0001 C CNN
+F 0 "#PWR034" H 3300 6800 50  0001 C CNN
 F 1 "+3.3V" H 3315 7123 50  0000 C CNN
 F 2 "" H 3300 6950 50  0001 C CNN
@@
 	4800 5100 4800 4950
 $Comp
-L power:GND #PWR036
+L power:GND #PWR037
 U 1 1 61A58E84
 P 4450 4800
-F 0 "#PWR036" H 4450 4550 50  0001 C CNN
+F 0 "#PWR037" H 4450 4550 50  0001 C CNN
 F 1 "GND" H 4455 4627 50  0000 C CNN
 F 2 "" H 4450 4800 50  0001 C CNN
@@
 	4450 4650 4500 4650
 $Comp
-L Device:R_US R20
+L Device:R_US R22
 U 1 1 61A58E8C
 P 3300 5200
-F 0 "R20" H 3368 5246 50  0000 L CNN
+F 0 "R22" H 3368 5246 50  0000 L CNN
 F 1 "1M" H 3368 5155 50  0000 L CNN
 F 2 "" V 3340 5190 50  0001 C CNN
@@
 Connection ~ 3300 4950
 $Comp
-L power:+3.3V #PWR032
+L power:+3.3V #PWR033
 U 1 1 61A58E97
 P 3300 5400
-F 0 "#PWR032" H 3300 5250 50  0001 C CNN
+F 0 "#PWR033" H 3300 5250 50  0001 C CNN
 F 1 "+3.3V" H 3315 5573 50  0000 C CNN
 F 2 "" H 3300 5400 50  0001 C CNN
@@
 	4800 3700 4800 3550
 $Comp
-L power:GND #PWR035
+L power:GND #PWR036
 U 1 1 61A5B280
 P 4450 3400
-F 0 "#PWR035" H 4450 3150 50  0001 C CNN
+F 0 "#PWR036" H 4450 3150 50  0001 C CNN
 F 1 "GND" H 4455 3227 50  0000 C CNN
 F 2 "" H 4450 3400 50  0001 C CNN
@@
 	4450 3250 4500 3250
 $Comp
-L Device:R_US R19
+L Device:R_US R21
 U 1 1 61A5B288
 P 3300 3800
-F 0 "R19" H 3368 3846 50  0000 L CNN
+F 0 "R21" H 3368 3846 50  0000 L CNN
 F 1 "1M" H 3368 3755 50  0000 L CNN
 F 2 "" V 3340 3790 50  0001 C CNN
@@
 Connection ~ 3300 3550
 $Comp
-L power:+3.3V #PWR031
+L power:+3.3V #PWR032
 U 1 1 61A5B293
 P 3300 4000
-F 0 "#PWR031" H 3300 3850 50  0001 C CNN
+F 0 "#PWR032" H 3300 3850 50  0001 C CNN
 F 1 "+3.3V" H 3315 4173 50  0000 C CNN
 F 2 "" H 3300 4000 50  0001 C CNN
@@
 	4800 2300 4800 2150
 $Comp
-L power:GND #PWR034
+L power:GND #PWR035
 U 1 1 61A5E76B
 P 4450 2000
-F 0 "#PWR034" H 4450 1750 50  0001 C CNN
+F 0 "#PWR035" H 4450 1750 50  0001 C CNN
 F 1 "GND" H 4455 1827 50  0000 C CNN
 F 2 "" H 4450 2000 50  0001 C CNN
@@
 	4450 1850 4500 1850
 $Comp
-L Device:R_US R18
+L Device:R_US R20
 U 1 1 61A5E773
 P 3300 2400
-F 0 "R18" H 3368 2446 50  0000 L CNN
+F 0 "R20" H 3368 2446 50  0000 L CNN
 F 1 "1M" H 3368 2355 50  0000 L CNN
 F 2 "" V 3340 2390 50  0001 C CNN
@@
 Connection ~ 3300 2150
 $Comp
-L power:+3.3V #PWR030
+L power:+3.3V #PWR031
 U 1 1 61A5E77E
 P 3300 2600
-F 0 "#PWR030" H 3300 2450 50  0001 C CNN
+F 0 "#PWR031" H 3300 2450 50  0001 C CNN
 F 1 "+3.3V" H 3315 2773 50  0000 C CNN
 F 2 "" H 3300 2600 50  0001 C CNN
@@
 AR Path="/61926AE2/619B6F67" Ref="R?"  Part="1"
 AR Path="/619B6F67" Ref="R?"  Part="1"
-AR Path="/619E7D55/619B6F67" Ref="R25"  Part="1"
-F 0 "R25" V 6250 6150 50  0000 L CNN
+AR Path="/619E7D55/619B6F67" Ref="R27"  Part="1"
+F 0 "R27" V 6250 6150 50  0000 L CNN
 F 1 "0" V 6168 6155 50  0000 L CNN
 F 2 "Resistor_SMD:R_0805_2012Metric_Pad1.20x1.40mm_HandSolder" V 6140 6190 50  0001 C CNN
@@
 AR Path="/61926AE2/619BB780" Ref="R?"  Part="1"
 AR Path="/619BB780" Ref="R?"  Part="1"
-AR Path="/619E7D55/619BB780" Ref="R23"  Part="1"
-F 0 "R23" V 6200 4600 50  0000 L CNN
+AR Path="/619E7D55/619BB780" Ref="R25"  Part="1"
+F 0 "R25" V 6200 4600 50  0000 L CNN
 F 1 "0" V 6118 4605 50  0000 L CNN
 F 2 "Resistor_SMD:R_0805_2012Metric_Pad1.20x1.40mm_HandSolder" V 6090 4640 50  0001 C CNN
@@
 AR Path="/61926AE2/619C0235" Ref="R?"  Part="1"
 AR Path="/619C0235" Ref="R?"  Part="1"
-AR Path="/619E7D55/619C0235" Ref="R22"  Part="1"
-F 0 "R22" V 6200 1800 50  0000 L CNN
+AR Path="/619E7D55/619C0235" Ref="R24"  Part="1"
+F 0 "R24" V 6200 1800 50  0000 L CNN
 F 1 "0" V 6118 1805 50  0000 L CNN
 F 2 "Resistor_SMD:R_0805_2012Metric_Pad1.20x1.40mm_HandSolder" V 6090 1840 50  0001 C CNN
@@
 AR Path="/61926AE2/619C6E50" Ref="R?"  Part="1"
 AR Path="/619C6E50" Ref="R?"  Part="1"
-AR Path="/619E7D55/619C6E50" Ref="R24"  Part="1"
-F 0 "R24" V 6250 3200 50  0000 L CNN
+AR Path="/619E7D55/619C6E50" Ref="R26"  Part="1"
+F 0 "R26" V 6250 3200 50  0000 L CNN
 F 1 "0" V 6168 3205 50  0000 L CNN
 F 2 "Resistor_SMD:R_0805_2012Metric_Pad1.20x1.40mm_HandSolder" V 6140 3240 50  0001 C CNN
@@
 Wire Wire Line
 	6550 3250 6550 3650
+Wire Wire Line
+	3300 6550 3700 6550
+Wire Wire Line
+	3700 6550 3700 6600
+Connection ~ 3300 6550
+Wire Wire Line
+	3300 6550 3300 6500
+Wire Wire Line
+	3300 6900 3700 6900
+Connection ~ 3300 6900
+$Comp
+L Device:C C?
+U 1 1 61A0A80F
+P 3700 6750
+AR Path="/61926AE2/61A0A80F" Ref="C?"  Part="1"
+AR Path="/619E7D55/61A0A80F" Ref="C27"  Part="1"
+F 0 "C27" H 3815 6796 50  0000 L CNN
+F 1 "1nF" H 3815 6705 50  0000 L CNN
+F 2 "Capacitor_SMD:C_0603_1608Metric_Pad1.08x0.95mm_HandSolder" H 3738 6600 50  0001 C CNN
+F 3 "~" H 3700 6750 50  0001 C CNN
+F 4 "1276-CL10B102KB8WPJCCT-ND" H 4200 6600 39  0000 C CNN "Digikey PN"
+	1    3700 6750
+	1    0    0    -1
+$EndComp
+Text Notes 3900 7050 2    50   ~ 0
+DNU
+Wire Wire Line
+	3300 5350 3700 5350
+$Comp
+L Device:C C?
+U 1 1 61A12CCE
+P 3700 5200
+AR Path="/61926AE2/61A12CCE" Ref="C?"  Part="1"
+AR Path="/619E7D55/61A12CCE" Ref="C26"  Part="1"
+F 0 "C26" H 3815 5246 50  0000 L CNN
+F 1 "1nF" H 3815 5155 50  0000 L CNN
+F 2 "Capacitor_SMD:C_0603_1608Metric_Pad1.08x0.95mm_HandSolder" H 3738 5050 50  0001 C CNN
+F 3 "~" H 3700 5200 50  0001 C CNN
+F 4 "1276-CL10B102KB8WPJCCT-ND" H 4200 5050 39  0000 C CNN "Digikey PN"
+	1    3700 5200
+	1    0    0    -1
+$EndComp
+Text Notes 3900 5500 2    50   ~ 0
+DNU
+Wire Wire Line
+	3300 3950 3700 3950
+$Comp
+L Device:C C?
+U 1 1 61A14E5F
+P 3700 3800
+AR Path="/61926AE2/61A14E5F" Ref="C?"  Part="1"
+AR Path="/619E7D55/61A14E5F" Ref="C25"  Part="1"
+F 0 "C25" H 3815 3846 50  0000 L CNN
+F 1 "1nF" H 3815 3755 50  0000 L CNN
+F 2 "Capacitor_SMD:C_0603_1608Metric_Pad1.08x0.95mm_HandSolder" H 3738 3650 50  0001 C CNN
+F 3 "~" H 3700 3800 50  0001 C CNN
+F 4 "1276-CL10B102KB8WPJCCT-ND" H 4200 3650 39  0000 C CNN "Digikey PN"
+	1    3700 3800
+	1    0    0    -1
+$EndComp
+Text Notes 3900 4100 2    50   ~ 0
+DNU
+Wire Wire Line
+	3300 2550 3700 2550
+$Comp
+L Device:C C?
+U 1 1 61A16E18
+P 3700 2400
+AR Path="/61926AE2/61A16E18" Ref="C?"  Part="1"
+AR Path="/619E7D55/61A16E18" Ref="C24"  Part="1"
+F 0 "C24" H 3815 2446 50  0000 L CNN
+F 1 "1nF" H 3815 2355 50  0000 L CNN
+F 2 "Capacitor_SMD:C_0603_1608Metric_Pad1.08x0.95mm_HandSolder" H 3738 2250 50  0001 C CNN
+F 3 "~" H 3700 2400 50  0001 C CNN
+F 4 "1276-CL10B102KB8WPJCCT-ND" H 4200 2250 39  0000 C CNN "Digikey PN"
+	1    3700 2400
+	1    0    0    -1
+$EndComp
+Text Notes 3900 2700 2    50   ~ 0
+DNU
+Wire Wire Line
+	3700 2250 3300 2250
+Connection ~ 3300 2250
+Wire Wire Line
+	3700 3650 3300 3650
+Connection ~ 3300 3650
+Wire Wire Line
+	3700 5050 3300 5050
+Connection ~ 3300 5050
 $EndSCHEMATC

Commit message: just kinda out here guys ya know what im saying
Parts:
- D600: renamed from D3; footprint (none) -> Package_TO_SOT_SMD:TO-269AA; Digikey PN (none) -> 641-1213-1-ND
- D601: renamed from D4; footprint (none) -> Package_TO_SOT_SMD:TO-269AA; Digikey PN (none) -> 641-1213-1-ND
- D602: renamed from D5; footprint (none) -> Package_TO_SOT_SMD:TO-269AA; Digikey PN (none) -> 641-1213-1-ND
- D603: renamed from D6; footprint (none) -> Package_TO_SOT_SMD:TO-269AA; Digikey PN (none) -> 641-1213-1-ND
- R600: renamed from R20; footprint (none) -> Resistor_SMD:R_0603_1608Metric_Pad0.98x0.95mm_HandSolder; Digikey PN (none) -> 511-1820-1-ND
- R601: renamed from R21; footprint (none) -> Resistor_SMD:R_0603_1608Metric_Pad0.98x0.95mm_HandSolder; Digikey PN (none) -> 511-1820-1-ND
- R602: renamed from R22; footprint (none) -> Resistor_SMD:R_0603_1608Metric_Pad0.98x0.95mm_HandSolder; Digikey PN (none) -> 511-1820-1-ND
- R603: renamed from R23; footprint (none) -> Resistor_SMD:R_0603_1608Metric_Pad0.98x0.95mm_HandSolder; Digikey PN (none) -> 511-1820-1-ND
- SW600: renamed from SW2; footprint (none) -> batteryless_gaming_device:EH_switch
- SW601: renamed from SW3; footprint (none) -> batteryless_gaming_device:EH_switch
- SW602: renamed from SW4; footprint (none) -> batteryless_gaming_device:EH_switch
- SW603: renamed from SW5; footprint (none) -> batteryless_gaming_device:EH_switch
- renumbered C24 to C600, C25 to C601, C26 to C602, C27 to C603, R24 to R604, R25 to R605, R26 to R606, R27 to R607
Connections:
- net GND: now also SW600.6 (A), SW600.7 (K), SW601.6 (A), SW601.7 (K), SW602.6 (A), SW602.7 (K), SW603.6 (A), SW603.7 (K)
- net at R607.1: now also D603.1 (+)
- no-connect marks 0 -> 4

Commit message: oh ya
Parts:
- SW600, SW601, SW602, SW603: footprint batteryless_gaming_device:EH_switch -> batteryless_gaming_device:EH_switch_v2
Changed lines of the file:
@@
 F 0 "SW603" H 3600 6909 50  0000 C CNN
 F 1 "EH_switch" H 3600 6818 50  0000 C CNN
-F 2 "batteryless_gaming_device:EH_switch" H 3800 6150 50  0001 C CNN
+F 2 "batteryless_gaming_device:EH_switch_v2" H 3800 6150 50  0001 C CNN
 F 3 "" H 3600 6450 50  0001 C CNN
 F 4 "CH721-ND;EG5982-ND" H 3600 6735 39  0000 C CNN "Digikey PN"
@@
 F 0 "SW602" H 3600 5359 50  0000 C CNN
 F 1 "EH_switch" H 3600 5268 50  0000 C CNN
-F 2 "batteryless_gaming_device:EH_switch" H 3800 4600 50  0001 C CNN
+F 2 "batteryless_gaming_device:EH_switch_v2" H 3800 4600 50  0001 C CNN
 F 3 "" H 3600 4900 50  0001 C CNN
 F 4 "CH721-ND;EG5982-ND" H 3600 5185 39  0000 C CNN "Digikey PN"
@@
 F 0 "SW601" H 3600 3959 50  0000 C CNN
 F 1 "EH_switch" H 3600 3868 50  0000 C CNN
-F 2 "batteryless_gaming_device:EH_switch" H 3800 3200 50  0001 C CNN
+F 2 "batteryless_gaming_device:EH_switch_v2" H 3800 3200 50  0001 C CNN
 F 3 "" H 3600 3500 50  0001 C CNN
 F 4 "CH721-ND;EG5982-ND" H 3600 3785 39  0000 C CNN "Digikey PN"
@@
 F 0 "SW600" H 3600 2559 50  0000 C CNN
 F 1 "EH_switch" H 3600 2468 50  0000 C CNN
-F 2 "batteryless_gaming_device:EH_switch" H 3800 1800 50  0001 C CNN
+F 2 "batteryless_gaming_device:EH_switch_v2" H 3800 1800 50  0001 C CNN
 F 3 "" H 3600 2100 50  0001 C CNN
 F 4 "CH721-ND;EG5982-ND" H 3600 2385 39  0000 C CNN "Digikey PN"
