File: KiCad/batteryless_gaming_device/batteryless_gaming_device.kicad_pcb (KiCad board)
At the start: 2 copper layers, 6 x 6 mm, 88 parts, among them J100 Voltage Source Select, J400 GPIO_breakout, J401 Multiplayer_Connector, J402 Program_Header, M300 Hand Generator, SW400 FSMSM, SW600 EH_switch, SW601 EH_switch, SW602 EH_switch, SW603 EH_switch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

Commit message: oh ya
Parts:
- removed C203: 10uF, Capacitor_SMD:C_0805_2012Metric_Pad1.18x1.45mm_HandSolder
- removed C403: 0.1uF, Capacitor_SMD:C_0603_1608Metric_Pad1.08x0.95mm_HandSolder
- added H104: MountingHole_Pad, MountingHole:MountingHole_3.2mm_M3_DIN965_Pad, F.Cu at (121.7, 122.1)
- added U101: E-ink_Display_Outline, batteryless_gaming_device:E-Ink_Display_1.54Inch, F.Cu at (91.1, 75.2)
- J400: footprint Connector_PinHeader_2.54mm:PinHeader_1x06_P2.54mm_Vertical -> Connector_PinHeader_2.54mm:PinHeader_1x04_P2.54mm_Vertical
- M300: footprint Connector_PinHeader_2.54mm:PinHeader_1x03_P2.54mm_Vertical -> Connector_PinHeader_2.00mm:PinHeader_1x03_P2.00mm_Vertical
- SW600, SW601, SW602, SW603: footprint batteryless_gaming_device:EH_switch -> batteryless_gaming_device:EH_switch_v2
- U100: footprint Connector_PinHeader_2.54mm:PinHeader_1x06_P2.54mm_Horizontal -> Connector_PinHeader_2.54mm:PinHeader_1x08_P2.54mm_Horizontal
- U400: value MSP430FR5994 -> MSP430FR5994IPM
- moved R301 106.0 mm to (82.3, 91.6), turned to 270 degrees
- moved R300 105.7 mm to (88.3, 87.2), turned to 180 degrees
- moved M300 105.1 mm to (83.3, 76.7), turned to 180 degrees
- moved D300 104.5 mm to (85.8, 84.4)
- moved R302 101.8 mm to (88.4, 89.2)
- moved H102 93.3 mm to (83.8, 63.5)
- moved TP200 85.7 mm to (121.9, 154.4), turned to 90 degrees
- moved C200 83.8 mm to (134.3, 152.9), turned to 270 degrees
- moved D200 83.7 mm to (128.9, 153.0), turned to 90 degrees
- moved TP201 80.1 mm to (121.9, 141.1), turned to 90 degrees
- moved C204 78.3 mm to (136.7, 147.0), turned to 90 degrees
- moved TP202 76.5 mm to (132.7, 140.7), turned to 90 degrees
- moved L200 76.1 mm to (132.1, 148.7), turned to 90 degrees
- moved SW600 75.9 mm to (83.9, 139.3), turned to 90 degrees
- moved H103 74.8 mm to (83.8, 153.0)
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Connections:
- J400 pad 4: /Microcontroller/P3.6 -> GND
- U400 pad 15: (no net) -> GND
- U400 pad 16: (no net) -> +3V3
- U400 pad 19: GND -> (no net)
- U400 pad 20: +3V3 -> (no net)
- U400 pad 25: (no net) -> /Microcontroller/P4.1
- U400 pad 26: (no net) -> /Microcontroller/P4.2
- U400 pad 27: (no net) -> /Microcontroller/P4.3
- U400 pad 28: (no net) -> /Microcontroller/P2.5
- U400 pad 29: (no net) -> /Microcontroller/P2.6_OR_OUT
- U400 pad 30: (no net) -> /Microcontroller/TEST_SBWTCK
- U400 pad 31: (no net) -> /Microcontroller/~RST~_SBWTDI0
- U400 pad 32: /Microcontroller/P4.1 -> /Microcontroller/P2.0_TXD
- U400 pad 33: /Microcontroller/P4.2 -> /Microcontroller/P2.1_RXD
- U400 pad 34: /Microcontroller/P4.3 -> (no net)
- U400 pad 35: /Microcontroller/P2.5 -> /Microcontroller/P3.4
- U400 pad 36: /Microcontroller/P2.6_OR_OUT -> /Microcontroller/P3.5
- U400 pad 37: /Microcontroller/TEST_SBWTCK -> (no net)
- U400 pad 38: /Microcontroller/~RST~_SBWTDI0 -> (no net)
- U400 pad 39: GND -> (no net)
- U400 pad 40: +3V3 -> (no net)
- U400 pad 41: /Microcontroller/P2.0_TXD -> /Microcontroller/P5.0
- U400 pad 42: /Microcontroller/P2.1_RXD -> /Button Generation/Button2
- U400 pad 43: (no net) -> /Microcontroller/P5.2
- U400 pad 44: (no net) -> /Button Generation/Button1
- U400 pad 47: /Microcontroller/P3.4 -> (no net)
- U400 pad 48: /Microcontroller/P3.5 -> GND
- U400 pad 49: /Microcontroller/P3.6 -> +3V3
- U400 pad 50: /Microcontroller/P3.7 -> (no net)
- U400 pad 53: /Microcontroller/P5.0 -> /Microcontroller/P6.0_TxD
- U400 pad 54: (no net) -> /Microcontroller/P6.1_RxD
- U400 pad 55: /Microcontroller/P5.2 -> /Button Generation/Button3
- U400 pad 56: /Button Generation/Button1 -> /Button Generation/Button4
- U400 pad 57: (no net) -> GND
- U400 pad 61: +3V3 -> Net-(C405-Pad1)
- U400 pad 62: (no net) -> Net-(C406-Pad1)
- U400 pad 63: (no net) -> GND
- U400 pad 64: (no net) -> +3V3
- U400 pad 8: /Microcontroller/P6.0_TxD -> (no net)
- U400 pad 9: /Microcontroller/P6.1_RxD -> (no net)
Routing:
- net GND: track 0.00 -> 106.5 mm, vias 0 -> 131
- net +3V3: track 0.00 -> 74.5 mm, vias 0 -> 11
- net /Button Generation/Button1: track 0.00 -> 72.0 mm, vias 0 -> 2
- net /Button Generation/Button4: track 0.00 -> 71.1 mm, vias 0 -> 3
- net /Button Generation/Button2: track 0.00 -> 63.3 mm, vias 0 -> 3
- net /Microcontroller/GeneratorVcc: track 0.00 -> 60.7 mm, vias 0 -> 2
- net /Microcontroller/P6.1_RxD: track 0.00 -> 53.9 mm, vias 0 -> 2
- net /Microcontroller/P6.0_TxD: track 0.00 -> 51.3 mm, vias 0 -> 2
- net /Button Generation/Button3: track 0.00 -> 50.8 mm, vias 0 -> 2
- net /Power Storage/Vin: track 0.00 -> 46.1 mm, vias 0 -> 8
- net /Microcontroller/P4.1: track 0.00 -> 46.0 mm
- net /Microcontroller/P4.2: track 0.00 -> 42.7 mm, vias 0 -> 1
- net /Microcontroller/P4.3: track 0.00 -> 39.5 mm, vias 0 -> 1
- net /Microcontroller/P5.2: track 0.00 -> 38.9 mm, vias 0 -> 1
- net /Microcontroller/~RST~_SBWTDI0: track 0.00 -> 38.8 mm, vias 0 -> 3
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- added copper zone on In2.Cu, net +3V3
- added copper zone on F.Cu, net /Power Storage/Vin
- added copper zone on In2.Cu, net /Power Storage/Vin
- added copper zone on B.Cu, net GND
- added copper zone on F.Cu, net GND
- added copper zone on In1.Cu, net GND
- added copper zone on In2.Cu, net GND
- added copper zone on F.Cu, net Net-(C500-Pad1)
- added copper zone on F.Cu, net Net-(C503-Pad1)
- added copper zone on F.Cu, net Net-(L200-Pad2)
- added copper zone on F.Cu, net Net-(L500-Pad2)
Other:
- board size 6 x 6 mm -> 73 x 99.1 mm
- copper layers 2 -> 4
- board text added: "Senior Design Fall 2021 Rev1 Designer: John Brose"

Commit message: k
Other:
- board text added: "3V3"
- board text added: "BQ255 In"
- board text added: "BUSY"
- board text added: "Boost In"
- board text added: "Boost Out"
- board text added: "CLK"
- board text added: "CS"
- board text added: "DC"
- board text added: "DIN"
- board text added: "GND"
- board text added: "Hand Generator In"
- board text added: "Multiplayer UART"
- board text added: "P3.4"
- board text added: "P3.5"
- board text added: "P6.0_TxD"
- board text added: "P6.1_RxD"
- board text added: "RST"
- board text added: "RXD <<"
- board text added: "SBWTCK"
- board text added: "SBWTDIO"
- board text added: "TXD >>"
- board text added: "VBAT"
- board text added: "VSTOR"
