File: KiCad/batteryless_gaming_device/hand_crank_generator.sch (KiCad schematic (older format))
At the start: 2 parts

Commit message: keep updating schematic
Parts:
- added R?: 180k, symbol Device:R_US
- added R?: 1M, symbol Device:R_US
- added U?: TPS62161DSG, Package_SON:WSON-8-1EP_2x2mm_P0.5mm_EP0.9x1.6mm_ThermalVias, symbol Regulator_Switching:TPS62161DSG
Connections:
- net labels added: generator_voltage
- wire segments 5 -> 12
Other:
- note added: "R1 = R2/(Vin/Vout - 1)\nVin=20,Vout=3.3,R2=1M\n=>R1=180k(lower is safer)"
Changed lines of the file:
@@
 $Descr A 11000 8500
 encoding utf-8
-Sheet 4 4
+Sheet 4 5
 Title ""
 Date ""
@@
 Text Notes 6650 2950 2    98   ~ 0
 Buck-Boost Converter
+$Comp
+L Device:R_US R?
+U 1 1 61917574
+P 4650 2200
+F 0 "R?" H 4718 2246 50  0000 L CNN
+F 1 "180k" H 4718 2155 50  0000 L CNN
+F 2 "" V 4690 2190 50  0001 C CNN
+F 3 "~" H 4650 2200 50  0001 C CNN
+	1    4650 2200
+	1    0    0    -1
+$EndComp
+$Comp
+L Device:R_US R?
+U 1 1 6191BF70
+P 4300 2000
+F 0 "R?" V 4095 2000 50  0000 C CNN
+F 1 "1M" V 4186 2000 50  0000 C CNN
+F 2 "" V 4340 1990 50  0001 C CNN
+F 3 "~" H 4300 2000 50  0001 C CNN
+	1    4300 2000
+	0    1    1    0
+$EndComp
+$Comp
+L power:GND #PWR?
+U 1 1 6191CFA0
+P 4650 2400
+F 0 "#PWR?" H 4650 2150 50  0001 C CNN
+F 1 "GND" H 4655 2227 50  0000 C CNN
+F 2 "" H 4650 2400 50  0001 C CNN
+F 3 "" H 4650 2400 50  0001 C CNN
+	1    4650 2400
+	1    0    0    -1
+$EndComp
+Wire Wire Line
+	4650 2400 4650 2350
+Wire Wire Line
+	4650 2050 4650 2000
+Wire Wire Line
+	4650 2000 4450 2000
+Wire Wire Line
+	3850 3500 3900 3500
+Wire Wire Line
+	3900 3500 3900 2000
+Wire Wire Line
+	3900 2000 4150 2000
+Text Notes 4000 1700 0    50   ~ 0
+R1 = R2/(Vin/Vout - 1)\nVin=20,Vout=3.3,R2=1M\n=>R1=180k(lower is safer)
+Wire Wire Line
+	4650 2000 5000 2000
+Connection ~ 4650 2000
+Text HLabel 5000 2000 2    50   Output ~ 0
+generator_voltage
+$Comp
+L Regulator_Switching:TPS62161DSG U?
+U 1 1 6199D11A
+P 5900 3700
+F 0 "U?" H 5900 4357 50  0000 C CNN
+F 1 "TPS62161DSG" H 5900 4266 50  0000 C CNN
+F 2 "Package_SON:WSON-8-1EP_2x2mm_P0.5mm_EP0.9x1.6mm_ThermalVias" H 6050 3350 50  0001 L CNN
+F 3 "http://www.ti.com/lit/ds/symlink/tps62160.pdf" H 5900 4250 50  0001 C CNN
+F 4 "296-TPS62161DSGTCT-ND" H 5900 4175 50  0000 C CNN "Digikey PN"
+	1    5900 3700
+	1    0    0    -1
+$EndComp
 $EndSCHEMATC

Commit message: k
Parts:
- added R?: 0, Resistor_SMD:R_0805_2012Metric_Pad1.20x1.40mm_HandSolder, symbol Device:R_US
Connections:
- wire segments 12 -> 13
Changed lines of the file:
@@
 	1    0    0    -1
 $EndComp
+$Comp
+L Device:R_US R?
+U 1 1 619B083B
+P 7550 3450
+AR Path="/61926AE2/619B083B" Ref="R?"  Part="1"
+AR Path="/619B083B" Ref="R?"  Part="1"
+AR Path="/619A7303/619B083B" Ref="R?"  Part="1"
+F 0 "R?" V 7700 3400 50  0000 L CNN
+F 1 "0" V 7618 3405 50  0000 L CNN
+F 2 "Resistor_SMD:R_0805_2012Metric_Pad1.20x1.40mm_HandSolder" V 7590 3440 50  0001 C CNN
+F 3 "~" H 7550 3450 50  0001 C CNN
+F 4 "YAG3755CT-ND" V 7450 3450 39  0000 C CNN "Digikey PN"
+	1    7550 3450
+	0    -1   -1   0
+$EndComp
+Wire Wire Line
+	7700 3450 7950 3450
 $EndSCHEMATC

Commit message: k
Parts:
- gave numbers to parts that had none: 6
Changed lines of the file:
@@
 P 2700 3900
 AR Path="/619AD5B9" Ref="M?"  Part="1"
-AR Path="/619A7303/619AD5B9" Ref="M?"  Part="1"
-F 0 "M?" H 2694 4244 50  0000 C CNN
+AR Path="/619A7303/619AD5B9" Ref="M1"  Part="1"
+F 0 "M1" H 2694 4244 50  0000 C CNN
 F 1 "Hand Generator" H 2694 4153 50  0000 C CNN
 F 2 "" H 2700 3710 50  0001 C CNN
@@
 P 3550 3900
 AR Path="/619AD5BF" Ref="D?"  Part="1"
-AR Path="/619A7303/619AD5BF" Ref="D?"  Part="1"
-F 0 "D?" H 3500 4525 50  0000 C CNN
+AR Path="/619A7303/619AD5BF" Ref="D2"  Part="1"
+F 0 "D2" H 3500 4525 50  0000 C CNN
 F 1 "DMA40U1800GU" H 3500 4434 50  0000 C CNN
 F 2 "Diode_THT:Diode_Bridge_IXYS_GUFP" H 3550 3300 50  0001 C CNN
@@
 	3000 4000 3150 4000
 $Comp
-L power:GND #PWR?
+L power:GND #PWR015
 U 1 1 61A827A8
 P 3950 4400
-F 0 "#PWR?" H 3950 4150 50  0001 C CNN
+F 0 "#PWR015" H 3950 4150 50  0001 C CNN
 F 1 "GND" H 3955 4227 50  0000 C CNN
 F 2 "" H 3950 4400 50  0001 C CNN
@@
 Buck-Boost Converter
 $Comp
-L Device:R_US R?
+L Device:R_US R11
 U 1 1 61917574
 P 4650 2200
-F 0 "R?" H 4718 2246 50  0000 L CNN
+F 0 "R11" H 4718 2246 50  0000 L CNN
 F 1 "180k" H 4718 2155 50  0000 L CNN
 F 2 "" V 4690 2190 50  0001 C CNN
@@
 $EndComp
 $Comp
-L Device:R_US R?
+L Device:R_US R10
 U 1 1 6191BF70
 P 4300 2000
-F 0 "R?" V 4095 2000 50  0000 C CNN
+F 0 "R10" V 4095 2000 50  0000 C CNN
 F 1 "1M" V 4186 2000 50  0000 C CNN
 F 2 "" V 4340 1990 50  0001 C CNN
@@
 $EndComp
 $Comp
-L power:GND #PWR?
+L power:GND #PWR016
 U 1 1 6191CFA0
 P 4650 2400
-F 0 "#PWR?" H 4650 2150 50  0001 C CNN
+F 0 "#PWR016" H 4650 2150 50  0001 C CNN
 F 1 "GND" H 4655 2227 50  0000 C CNN
 F 2 "" H 4650 2400 50  0001 C CNN
@@
 generator_voltage
 $Comp
-L Regulator_Switching:TPS62161DSG U?
+L Regulator_Switching:TPS62161DSG U3
 U 1 1 6199D11A
 P 5900 3700
-F 0 "U?" H 5900 4357 50  0000 C CNN
+F 0 "U3" H 5900 4357 50  0000 C CNN
 F 1 "TPS62161DSG" H 5900 4266 50  0000 C CNN
 F 2 "Package_SON:WSON-8-1EP_2x2mm_P0.5mm_EP0.9x1.6mm_ThermalVias" H 6050 3350 50  0001 L CNN
@@
 AR Path="/61926AE2/619B083B" Ref="R?"  Part="1"
 AR Path="/619B083B" Ref="R?"  Part="1"
-AR Path="/619A7303/619B083B" Ref="R?"  Part="1"
-F 0 "R?" V 7700 3400 50  0000 L CNN
+AR Path="/619A7303/619B083B" Ref="R12"  Part="1"
+F 0 "R12" V 7700 3400 50  0000 L CNN
 F 1 "0" V 7618 3405 50  0000 L CNN
 F 2 "Resistor_SMD:R_0805_2012Metric_Pad1.20x1.40mm_HandSolder" V 7590 3440 50  0001 C CNN

Commit message: just kinda out here guys ya know what im saying
Parts:
- removed D2: DMA40U1800GU, Diode_THT:Diode_Bridge_IXYS_GUFP, symbol Diode_Bridge:DMA40U1800GU
- removed R11: 180k, symbol Device:R_US
- removed U3: TPS62161DSG, Package_SON:WSON-8-1EP_2x2mm_P0.5mm_EP0.9x1.6mm_ThermalVias, symbol Regulator_Switching:TPS62161DSG
- added D300: SDA006, Package_TO_SOT_SMD:SOT-363_SC-70-6_Handsoldering, symbol batteryless_gaming_device-rescue:SDA006
- added R302: 1M, Resistor_SMD:R_0603_1608Metric_Pad0.98x0.95mm_HandSolder, symbol Device:R_US
- M300: renamed from M1; footprint (none) -> Connector_PinHeader_2.54mm:PinHeader_1x03_P2.54mm_Vertical
- R300: renamed from R10; footprint (none) -> Resistor_SMD:R_0603_1608Metric_Pad0.98x0.95mm_HandSolder; Digikey PN (none) -> 511-1820-1-ND
- renumbered R12 to R301
Connections:
- wire segments 13 -> 17
Other:
- note removed: "Buck-Boost Converter"
- moved on the sheet: M300, R300, R301
Changed lines of the file:
@@
 L Motor:Motor_Servo M?
 U 1 1 619AD5B9
-P 2700 3900
+P 4250 4900
 AR Path="/619AD5B9" Ref="M?"  Part="1"
-AR Path="/619A7303/619AD5B9" Ref="M1"  Part="1"
-F 0 "M1" H 2694 4244 50  0000 C CNN
-F 1 "Hand Generator" H 2694 4153 50  0000 C CNN
-F 2 "" H 2700 3710 50  0001 C CNN
-F 3 "http://forums.parallax.com/uploads/attachments/46831/74481.png" H 2700 3710 50  0001 C CNN
-	1    2700 3900
+AR Path="/619A7303/619AD5B9" Ref="M300"  Part="1"
+F 0 "M300" H 4244 5244 50  0000 C CNN
+F 1 "Hand Generator" H 4244 5153 50  0000 C CNN
+F 2 "Connector_PinHeader_2.54mm:PinHeader_1x03_P2.54mm_Vertical" H 4250 4710 50  0001 C CNN
+F 3 "http://forums.parallax.com/uploads/attachments/46831/74481.png" H 4250 4710 50  0001 C CNN
+	1    4250 4900
 	-1   0    0    -1
 $EndComp
+Wire Wire Line
+	4550 4800 4700 4800
+Wire Wire Line
+	4550 4900 4700 4900
+Wire Wire Line
+	4550 5000 4700 5000
 $Comp
-L Diode_Bridge:DMA40U1800GU D?
-U 1 1 619AD5BF
-P 3550 3900
-AR Path="/619AD5BF" Ref="D?"  Part="1"
-AR Path="/619A7303/619AD5BF" Ref="D2"  Part="1"
-F 0 "D2" H 3500 4525 50  0000 C CNN
-F 1 "DMA40U1800GU" H 3500 4434 50  0000 C CNN
-F 2 "Diode_THT:Diode_Bridge_IXYS_GUFP" H 3550 3300 50  0001 C CNN
-F 3 "https://ixapps.ixys.com/Datasheet/DMA40U1800GU.pdf" H 3550 4600 50  0001 C CNN
-	1    3550 3900
+L power:GND #PWR0300
+U 1 1 61A827A8
+P 5500 5400
+F 0 "#PWR0300" H 5500 5150 50  0001 C CNN
+F 1 "GND" H 5505 5227 50  0000 C CNN
+F 2 "" H 5500 5400 50  0001 C CNN
+F 3 "" H 5500 5400 50  0001 C CNN
+	1    5500 5400
 	1    0    0    -1
 $EndComp
 Wire Wire Line
-	3000 3800 3150 3800
+	5500 5300 5500 5400
 Wire Wire Line
-	3000 3900 3150 3900
+	5400 5300 5500 5300
+Text HLabel 6350 4500 2    50   Output ~ 0
+Vout
+$Comp
+L Device:R_US R300
+U 1 1 6191BF70
+P 5850 3000
+F 0 "R300" V 5645 3000 50  0000 C CNN
+F 1 "1M" V 5736 3000 50  0000 C CNN
+F 2 "Resistor_SMD:R_0603_1608Metric_Pad0.98x0.95mm_HandSolder" V 5890 2990 50  0001 C CNN
+F 3 "~" H 5850 3000 50  0001 C CNN
+F 4 "511-1820-1-ND" V 5950 3000 39  0000 C CNN "Digikey PN"
+	1    5850 3000
+	0    1    1    0
+$EndComp
 Wire Wire Line
-	3000 4000 3150 4000
+	6200 3000 6000 3000
+Wire Wire Line
+	5400 4500 5450 4500
+Wire Wire Line
+	5450 4500 5450 3000
+Wire Wire Line
+	5450 3000 5700 3000
+Text Notes 5550 2700 0    50   ~ 0
+R1 = R2/(Vin/Vout - 1)\nVin=20,Vout=3.3,R2=1M\n=>R1=180k(lower is safer)
+Wire Wire Line
+	6200 3000 6550 3000
+Connection ~ 6200 3000
+Text HLabel 6550 3000 2    50   Output ~ 0
+generator_voltage
 $Comp
-L power:GND #PWR015
-U 1 1 61A827A8
-P 3950 4400
-F 0 "#PWR015" H 3950 4150 50  0001 C CNN
-F 1 "GND" H 3955 4227 50  0000 C CNN
-F 2 "" H 3950 4400 50  0001 C CNN
-F 3 "" H 3950 4400 50  0001 C CNN
-	1    3950 4400
+L Device:R_US R?
+U 1 1 619B083B
+P 6000 4500
+AR Path="/61926AE2/619B083B" Ref="R?"  Part="1"
+AR Path="/619B083B" Ref="R?"  Part="1"
+AR Path="/619A7303/619B083B" Ref="R301"  Part="1"
+F 0 "R301" V 6150 4450 50  0000 L CNN
+F 1 "0" V 6068 4455 50  0000 L CNN
+F 2 "Resistor_SMD:R_0805_2012Metric_Pad1.20x1.40mm_HandSolder" V 6040 4490 50  0001 C CNN
+F 3 "~" H 6000 4500 50  0001 C CNN
+F 4 "YAG3755CT-ND" V 5900 4500 39  0000 C CNN "Digikey PN"
+	1    6000 4500
+	0    -1   -1   0
+$EndComp
+Wire Wire Line
+	6150 4500 6350 4500
+Connection ~ 5450 4500
+Wire Wire Line
+	5450 4500 5550 4500
+$Comp
+L Device:R_US R302
+U 1 1 6196F794
+P 6200 3300
+F 0 "R302" H 6100 3200 50  0000 C CNN
+F 1 "1M" H 6086 3300 50  0000 C CNN
+F 2 "Resistor_SMD:R_0603_1608Metric_Pad0.98x0.95mm_HandSolder" V 6240 3290 50  0001 C CNN
+F 3 "~" H 6200 3300 50  0001 C CNN
+F 4 "511-1820-1-ND" H 5850 3400 39  0000 C CNN "Digikey PN"
+	1    6200 3300
+	-1   0    0    1
+$EndComp
+Wire Wire Line
+	6200 3000 6200 3150
+$Comp
+L power:GND #PWR0301
+U 1 1 619709AA
+P 6200 3500
+F 0 "#PWR0301" H 6200 3250 50  0001 C CNN
+F 1 "GND" H 6205 3327 50  0000 C CNN
+F 2 "" H 6200 3500 50  0001 C CNN
+F 3 "" H 6200 3500 50  0001 C CNN
+	1    6200 3500
 	1    0    0    -1
 $EndComp
 Wire Wire Line
-	3950 4300 3950 4400
-Wire Wire Line
-	3850 4300 3950 4300
-Text HLabel 7950 3450 2    50   Output ~ 0
-Vout
-Wire Notes Line
-	4900 2750 4900 4500
-Wire Notes Line
-	4900 4500 6950 4500
-Wire Notes Line
-	6950 4500 6950 2750
-Wire Notes Line
-	4900 2750 6950 2750
-Text Notes 6650 2950 2    98   ~ 0
-Buck-Boost Converter
+	6200 3450 6200 3500
 $Comp
-L Device:R_US R11
-U 1 1 61917574
-P 4650 2200
-F 0 "R11" H 4718 2246 50  0000 L CNN
-F 1 "180k" H 4718 2155 50  0000 L CNN
-F 2 "" V 4690 2190 50  0001 C CNN
-F 3 "~" H 4650 2200 50  0001 C CNN
-	1    4650 2200
-	1    0    0    -1
-$EndComp
-$Comp
-L Device:R_US R10
-U 1 1 6191BF70
-P 4300 2000
-F 0 "R10" V 4095 2000 50  0000 C CNN
-F 1 "1M" V 4186 2000 50  0000 C CNN
-F 2 "" V 4340 1990 50  0001 C CNN
-F 3 "~" H 4300 2000 50  0001 C CNN
-	1    4300 2000
-	0    1    1    0
-$EndComp
-$Comp
-L power:GND #PWR016
-U 1 1 6191CFA0
-P 4650 2400
-F 0 "#PWR016" H 4650 2150 50  0001 C CNN
-F 1 "GND" H 4655 2227 50  0000 C CNN
-F 2 "" H 4650 2400 50  0001 C CNN
-F 3 "" H 4650 2400 50  0001 C CNN
-	1    4650 2400
+L batteryless_gaming_device-rescue:SDA006 D300
+U 1 1 619799AF
+P 5100 4400
+F 0 "D300" H 5050 4599 50  0000 C CNN
+F 1 "SDA006" H 5050 4500 50  0000 C CNN
+F 2 "Package_TO_SOT_SMD:SOT-363_SC-70-6_Handsoldering" H 5100 4400 50  0001 C CNN
+F 3 "" H 5100 4400 50  0001 C CNN
+F 4 "SDA006-7DICT-ND" H 5050 4425 39  0000 C CNN "Digikey PN"
+	1    5100 4400
 	1    0    0    -1
 $EndComp
 Wire Wire Line
-	4650 2400 4650 2350
+	5400 4600 5550 4600
 Wire Wire Line
-	4650 2050 4650 2000
+	5550 4600 5550 4500
+Connection ~ 5550 4500
 Wire Wire Line
-	4650 2000 4450 2000
-Wire Wire Line
-	3850 3500 3900 3500
-Wire Wire Line
-	3900 3500 3900 2000
-Wire Wire Line
-	3900 2000 4150 2000
-Text Notes 4000 1700 0    50   ~ 0
-R1 = R2/(Vin/Vout - 1)\nVin=20,Vout=3.3,R2=1M\n=>R1=180k(lower is safer)
-Wire Wire Line
-	4650 2000 5000 2000
-Connection ~ 4650 2000
-Text HLabel 5000 2000 2    50   Output ~ 0
-generator_voltage
-$Comp
-L Regulator_Switching:TPS62161DSG U3
-U 1 1 6199D11A
-P 5900 3700
-F 0 "U3" H 5900 4357 50  0000 C CNN
-F 1 "TPS62161DSG" H 5900 4266 50  0000 C CNN
-F 2 "Package_SON:WSON-8-1EP_2x2mm_P0.5mm_EP0.9x1.6mm_ThermalVias" H 6050 3350 50  0001 L CNN
-F 3 "http://www.ti.com/lit/ds/symlink/tps62160.pdf" H 5900 4250 50  0001 C CNN
-F 4 "296-TPS62161DSGTCT-ND" H 5900 4175 50  0000 C CNN "Digikey PN"
-	1    5900 3700
-	1    0    0    -1
-$EndComp
-$Comp
-L Device:R_US R?
-U 1 1 619B083B
-P 7550 3450
-AR Path="/61926AE2/619B083B" Ref="R?"  Part="1"
-AR Path="/619B083B" Ref="R?"  Part="1"
-AR Path="/619A7303/619B083B" Ref="R12"  Part="1"
-F 0 "R12" V 7700 3400 50  0000 L CNN
-F 1 "0" V 7618 3405 50  0000 L CNN
-F 2 "Resistor_SMD:R_0805_2012Metric_Pad1.20x1.40mm_HandSolder" V 7590 3440 50  0001 C CNN
-F 3 "~" H 7550 3450 50  0001 C CNN
-F 4 "YAG3755CT-ND" V 7450 3450 39  0000 C CNN "Digikey PN"
-	1    7550 3450
-	0    -1   -1   0
-$EndComp
-Wire Wire Line
-	7700 3450 7950 3450
+	5550 4500 5850 4500
 $EndSCHEMATC

Commit message: oh ya
Parts:
- M300: footprint Connector_PinHeader_2.54mm:PinHeader_1x03_P2.54mm_Vertical -> Connector_PinHeader_2.00mm:PinHeader_1x03_P2.00mm_Vertical; Digikey PN (none) -> A100097-ND
Changed lines of the file:
@@
 F 0 "M300" H 4244 5244 50  0000 C CNN
 F 1 "Hand Generator" H 4244 5153 50  0000 C CNN
-F 2 "Connector_PinHeader_2.54mm:PinHeader_1x03_P2.54mm_Vertical" H 4250 4710 50  0001 C CNN
+F 2 "Connector_PinHeader_2.00mm:PinHeader_1x03_P2.00mm_Vertical" H 4250 4710 50  0001 C CNN
 F 3 "http://forums.parallax.com/uploads/attachments/46831/74481.png" H 4250 4710 50  0001 C CNN
+F 4 "A100097-ND" H 4250 5100 39  0000 C CNN "Digikey PN"
 	1    4250 4900
 	-1   0    0    -1

Commit message: updated
Parts:
- removed R300, R302: 1M, Resistor_SMD:R_0603_1608Metric_Pad0.98x0.95mm_HandSolder, symbol Device:R_US
Other:
- note removed: "R1 = R2/(Vin/Vout - 1)\nVin=20,Vout=3.3,R2=1M\n=>R1=180k(lower is safer)"
Changed lines of the file:
@@
 Vout
-$Comp
-L Device:R_US R300
-U 1 1 6191BF70
-P 5850 3000
-F 0 "R300" V 5645 3000 50  0000 C CNN
-F 1 "1M" V 5736 3000 50  0000 C CNN
-F 2 "Resistor_SMD:R_0603_1608Metric_Pad0.98x0.95mm_HandSolder" V 5890 2990 50  0001 C CNN
-F 3 "~" H 5850 3000 50  0001 C CNN
-F 4 "511-1820-1-ND" V 5950 3000 39  0000 C CNN "Digikey PN"
-	1    5850 3000
-	0    1    1    0
-$EndComp
-Wire Wire Line
-	6200 3000 6000 3000
-Wire Wire Line
-	5400 4500 5450 4500
-Wire Wire Line
-	5450 4500 5450 3000
-Wire Wire Line
-	5450 3000 5700 3000
-Text Notes 5550 2700 0    50   ~ 0
-R1 = R2/(Vin/Vout - 1)\nVin=20,Vout=3.3,R2=1M\n=>R1=180k(lower is safer)
-Wire Wire Line
-	6200 3000 6550 3000
-Connection ~ 6200 3000
-Text HLabel 6550 3000 2    50   Output ~ 0
-generator_voltage
 $Comp
 L Device:R_US R?
@@
 Wire Wire Line
 	6150 4500 6350 4500
-Connection ~ 5450 4500
-Wire Wire Line
-	5450 4500 5550 4500
-$Comp
-L Device:R_US R302
-U 1 1 6196F794
-P 6200 3300
-F 0 "R302" H 6100 3200 50  0000 C CNN
-F 1 "1M" H 6086 3300 50  0000 C CNN
-F 2 "Resistor_SMD:R_0603_1608Metric_Pad0.98x0.95mm_HandSolder" V 6240 3290 50  0001 C CNN
-F 3 "~" H 6200 3300 50  0001 C CNN
-F 4 "511-1820-1-ND" H 5850 3400 39  0000 C CNN "Digikey PN"
-	1    6200 3300
-	-1   0    0    1
-$EndComp
-Wire Wire Line
-	6200 3000 6200 3150
-$Comp
-L power:GND #PWR0301
-U 1 1 619709AA
-P 6200 3500
-F 0 "#PWR0301" H 6200 3250 50  0001 C CNN
-F 1 "GND" H 6205 3327 50  0000 C CNN
-F 2 "" H 6200 3500 50  0001 C CNN
-F 3 "" H 6200 3500 50  0001 C CNN
-	1    6200 3500
-	1    0    0    -1
-$EndComp
-Wire Wire Line
-	6200 3450 6200 3500
 $Comp
 L batteryless_gaming_device-rescue:SDA006 D300
@@
 Wire Wire Line
 	5550 4500 5850 4500
+Wire Wire Line
+	5400 4500 5550 4500
 $EndSCHEMATC
