File: KiCad/batteryless_gaming_device/micro_msp430fr5994.sch (KiCad schematic (older format))
At the start: 13 parts

Commit message: updated schematic
Connections:
- net labels added: Button1, Button2, Button3, Button4, GeneratorVcc, VBAT_OK
Other:
- note added: "Energy\nHarvesting\nGPIO/Analog In"
- note added: "possibly add mosfet to switch 3.3V logic"
Changed lines of the file:
@@
 $Descr A 11000 8500
 encoding utf-8
-Sheet 5 5
+Sheet 4 6
 Title ""
 Date ""
@@
 Text Notes 6950 5300 0    79   ~ 0
 Programming Interface
+Text HLabel 1250 1500 0    50   Input ~ 0
+Button1
+Text HLabel 1250 1600 0    50   Input ~ 0
+Button2
+Text HLabel 1250 1700 0    50   Input ~ 0
+Button3
+Text HLabel 1250 1800 0    50   Input ~ 0
+Button4
+Wire Notes Line
+	1750 2050 1750 1000
+Wire Notes Line
+	1750 1000 750  1000
+Wire Notes Line
+	750  1000 750  2050
+Text Notes 800  1400 0    79   ~ 0
+Energy\nHarvesting\nGPIO/Analog In
+Text HLabel 1450 1950 0    50   Input ~ 0
+GeneratorVcc
+Wire Notes Line
+	1750 3900 1750 2850
+Wire Notes Line
+	1750 2850 750  2850
+Wire Notes Line
+	750  2850 750  3900
+Text Notes 800  3250 0    79   ~ 0
+Energy\nHarvesting\nGPIO/Analog In
+Wire Notes Line
+	750  2050 1750 2050
+Wire Notes Line
+	750  3900 1750 3900
+Text HLabel 1250 3600 0    50   Input ~ 0
+VBAT_OK
+Text Notes 850  3750 0    50   ~ 0
+possibly add mosfet to switch 3.3V logic
 $EndSCHEMATC

Commit message: k
Parts:
- removed C?: 10uF, symbol Device:CP1
- added C?: 10uF, symbol Device:C
- C?: Digikey PN (none) -> 1276-CL10B102KB8WPJCCT-ND
- C? (x4): Digikey PN (none) -> 296-21684-1-ND
- SW?: value PTS636 SMG25J SMTR LFS -> FSMSM; footprint (none) -> Button_Switch_SMD:SW_SPST_FSMSM; Digikey PN CKN12327-1-ND -> 450-1140-ND
- U?: Digikey PN (none) -> 296-45560-1-ND
Connections:
- net labels added: V_program
- wire segments 81 -> 80
Other:
- note added: "or just connect to ADC"
Changed lines of the file:
@@
 AR Path="/6192B25C" Ref="U?"  Part="1"
 AR Path="/61926AE2/6192B25C" Ref="U?"  Part="1"
-F 0 "U?" H 4325 1567 50  0000 C CNN
-F 1 "MSP430FR5994" H 4325 1476 50  0000 C CNN
+F 0 "U?" H 4350 1650 50  0000 C CNN
+F 1 "MSP430FR5994" H 4350 1550 50  0000 C CNN
 F 2 "" V 3400 1200 354 0001 C CNN
 F 3 "" V 3400 1200 354 0001 C CNN
+F 4 "296-45560-1-ND" H 4350 1450 39  0000 C CNN "Digikey PN"
 	1    4300 1400
 	1    0    0    -1
@@
 F 2 "" H 5888 3600 50  0001 C CNN
 F 3 "~" H 5850 3750 50  0001 C CNN
+F 4 "296-21684-1-ND" H 6300 4050 39  0000 C CNN "Digikey PN"
 	1    5850 3750
 	1    0    0    -1
@@
 Wire Wire Line
 	7400 6100 7400 5950
-$Comp
-L power:+3.3V #PWR?
-U 1 1 6194A2D7
-P 7300 5800
-F 0 "#PWR?" H 7300 5650 50  0001 C CNN
-F 1 "+3.3V" H 7315 5973 50  0000 C CNN
-F 2 "" H 7300 5800 50  0001 C CNN
-F 3 "" H 7300 5800 50  0001 C CNN
-	1    7300 5800
-	1    0    0    -1
-$EndComp
-Wire Wire Line
-	7300 5800 7300 5850
-Wire Wire Line
-	7300 5850 8000 5850
 NoConn ~ 5400 5800
 NoConn ~ 5400 5900
@@
 P 8900 1400
 F 0 "SW?" H 8900 1743 50  0000 C CNN
-F 1 "PTS636 SMG25J SMTR LFS" H 8900 1660 39  0000 C CNN
-F 2 "" H 8900 1600 50  0001 C CNN
+F 1 "FSMSM" H 8900 1660 39  0000 C CNN
+F 2 "Button_Switch_SMD:SW_SPST_FSMSM" H 8900 1600 50  0001 C CNN
 F 3 "~" H 8900 1600 50  0001 C CNN
-F 4 "CKN12327-1-ND" H 8900 1585 39  0000 C CNN "Digikey PN"
+F 4 "450-1140-ND" H 8900 1585 39  0000 C CNN "Digikey PN"
 	1    8900 1400
 	1    0    0    -1
@@
 $EndComp
 $Comp
-L Device:C C?
-U 1 1 6191DC18
-P 9500 1600
-F 0 "C?" H 9615 1646 50  0000 L CNN
-F 1 "1nF" H 9615 1555 50  0000 L CNN
-F 2 "" H 9538 1450 50  0001 C CNN
-F 3 "~" H 9500 1600 50  0001 C CNN
-	1    9500 1600
-	1    0    0    -1
-$EndComp
-$Comp
 L power:GND #PWR?
 U 1 1 6191E35F
@@
 	7900 3200 7900 3500
 $Comp
-L Device:CP1 C?
-U 1 1 619320E0
-P 7900 3750
-F 0 "C?" H 8015 3796 50  0000 L CNN
-F 1 "10uF" H 8015 3705 50  0000 L CNN
-F 2 "" H 7900 3750 50  0001 C CNN
-F 3 "~" H 7900 3750 50  0001 C CNN
-	1    7900 3750
-	1    0    0    -1
-$EndComp
-$Comp
 L Device:C C?
 U 1 1 619313AD
@@
 F 2 "" H 7388 3600 50  0001 C CNN
 F 3 "~" H 7350 3750 50  0001 C CNN
+F 4 "296-21684-1-ND" H 6300 4200 39  0000 C CNN "Digikey PN"
 	1    7350 3750
 	1    0    0    -1
@@
 F 2 "" H 6888 3600 50  0001 C CNN
 F 3 "~" H 6850 3750 50  0001 C CNN
+F 4 "296-21684-1-ND" H 6300 4150 39  0000 C CNN "Digikey PN"
 	1    6850 3750
 	1    0    0    -1
@@
 F 2 "" H 6438 3600 50  0001 C CNN
 F 3 "~" H 6400 3750 50  0001 C CNN
+F 4 "296-21684-1-ND" H 6300 4100 39  0000 C CNN "Digikey PN"
 	1    6400 3750
 	1    0    0    -1
@@
 Text Notes 850  3750 0    50   ~ 0
 possibly add mosfet to switch 3.3V logic
+Text HLabel 7350 5850 0    50   Output ~ 0
+V_program
+Wire Wire Line
+	7350 5850 8000 5850
+Text Notes 850  3850 0    50   ~ 0
+or just connect to ADC
+$Comp
+L Device:C C?
+U 1 1 619E966F
+P 7900 3750
+F 0 "C?" H 8015 3796 50  0000 L CNN
+F 1 "10uF" H 8015 3705 50  0000 L CNN
+F 2 "" H 7938 3600 50  0001 C CNN
+F 3 "~" H 7900 3750 50  0001 C CNN
+F 4 "399-11939-1-ND" H 7950 3450 39  0000 C CNN "Digikey PN"
+	1    7900 3750
+	1    0    0    -1
+$EndComp
+$Comp
+L Device:C C?
+U 1 1 6191DC18
+P 9500 1600
+F 0 "C?" H 9615 1646 50  0000 L CNN
+F 1 "1nF" H 9615 1555 50  0000 L CNN
+F 2 "" H 9538 1450 50  0001 C CNN
+F 3 "~" H 9500 1600 50  0001 C CNN
+F 4 "1276-CL10B102KB8WPJCCT-ND" H 10000 1450 39  0000 C CNN "Digikey PN"
+	1    9500 1600
+	1    0    0    -1
+$EndComp
 $EndSCHEMATC

Commit message: k
Parts:
- C11, C12, C13, C14, C18: renamed from C?; footprint (none) -> Capacitor_SMD:C_0603_1608Metric_Pad1.08x0.95mm_HandSolder
- C15: renamed from C?; footprint (none) -> Capacitor_SMD:C_0805_2012Metric_Pad1.18x1.45mm_HandSolder
- C16, C17: renamed from C?; footprint (none) -> Capacitor_SMD:C_0603_1608Metric_Pad1.08x0.95mm_HandSolder; Digikey PN (none) -> 311-4030-1-ND
- gave numbers to parts that had none: 5
Connections:
- net labels added: P2.5, P2.5_CS, P4.1, P4.1_Busy, P4.2, P4.2_RST, P4.3, P4.3_DC, P5.0, P5.0_DIN, P5.2, P5.2_CLK
- wire segments 80 -> 92
Other:
- note removed: "Maybe need to add protection for 3.3V in, in case \nboost regulator is also outputting 3.3V"
Changed lines of the file:
@@
 P 4300 1400
 AR Path="/6192B25C" Ref="U?"  Part="1"
-AR Path="/61926AE2/6192B25C" Ref="U?"  Part="1"
-F 0 "U?" H 4350 1650 50  0000 C CNN
+AR Path="/61926AE2/6192B25C" Ref="U4"  Part="1"
+F 0 "U4" H 4350 1650 50  0000 C CNN
 F 1 "MSP430FR5994" H 4350 1550 50  0000 C CNN
 F 2 "" V 3400 1200 354 0001 C CNN
@@
 $EndComp
 $Comp
-L Device:C C?
+L Device:C C11
 U 1 1 6192E176
 P 5850 3750
-F 0 "C?" H 5965 3796 50  0000 L CNN
+F 0 "C11" H 5965 3796 50  0000 L CNN
 F 1 "0.1uF" H 5965 3705 50  0000 L CNN
-F 2 "" H 5888 3600 50  0001 C CNN
+F 2 "Capacitor_SMD:C_0603_1608Metric_Pad1.08x0.95mm_HandSolder" H 5888 3600 50  0001 C CNN
 F 3 "~" H 5850 3750 50  0001 C CNN
 F 4 "296-21684-1-ND" H 6300 4050 39  0000 C CNN "Digikey PN"
@@
 Connection ~ 5500 4200
 $Comp
-L power:GND #PWR?
+L power:GND #PWR017
 U 1 1 61935151
 P 5750 4300
-F 0 "#PWR?" H 5750 4050 50  0001 C CNN
+F 0 "#PWR017" H 5750 4050 50  0001 C CNN
 F 1 "GND" H 5755 4127 50  0000 C CNN
 F 2 "" H 5750 4300 50  0001 C CNN
@@
 Connection ~ 5500 3200
 $Comp
-L power:+3.3V #PWR?
+L power:+3.3V #PWR020
 U 1 1 6193DF42
 P 7950 3100
-F 0 "#PWR?" H 7950 2950 50  0001 C CNN
+F 0 "#PWR020" H 7950 2950 50  0001 C CNN
 F 1 "+3.3V" H 7965 3273 50  0000 C CNN
 F 2 "" H 7950 3100 50  0001 C CNN
@@
 Wire Wire Line
 	7950 3200 7950 3100
-Text Notes 9150 6550 2    50   ~ 0
-Maybe need to add protection for 3.3V in, in case \nboost regulator is also outputting 3.3V
 Text Label 8000 5450 2    50   ~ 0
 TEST_SBWTCK
@@
 TGT_GND
 $Comp
-L Connector_Generic:Conn_01x06 J?
+L Connector_Generic:Conn_01x06 J2
 U 1 1 61940A05
 P 8200 5650
-F 0 "J?" H 8280 5642 50  0000 L CNN
+F 0 "J2" H 8280 5642 50  0000 L CNN
 F 1 "Program Header" H 8280 5551 50  0000 L CNN
 F 2 "" H 8200 5650 50  0001 C CNN
@@
 $EndComp
 $Comp
-L power:GND #PWR?
+L power:GND #PWR019
 U 1 1 6194303F
 P 7400 6100
-F 0 "#PWR?" H 7400 5850 50  0001 C CNN
+F 0 "#PWR019" H 7400 5850 50  0001 C CNN
 F 1 "GND" H 7405 5927 50  0000 C CNN
 F 2 "" H 7400 6100 50  0001 C CNN
@@
 P2.1_RXD
 $Comp
-L Switch:SW_Push SW?
+L Switch:SW_Push SW1
 U 1 1 6191AF25
 P 8900 1400
-F 0 "SW?" H 8900 1743 50  0000 C CNN
+F 0 "SW1" H 8900 1743 50  0000 C CNN
 F 1 "FSMSM" H 8900 1660 39  0000 C CNN
 F 2 "Button_Switch_SMD:SW_SPST_FSMSM" H 8900 1600 50  0001 C CNN
@@
 $EndComp
 $Comp
-L Device:R_US R?
+L Device:R_US R13
 U 1 1 6191CB81
 P 9500 1200
-F 0 "R?" H 9568 1246 50  0000 L CNN
+F 0 "R13" H 9568 1246 50  0000 L CNN
 F 1 "47k" H 9568 1155 50  0000 L CNN
 F 2 "" V 9540 1190 50  0001 C CNN
@@
 $EndComp
 $Comp
-L power:GND #PWR?
+L power:GND #PWR023
 U 1 1 6191E35F
 P 9500 1800
-F 0 "#PWR?" H 9500 1550 50  0001 C CNN
+F 0 "#PWR023" H 9500 1550 50  0001 C CNN
 F 1 "GND" H 9505 1627 50  0000 C CNN
 F 2 "" H 9500 1800 50  0001 C CNN
@@
 	9500 1750 9500 1800
 $Comp
-L power:GND #PWR?
+L power:GND #PWR021
 U 1 1 619249D7
 P 8650 1500
-F 0 "#PWR?" H 8650 1250 50  0001 C CNN
+F 0 "#PWR021" H 8650 1250 50  0001 C CNN
 F 1 "GND" H 8655 1327 50  0000 C CNN
 F 2 "" H 8650 1500 50  0001 C CNN
@@
 	8650 1400 8700 1400
 $Comp
-L power:+3.3V #PWR?
+L power:+3.3V #PWR022
 U 1 1 61926666
 P 9500 1000
-F 0 "#PWR?" H 9500 850 50  0001 C CNN
+F 0 "#PWR022" H 9500 850 50  0001 C CNN
 F 1 "+3.3V" H 9515 1173 50  0000 C CNN
 F 2 "" H 9500 1000 50  0001 C CNN
@@
 	6400 3900 6400 4000
 $Comp
-L power:GND #PWR?
+L power:GND #PWR018
 U 1 1 6193B7AC
 P 7100 4100
-F 0 "#PWR?" H 7100 3850 50  0001 C CNN
+F 0 "#PWR018" H 7100 3850 50  0001 C CNN
 F 1 "GND" H 7105 3927 50  0000 C CNN
 F 2 "" H 7100 4100 50  0001 C CNN
@@
 	7900 3200 7900 3500
 $Comp
-L Device:C C?
+L Device:C C14
 U 1 1 619313AD
 P 7350 3750
-F 0 "C?" H 7465 3796 50  0000 L CNN
+F 0 "C14" H 7465 3796 50  0000 L CNN
 F 1 "0.1uF" H 7465 3705 50  0000 L CNN
-F 2 "" H 7388 3600 50  0001 C CNN
+F 2 "Capacitor_SMD:C_0603_1608Metric_Pad1.08x0.95mm_HandSolder" H 7388 3600 50  0001 C CNN
 F 3 "~" H 7350 3750 50  0001 C CNN
 F 4 "296-21684-1-ND" H 6300 4200 39  0000 C CNN "Digikey PN"
@@
 $EndComp
 $Comp
-L Device:C C?
+L Device:C C13
 U 1 1 61930F42
 P 6850 3750
-F 0 "C?" H 6965 3796 50  0000 L CNN
+F 0 "C13" H 6965 3796 50  0000 L CNN
 F 1 "0.1uF" H 6965 3705 50  0000 L CNN
-F 2 "" H 6888 3600 50  0001 C CNN
+F 2 "Capacitor_SMD:C_0603_1608Metric_Pad1.08x0.95mm_HandSolder" H 6888 3600 50  0001 C CNN
 F 3 "~" H 6850 3750 50  0001 C CNN
 F 4 "296-21684-1-ND" H 6300 4150 39  0000 C CNN "Digikey PN"
@@
 $EndComp
 $Comp
-L Device:C C?
+L Device:C C12
 U 1 1 61930AF3
 P 6400 3750
-F 0 "C?" H 6515 3796 50  0000 L CNN
+F 0 "C12" H 6515 3796 50  0000 L CNN
 F 1 "0.1uF" H 6515 3705 50  0000 L CNN
-F 2 "" H 6438 3600 50  0001 C CNN
+F 2 "Capacitor_SMD:C_0603_1608Metric_Pad1.08x0.95mm_HandSolder" H 6438 3600 50  0001 C CNN
 F 3 "~" H 6400 3750 50  0001 C CNN
 F 4 "296-21684-1-ND" H 6300 4100 39  0000 C CNN "Digikey PN"
@@
 AVCC
 $Comp
-L Device:Crystal Y?
+L Device:Crystal Y1
 U 1 1 6195C01B
 P 8850 4650
-F 0 "Y?" V 8917 4494 50  0000 C CNN
+F 0 "Y1" V 8917 4494 50  0000 C CNN
 F 1 "ECS-.327-12.5-34R-C-TR" V 8851 4116 39  0000 C CNN
 F 2 "" H 8850 4650 50  0001 C CNN
@@
 $EndComp
 $Comp
-L Device:C C?
+L Device:C C17
 U 1 1 6195EA6D
 P 9200 4850
-F 0 "C?" V 9150 4900 50  0000 L CNN
+F 0 "C17" V 9150 4900 50  0000 L CNN
 F 1 "22pF" V 9150 4600 50  0000 L CNN
-F 2 "" H 9238 4700 50  0001 C CNN
+F 2 "Capacitor_SMD:C_0603_1608Metric_Pad1.08x0.95mm_HandSolder" H 9238 4700 50  0001 C CNN
 F 3 "~" H 9200 4850 50  0001 C CNN
+F 4 "311-4030-1-ND" V 9050 4850 39  0000 C CNN "Digikey PN"
 	1    9200 4850
 	0    -1   -1   0
 $EndComp
 $Comp
-L Device:C C?
+L Device:C C16
 U 1 1 6195E432
 P 9200 4450
-F 0 "C?" V 9250 4500 50  0000 L CNN
+F 0 "C16" V 9250 4500 50  0000 L CNN
 F 1 "22pF" V 9250 4200 50  0000 L CNN
-F 2 "" H 9238 4300 50  0001 C CNN
+F 2 "Capacitor_SMD:C_0603_1608Metric_Pad1.08x0.95mm_HandSolder" H 9238 4300 50  0001 C CNN
 F 3 "~" H 9200 4450 50  0001 C CNN
+F 4 "311-4030-1-ND" V 9350 4450 39  0000 C CNN "Digikey PN"
 	1    9200 4450
 	0    -1   -1   0
@@
 	8850 4450 8850 4500
 $Comp
-L power:GND #PWR?
+L power:GND #PWR024
 U 1 1 6197ADE6
 P 10000 4700
-F 0 "#PWR?" H 10000 4450 50  0001 C CNN
+F 0 "#PWR024" H 10000 4450 50  0001 C CNN
 F 1 "GND" H 10005 4527 50  0000 C CNN
 F 2 "" H 10000 4700 50  0001 C CNN
@@
 or just connect to ADC
 $Comp
-L Device:C C?
+L Device:C C15
 U 1 1 619E966F
 P 7900 3750
-F 0 "C?" H 8015 3796 50  0000 L CNN
+F 0 "C15" H 8015 3796 50  0000 L CNN
 F 1 "10uF" H 8015 3705 50  0000 L CNN
-F 2 "" H 7938 3600 50  0001 C CNN
+F 2 "Capacitor_SMD:C_0805_2012Metric_Pad1.18x1.45mm_HandSolder" H 7938 3600 50  0001 C CNN
 F 3 "~" H 7900 3750 50  0001 C CNN
 F 4 "399-11939-1-ND" H 7950 3450 39  0000 C CNN "Digikey PN"
@@
 $EndComp
 $Comp
-L Device:C C?
+L Device:C C18
 U 1 1 6191DC18
 P 9500 1600
-F 0 "C?" H 9615 1646 50  0000 L CNN
+F 0 "C18" H 9615 1646 50  0000 L CNN
 F 1 "1nF" H 9615 1555 50  0000 L CNN
-F 2 "" H 9538 1450 50  0001 C CNN
+F 2 "Capacitor_SMD:C_0603_1608Metric_Pad1.08x0.95mm_HandSolder" H 9538 1450 50  0001 C CNN
 F 3 "~" H 9500 1600 50  0001 C CNN
 F 4 "1276-CL10B102KB8WPJCCT-ND" H 10000 1450 39  0000 C CNN "Digikey PN"
@@
 	1    0    0    -1
 $EndComp
+Text HLabel 9300 2600 2    50   Output ~ 0
+P4.1
+Text HLabel 9300 2700 2    50   Output ~ 0
+P4.2
+Text HLabel 9300 2800 2    50   Output ~ 0
+P4.3
+Text HLabel 9300 2900 2    50   Output ~ 0
+P2.5
+Text HLabel 9300 3000 2    50   Output ~ 0
+P5.2
+Text HLabel 9300 3100 2    50   Output ~ 0
+P5.0
+Text Label 3000 4300 2    50   ~ 0
+P4.1_Busy
+Text Label 2950 4400 2    50   ~ 0
+P4.2_RST
+Text Label 2925 4500 2    50   ~ 0
+P4.3_DC
+Wire Wire Line
+	3250 2900 2450 2900
+Text Label 2900 2900 2    50   ~ 0
+P2.5_CS
+Wire Wire Line
+	2450 4300 3250 4300
+Wire Wire Line
+	2450 4400 3250 4400
+Wire Wire Line
+	2450 4500 3250 4500
+Wire Wire Line
+	3250 5100 2450 5100
+Wire Wire Line
+	3250 5300 2450 5300
+Text Label 3000 5300 2    50   ~ 0
+P5.2_CLK
+Text Label 3000 5100 2    50   ~ 0
+P5.0_DIN
+Wire Wire Line
+	8750 2600 9300 2600
+Wire Wire Line
+	8750 2700 9300 2700
+Wire Wire Line
+	8750 2800 9300 2800
+Wire Wire Line
+	8750 2900 9300 2900
+Wire Wire Line
+	8750 3000 9300 3000
+Wire Wire Line
+	8750 3100 9300 3100
+Text Label 9065 2900 2    50   ~ 0
+P2.5_CS
+Text Label 9140 2600 2    50   ~ 0
+P4.1_Busy
+Text Label 9100 2700 2    50   ~ 0
+P4.2_RST
+Text Label 9065 2800 2    50   ~ 0
+P4.3_DC
+Text Label 9105 3000 2    50   ~ 0
+P5.2_CLK
+Text Label 9090 3100 2    50   ~ 0
+P5.0_DIN
 $EndSCHEMATC

Commit message: k
Parts:
- renumbered C11 to C10, C12 to C11, C13 to C12, C14 to C13, C15 to C14, C16 to C15, C17 to C16, C18 to C17
Connections:
- net labels added: P5.3_Button1, P5.5_Button2, P5.6_Button3, P5.7_Button4
- wire segments 92 -> 106
Other:
- note added: "E-ink Display"
Changed lines of the file:
@@
 $EndComp
 $Comp
-L Device:C C11
+L Device:C C10
 U 1 1 6192E176
 P 5850 3750
-F 0 "C11" H 5965 3796 50  0000 L CNN
+F 0 "C10" H 5965 3796 50  0000 L CNN
 F 1 "0.1uF" H 5965 3705 50  0000 L CNN
 F 2 "Capacitor_SMD:C_0603_1608Metric_Pad1.08x0.95mm_HandSolder" H 5888 3600 50  0001 C CNN
@@
 	7900 3200 7900 3500
 $Comp
-L Device:C C14
+L Device:C C13
 U 1 1 619313AD
 P 7350 3750
-F 0 "C14" H 7465 3796 50  0000 L CNN
+F 0 "C13" H 7465 3796 50  0000 L CNN
 F 1 "0.1uF" H 7465 3705 50  0000 L CNN
 F 2 "Capacitor_SMD:C_0603_1608Metric_Pad1.08x0.95mm_HandSolder" H 7388 3600 50  0001 C CNN
@@
 $EndComp
 $Comp
-L Device:C C13
+L Device:C C12
 U 1 1 61930F42
 P 6850 3750
-F 0 "C13" H 6965 3796 50  0000 L CNN
+F 0 "C12" H 6965 3796 50  0000 L CNN
 F 1 "0.1uF" H 6965 3705 50  0000 L CNN
 F 2 "Capacitor_SMD:C_0603_1608Metric_Pad1.08x0.95mm_HandSolder" H 6888 3600 50  0001 C CNN
@@
 $EndComp
 $Comp
-L Device:C C12
+L Device:C C11
 U 1 1 61930AF3
 P 6400 3750
-F 0 "C12" H 6515 3796 50  0000 L CNN
+F 0 "C11" H 6515 3796 50  0000 L CNN
 F 1 "0.1uF" H 6515 3705 50  0000 L CNN
 F 2 "Capacitor_SMD:C_0603_1608Metric_Pad1.08x0.95mm_HandSolder" H 6438 3600 50  0001 C CNN
@@
 $EndComp
 $Comp
-L Device:C C17
+L Device:C C16
 U 1 1 6195EA6D
 P 9200 4850
-F 0 "C17" V 9150 4900 50  0000 L CNN
+F 0 "C16" V 9150 4900 50  0000 L CNN
 F 1 "22pF" V 9150 4600 50  0000 L CNN
 F 2 "Capacitor_SMD:C_0603_1608Metric_Pad1.08x0.95mm_HandSolder" H 9238 4700 50  0001 C CNN
@@
 $EndComp
 $Comp
-L Device:C C16
+L Device:C C15
 U 1 1 6195E432
 P 9200 4450
-F 0 "C16" V 9250 4500 50  0000 L CNN
+F 0 "C15" V 9250 4500 50  0000 L CNN
 F 1 "22pF" V 9250 4200 50  0000 L CNN
 F 2 "Capacitor_SMD:C_0603_1608Metric_Pad1.08x0.95mm_HandSolder" H 9238 4300 50  0001 C CNN
@@
 Button4
 Wire Notes Line
-	1750 2050 1750 1000
-Wire Notes Line
-	1750 1000 750  1000
-Wire Notes Line
 	750  1000 750  2050
 Text Notes 800  1400 0    79   ~ 0
@@
 GeneratorVcc
 Wire Notes Line
-	1750 3900 1750 2850
-Wire Notes Line
-	1750 2850 750  2850
-Wire Notes Line
 	750  2850 750  3900
 Text Notes 800  3250 0    79   ~ 0
 Energy\nHarvesting\nGPIO/Analog In
-Wire Notes Line
-	750  2050 1750 2050
-Wire Notes Line
-	750  3900 1750 3900
 Text HLabel 1250 3600 0    50   Input ~ 0
 VBAT_OK
@@
 or just connect to ADC
 $Comp
-L Device:C C15
+L Device:C C14
 U 1 1 619E966F
 P 7900 3750
-F 0 "C15" H 8015 3796 50  0000 L CNN
+F 0 "C14" H 8015 3796 50  0000 L CNN
 F 1 "10uF" H 8015 3705 50  0000 L CNN
 F 2 "Capacitor_SMD:C_0805_2012Metric_Pad1.18x1.45mm_HandSolder" H 7938 3600 50  0001 C CNN
@@
 $EndComp
 $Comp
-L Device:C C18
+L Device:C C17
 U 1 1 6191DC18
 P 9500 1600
-F 0 "C18" H 9615 1646 50  0000 L CNN
+F 0 "C17" H 9615 1646 50  0000 L CNN
 F 1 "1nF" H 9615 1555 50  0000 L CNN
 F 2 "Capacitor_SMD:C_0603_1608Metric_Pad1.08x0.95mm_HandSolder" H 9538 1450 50  0001 C CNN
@@
 Text Label 9090 3100 2    50   ~ 0
 P5.0_DIN
+Wire Wire Line
+	1450 1950 2200 1950
+Wire Wire Line
+	2200 1950 2200 3300
+Wire Wire Line
+	2200 3300 3250 3300
+Wire Wire Line
+	3250 5400 2450 5400
+Wire Wire Line
+	3250 5600 2450 5600
+Wire Wire Line
+	3250 5700 2450 5700
+Wire Wire Line
+	3250 5800 2450 5800
+Text Label 3150 5400 2    50   ~ 0
+P5.3_Button1
+Text Label 3150 5600 2    50   ~ 0
+P5.5_Button2
+Text Label 3150 5700 2    50   ~ 0
+P5.6_Button3
+Text Label 3150 5800 2    50   ~ 0
+P5.7_Button4
+Text Label 1800 1500 2    50   ~ 0
+P5.3_Button1
+Wire Wire Line
+	1250 1500 1800 1500
+Wire Wire Line
+	1250 1600 1800 1600
+Wire Wire Line
+	1250 1700 1800 1700
+Wire Wire Line
+	1250 1800 1800 1800
+Wire Notes Line
+	750  1000 1850 1000
+Wire Notes Line
+	750  2050 1850 2050
+Wire Notes Line
+	1850 1000 1850 2050
+Text Label 1800 1600 2    50   ~ 0
+P5.5_Button2
+Text Label 1800 1700 2    50   ~ 0
+P5.6_Button3
+Text Label 1800 1800 2    50   ~ 0
+P5.7_Button4
+Wire Notes Line
+	750  2850 1850 2850
+Wire Notes Line
+	750  3900 1850 3900
+Wire Notes Line
+	1850 2850 1850 3900
+Wire Wire Line
+	1250 3600 2200 3600
+Wire Wire Line
+	2200 3600 2200 3400
+Wire Wire Line
+	2200 3400 3250 3400
+Wire Notes Line
+	8400 2100 10500 2100
+Wire Notes Line
+	8400 3350 10500 3350
+Wire Notes Line
+	8400 2100 8400 3350
+Text Notes 8500 2250 0    79   ~ 0
+E-ink Display
 $EndSCHEMATC

Commit message: just kinda out here guys ya know what im saying
Parts:
- added J400: GPIO_breakout, Connector_PinHeader_2.54mm:PinHeader_1x06_P2.54mm_Vertical, symbol Connector_Generic:Conn_01x06
- added J401: Multiplayer_Connector, Connector_PinHeader_2.54mm:PinHeader_1x02_P2.54mm_Horizontal, symbol Connector_Generic:Conn_01x02
- added R400: 0, Resistor_SMD:R_0805_2012Metric_Pad1.20x1.40mm_HandSolder, symbol Device:R_US
- added U401: SN74HCS32, Package_SO:TSSOP-14_4.4x5mm_P0.65mm, symbol batteryless_gaming_device-rescue:SN74HCS32
- J402: renamed from J2; value Program Header -> Program_Header; footprint (none) -> Connector_PinHeader_2.54mm:PinHeader_1x06_P2.54mm_Vertical
- R401: renamed from R13; footprint (none) -> Resistor_SMD:R_0603_1608Metric_Pad0.98x0.95mm_HandSolder; Digikey PN (none) -> RMCF0603JT47K0CT-ND
- U400: renamed from U4; footprint (none) -> Package_QFP:LQFP-64_10x10mm_P0.5mm
- Y400: renamed from Y1; footprint (none) -> Crystal:Crystal_SMD_3215-2Pin_3.2x1.5mm
- renumbered C10 to C400, C11 to C401, C12 to C402, C13 to C403, C14 to C404, C15 to C405, C16 to C406, C17 to C407, SW1 to SW400
Connections:
- net labels added: P2.6_OR_OUT, P3.4, P3.5, P3.6, P3.7, P6.0_TxD, P6.1_RxD, SN_3A_IN, SN_3B_IN
- wire segments 106 -> 132
- no-connect marks 18 -> 48
Other:
- note added: "BUTTON OR COUNTER"
- note added: "GPIO\nBREAKOUT"
- note added: "MULTIPLAYER\nPORT"
- note removed: "or just connect to ADC"
- note removed: "possibly add mosfet to switch 3.3V logic"
