File: KiCad/batteryless_gaming_device/power_regulation.sch (KiCad schematic (older format))
At the start: 11 parts

Commit message: k
Parts:
- removed D?: D, symbol Device:D
- added R? (x2): 0, Resistor_SMD:R_0805_2012Metric_Pad1.20x1.40mm_HandSolder, symbol Device:R_US
- added TP? (x2): TestPoint, TestPoint:TestPoint_Pad_D2.0mm, symbol Connector:TestPoint
- C? (x3): Digikey PN (none) -> 399-11939-1-ND
- C?: Digikey PN (none) -> 311-1344-1-ND
- C?, U?: Digikey PN (none) -> 296-21684-1-ND
- R?: value 1.24M -> 1M
- R?: value 200k -> 180k
Connections:
- net labels added: Vout
- net labels removed: +3.3V
- wire segments 56 -> 58
Other:
- note added: "R1=R2*(Vout/Vfb-1)\nVout=3.3V,Vfb=0.5V,R2<200k\nR2=180k=>R1=1.00M"
- note removed: "R1=R2*(Vout/Vfb-1)\nVout=3.6V,Vfb=0.5V,R2<200k\nR2=200k=>R1=1.24M"
Changed lines of the file:
@@
 AR Path="/619505DB" Ref="U?"  Part="1"
 AR Path="/61941831/619505DB" Ref="U?"  Part="1"
-F 0 "U?" H 5300 4417 50  0000 C CNN
-F 1 "TPS61201DRC" H 5300 4326 50  0000 C CNN
+F 0 "U?" H 5300 4415 50  0000 C CNN
+F 1 "TPS61201DRC" H 5300 4350 50  0000 C CNN
 F 2 "Package_SON:Texas_S-PVSON-N10_ThermalVias" H 5300 3500 50  0001 C CNN
 F 3 "http://www.ti.com/lit/ds/symlink/tps61200.pdf" H 5300 3950 50  0001 C CNN
+F 4 "296-21684-1-ND" H 5300 4290 39  0000 C CNN "Digikey PN"
 	1    5300 3950
 	1    0    0    -1
@@
 F 2 "" H 4150 3900 50  0001 C CNN
 F 3 "~" H 4150 3900 50  0001 C CNN
+F 4 "399-11939-1-ND" H 3950 3650 39  0000 C CNN "Digikey PN"
 	1    4150 3900
 	1    0    0    -1
@@
 F 2 "" H 6900 4000 50  0001 C CNN
 F 3 "~" H 6900 4000 50  0001 C CNN
+F 4 "399-11939-1-ND" H 7400 3750 39  0000 C CNN "Digikey PN"
 	1    6900 4000
 	1    0    0    -1
@@
 F 2 "" H 7300 4000 50  0001 C CNN
 F 3 "~" H 7300 4000 50  0001 C CNN
+F 4 "399-11939-1-ND" H 7400 3800 39  0000 C CNN "Digikey PN"
 	1    7300 4000
 	1    0    0    -1
@@
 F 2 "" H 4500 3900 50  0001 C CNN
 F 3 "~" H 4500 3900 50  0001 C CNN
+F 4 "311-1344-1-ND" H 4700 3650 39  0000 C CNN "Digikey PN"
 	1    4500 3900
 	1    0    0    -1
@@
 F 2 "" H 6500 4000 50  0001 C CNN
 F 3 "~" H 6500 4000 50  0001 C CNN
+F 4 "296-21684-1-ND" H 6590 3810 39  0000 C CNN "Digikey PN"
 	1    6500 4000
 	1    0    0    -1
@@
 AR Path="/61941831/61950619" Ref="R?"  Part="1"
 F 0 "R?" H 6218 4096 50  0000 L CNN
-F 1 "1.24M" H 6218 4005 50  0000 L CNN
+F 1 "1M" H 6218 4005 50  0000 L CNN
 F 2 "" V 6190 4040 50  0001 C CNN
 F 3 "~" H 6150 4050 50  0001 C CNN
@@
 AR Path="/61941831/6195061F" Ref="R?"  Part="1"
 F 0 "R?" H 6218 4446 50  0000 L CNN
-F 1 "200k" H 6218 4355 50  0000 L CNN
+F 1 "180k" H 6218 4355 50  0000 L CNN
 F 2 "" V 6190 4390 50  0001 C CNN
 F 3 "~" H 6150 4400 50  0001 C CNN
@@
 	6500 3850 6500 3900
 Wire Wire Line
-	6500 3850 6750 3850
-Wire Wire Line
 	6900 3850 6900 3900
 Connection ~ 6500 3850
 Wire Wire Line
-	6900 3850 7300 3850
+	6900 3850 7150 3850
 Wire Wire Line
 	7300 3850 7300 3900
@@
 Connection ~ 6150 4200
 Text Notes 6250 4800 0    50   ~ 0
-R1=R2*(Vout/Vfb-1)\nVout=3.6V,Vfb=0.5V,R2<200k\nR2=200k=>R1=1.24M
+R1=R2*(Vout/Vfb-1)\nVout=3.3V,Vfb=0.5V,R2<200k\nR2=180k=>R1=1.00M
 Text Notes 6200 3950 0    50   ~ 0
 R1
@@
 R2
 Wire Wire Line
-	4000 3750 4150 3750
+	3350 3750 3500 3750
+Wire Wire Line
+	4150 3750 4500 3750
+Text HLabel 3350 3750 0    50   Input ~ 0
+Vin
+Wire Wire Line
+	6500 3850 6900 3850
+Text HLabel 8150 3850 2    50   Output ~ 0
+Vout
+Connection ~ 7300 3850
+$Comp
+L Device:R_US R?
+U 1 1 6199BF77
+P 7800 3850
+AR Path="/61926AE2/6199BF77" Ref="R?"  Part="1"
+AR Path="/6199BF77" Ref="R?"  Part="1"
+AR Path="/61941831/6199BF77" Ref="R?"  Part="1"
+F 0 "R?" V 7950 3800 50  0000 L CNN
+F 1 "0" V 7868 3805 50  0000 L CNN
+F 2 "Resistor_SMD:R_0805_2012Metric_Pad1.20x1.40mm_HandSolder" V 7840 3840 50  0001 C CNN
+F 3 "~" H 7800 3850 50  0001 C CNN
+F 4 "YAG3755CT-ND" V 7700 3850 39  0000 C CNN "Digikey PN"
+	1    7800 3850
+	0    -1   -1   0
+$EndComp
+Wire Wire Line
+	7300 3850 7650 3850
+Wire Wire Line
+	7950 3850 8150 3850
+$Comp
+L Device:R_US R?
+U 1 1 619A0830
+P 3650 3750
+AR Path="/61926AE2/619A0830" Ref="R?"  Part="1"
+AR Path="/619A0830" Ref="R?"  Part="1"
+AR Path="/61941831/619A0830" Ref="R?"  Part="1"
+F 0 "R?" V 3800 3700 50  0000 L CNN
+F 1 "0" V 3718 3705 50  0000 L CNN
+F 2 "Resistor_SMD:R_0805_2012Metric_Pad1.20x1.40mm_HandSolder" V 3690 3740 50  0001 C CNN
+F 3 "~" H 3650 3750 50  0001 C CNN
+F 4 "YAG3755CT-ND" V 3550 3750 39  0000 C CNN "Digikey PN"
+	1    3650 3750
+	0    -1   -1   0
+$EndComp
+Wire Wire Line
+	3800 3750 3950 3750
 Connection ~ 4150 3750
-Wire Wire Line
-	4150 3750 4500 3750
-$Comp
-L Device:D D?
-U 1 1 61950678
-P 6950 3700
-AR Path="/61950678" Ref="D?"  Part="1"
-AR Path="/61941831/61950678" Ref="D?"  Part="1"
-F 0 "D?" H 6950 3483 50  0000 C CNN
-F 1 "D" H 6950 3574 50  0000 C CNN
-F 2 "" H 6950 3700 50  0001 C CNN
-F 3 "~" H 6950 3700 50  0001 C CNN
-	1    6950 3700
-	-1   0    0    1
-$EndComp
-Wire Wire Line
-	6750 3850 6750 3700
-Wire Wire Line
-	6750 3700 6800 3700
-Connection ~ 6750 3850
-Wire Wire Line
-	6750 3850 6900 3850
-$Comp
-L power:+3.3V #PWR?
-U 1 1 61950682
-P 7200 3650
-AR Path="/61950682" Ref="#PWR?"  Part="1"
-AR Path="/61941831/61950682" Ref="#PWR?"  Part="1"
-F 0 "#PWR?" H 7200 3500 50  0001 C CNN
-F 1 "+3.3V" H 7215 3823 50  0000 C CNN
-F 2 "" H 7200 3650 50  0001 C CNN
-F 3 "" H 7200 3650 50  0001 C CNN
-	1    7200 3650
-	1    0    0    -1
-$EndComp
-Wire Wire Line
-	7100 3700 7200 3700
-Wire Wire Line
-	7200 3700 7200 3650
-Text HLabel 4000 3750 0    50   Input ~ 0
-Vin
+$Comp
+L Connector:TestPoint TP?
+U 1 1 619A27A4
+P 3950 3700
+F 0 "TP?" H 4008 3818 50  0000 L CNN
+F 1 "TestPoint" H 4008 3727 50  0000 L CNN
+F 2 "TestPoint:TestPoint_Pad_D2.0mm" H 4150 3700 50  0001 C CNN
+F 3 "~" H 4150 3700 50  0001 C CNN
+	1    3950 3700
+	1    0    0    -1
+$EndComp
+Wire Wire Line
+	3950 3700 3950 3750
+Connection ~ 3950 3750
+Wire Wire Line
+	3950 3750 4150 3750
+$Comp
+L Connector:TestPoint TP?
+U 1 1 619A4F8F
+P 7150 3800
+F 0 "TP?" H 7208 3918 50  0000 L CNN
+F 1 "TestPoint" H 7208 3827 50  0000 L CNN
+F 2 "TestPoint:TestPoint_Pad_D2.0mm" H 7350 3800 50  0001 C CNN
+F 3 "~" H 7350 3800 50  0001 C CNN
+	1    7150 3800
+	1    0    0    -1
+$EndComp
+Wire Wire Line
+	7150 3800 7150 3850
+Connection ~ 7150 3850
+Wire Wire Line
+	7150 3850 7300 3850
 $EndSCHEMATC

Commit message: k
Parts:
- C19, C23, C24: renamed from C?; footprint (none) -> Capacitor_SMD:C_0805_2012Metric_Pad1.18x1.45mm_HandSolder
- C20, C22: renamed from C?; footprint (none) -> Capacitor_SMD:C_0603_1608Metric_Pad1.08x0.95mm_HandSolder
- C21: renamed from C?; footprint (none) -> Capacitor_SMD:C_0603_1608Metric_Pad1.08x0.95mm_HandSolder; Digikey PN (none) -> 1276-1946-1-ND
- gave numbers to parts that had none: 8
Changed lines of the file:
@@
 P 5300 3950
 AR Path="/619505DB" Ref="U?"  Part="1"
-AR Path="/61941831/619505DB" Ref="U?"  Part="1"
-F 0 "U?" H 5300 4415 50  0000 C CNN
+AR Path="/61941831/619505DB" Ref="U5"  Part="1"
+F 0 "U5" H 5300 4415 50  0000 C CNN
 F 1 "TPS61201DRC" H 5300 4350 50  0000 C CNN
 F 2 "Package_SON:Texas_S-PVSON-N10_ThermalVias" H 5300 3500 50  0001 C CNN
@@
 P 5300 3400
 AR Path="/619505E1" Ref="L?"  Part="1"
-AR Path="/61941831/619505E1" Ref="L?"  Part="1"
-F 0 "L?" V 5490 3400 50  0000 C CNN
+AR Path="/61941831/619505E1" Ref="L2"  Part="1"
+F 0 "L2" V 5490 3400 50  0000 C CNN
 F 1 "2.2u" V 5399 3400 50  0000 C CNN
 F 2 "" H 5300 3400 50  0001 C CNN
@@
 P 4150 3900
 AR Path="/619505E7" Ref="C?"  Part="1"
-AR Path="/61941831/619505E7" Ref="C?"  Part="1"
-F 0 "C?" H 4242 3946 50  0000 L CNN
+AR Path="/61941831/619505E7" Ref="C19"  Part="1"
+F 0 "C19" H 4242 3946 50  0000 L CNN
 F 1 "10uF" H 4242 3855 50  0000 L CNN
-F 2 "" H 4150 3900 50  0001 C CNN
+F 2 "Capacitor_SMD:C_0805_2012Metric_Pad1.18x1.45mm_HandSolder" H 4150 3900 50  0001 C CNN
 F 3 "~" H 4150 3900 50  0001 C CNN
 F 4 "399-11939-1-ND" H 3950 3650 39  0000 C CNN "Digikey PN"
@@
 P 5300 4550
 AR Path="/619505ED" Ref="#PWR?"  Part="1"
-AR Path="/61941831/619505ED" Ref="#PWR?"  Part="1"
-F 0 "#PWR?" H 5300 4300 50  0001 C CNN
+AR Path="/61941831/619505ED" Ref="#PWR026"  Part="1"
+F 0 "#PWR026" H 5300 4300 50  0001 C CNN
 F 1 "GND" H 5305 4377 50  0000 C CNN
 F 2 "" H 5300 4550 50  0001 C CNN
@@
 P 6900 4000
 AR Path="/619505F3" Ref="C?"  Part="1"
-AR Path="/61941831/619505F3" Ref="C?"  Part="1"
-F 0 "C?" H 6992 4046 50  0000 L CNN
+AR Path="/61941831/619505F3" Ref="C23"  Part="1"
+F 0 "C23" H 6992 4046 50  0000 L CNN
 F 1 "10uF" H 6992 3955 50  0000 L CNN
-F 2 "" H 6900 4000 50  0001 C CNN
+F 2 "Capacitor_SMD:C_0805_2012Metric_Pad1.18x1.45mm_HandSolder" H 6900 4000 50  0001 C CNN
 F 3 "~" H 6900 4000 50  0001 C CNN
 F 4 "399-11939-1-ND" H 7400 3750 39  0000 C CNN "Digikey PN"
@@
 P 5850 4050
 AR Path="/619505F9" Ref="C?"  Part="1"
-AR Path="/61941831/619505F9" Ref="C?"  Part="1"
-F 0 "C?" H 5942 4096 50  0000 L CNN
+AR Path="/61941831/619505F9" Ref="C21"  Part="1"
+F 0 "C21" H 5942 4096 50  0000 L CNN
 F 1 "1uF" H 5942 4005 50  0000 L CNN
-F 2 "" H 5850 4050 50  0001 C CNN
+F 2 "Capacitor_SMD:C_0603_1608Metric_Pad1.08x0.95mm_HandSolder" H 5850 4050 50  0001 C CNN
 F 3 "~" H 5850 4050 50  0001 C CNN
+F 4 "1276-1946-1-ND" H 5900 4200 39  0000 C CNN "Digikey PN"
 	1    5850 4050
 	1    0    0    -1
@@
 P 5850 4200
 AR Path="/619505FF" Ref="#PWR?"  Part="1"
-AR Path="/61941831/619505FF" Ref="#PWR?"  Part="1"
-F 0 "#PWR?" H 5850 3950 50  0001 C CNN
+AR Path="/61941831/619505FF" Ref="#PWR027"  Part="1"
+F 0 "#PWR027" H 5850 3950 50  0001 C CNN
 F 1 "GND" H 5855 4027 50  0000 C CNN
 F 2 "" H 5850 4200 50  0001 C CNN
@@
 P 7300 4000
 AR Path="/61950607" Ref="C?"  Part="1"
-AR Path="/61941831/61950607" Ref="C?"  Part="1"
-F 0 "C?" H 7392 4046 50  0000 L CNN
+AR Path="/61941831/61950607" Ref="C24"  Part="1"
+F 0 "C24" H 7392 4046 50  0000 L CNN
 F 1 "10uF" H 7392 3955 50  0000 L CNN
-F 2 "" H 7300 4000 50  0001 C CNN
+F 2 "Capacitor_SMD:C_0805_2012Metric_Pad1.18x1.45mm_HandSolder" H 7300 4000 50  0001 C CNN
 F 3 "~" H 7300 4000 50  0001 C CNN
 F 4 "399-11939-1-ND" H 7400 3800 39  0000 C CNN "Digikey PN"
@@
 P 4500 3900
 AR Path="/6195060D" Ref="C?"  Part="1"
-AR Path="/61941831/6195060D" Ref="C?"  Part="1"
-F 0 "C?" H 4592 3946 50  0000 L CNN
+AR Path="/61941831/6195060D" Ref="C20"  Part="1"
+F 0 "C20" H 4592 3946 50  0000 L CNN
 F 1 "0.1uF" H 4592 3855 50  0000 L CNN
-F 2 "" H 4500 3900 50  0001 C CNN
+F 2 "Capacitor_SMD:C_0603_1608Metric_Pad1.08x0.95mm_HandSolder" H 4500 3900 50  0001 C CNN
 F 3 "~" H 4500 3900 50  0001 C CNN
 F 4 "311-1344-1-ND" H 4700 3650 39  0000 C CNN "Digikey PN"
@@
 P 6500 4000
 AR Path="/61950613" Ref="C?"  Part="1"
-AR Path="/61941831/61950613" Ref="C?"  Part="1"
-F 0 "C?" H 6592 4046 50  0000 L CNN
+AR Path="/61941831/61950613" Ref="C22"  Part="1"
+F 0 "C22" H 6592 4046 50  0000 L CNN
 F 1 "0.1uF" H 6592 3955 50  0000 L CNN
-F 2 "" H 6500 4000 50  0001 C CNN
+F 2 "Capacitor_SMD:C_0603_1608Metric_Pad1.08x0.95mm_HandSolder" H 6500 4000 50  0001 C CNN
 F 3 "~" H 6500 4000 50  0001 C CNN
 F 4 "296-21684-1-ND" H 6590 3810 39  0000 C CNN "Digikey PN"
@@
 P 6150 4050
 AR Path="/61950619" Ref="R?"  Part="1"
-AR Path="/61941831/61950619" Ref="R?"  Part="1"
-F 0 "R?" H 6218 4096 50  0000 L CNN
+AR Path="/61941831/61950619" Ref="R15"  Part="1"
+F 0 "R15" H 6218 4096 50  0000 L CNN
 F 1 "1M" H 6218 4005 50  0000 L CNN
 F 2 "" V 6190 4040 50  0001 C CNN
@@
 P 6150 4400
 AR Path="/6195061F" Ref="R?"  Part="1"
-AR Path="/61941831/6195061F" Ref="R?"  Part="1"
-F 0 "R?" H 6218 4446 50  0000 L CNN
+AR Path="/61941831/6195061F" Ref="R16"  Part="1"
+F 0 "R16" H 6218 4446 50  0000 L CNN
 F 1 "180k" H 6218 4355 50  0000 L CNN
 F 2 "" V 6190 4390 50  0001 C CNN
@@
 P 4350 4150
 AR Path="/61950641" Ref="#PWR?"  Part="1"
-AR Path="/61941831/61950641" Ref="#PWR?"  Part="1"
-F 0 "#PWR?" H 4350 3900 50  0001 C CNN
+AR Path="/61941831/61950641" Ref="#PWR025"  Part="1"
+F 0 "#PWR025" H 4350 3900 50  0001 C CNN
 F 1 "GND" H 4355 3977 50  0000 C CNN
 F 2 "" H 4350 4150 50  0001 C CNN
@@
 P 6900 4200
 AR Path="/6195065B" Ref="#PWR?"  Part="1"
-AR Path="/61941831/6195065B" Ref="#PWR?"  Part="1"
-F 0 "#PWR?" H 6900 3950 50  0001 C CNN
+AR Path="/61941831/6195065B" Ref="#PWR029"  Part="1"
+F 0 "#PWR029" H 6900 3950 50  0001 C CNN
 F 1 "GND" H 6905 4027 50  0000 C CNN
 F 2 "" H 6900 4200 50  0001 C CNN
@@
 P 6150 4600
 AR Path="/61950666" Ref="#PWR?"  Part="1"
-AR Path="/61941831/61950666" Ref="#PWR?"  Part="1"
-F 0 "#PWR?" H 6150 4350 50  0001 C CNN
+AR Path="/61941831/61950666" Ref="#PWR028"  Part="1"
+F 0 "#PWR028" H 6150 4350 50  0001 C CNN
 F 1 "GND" H 6155 4427 50  0000 C CNN
 F 2 "" H 6150 4600 50  0001 C CNN
@@
 AR Path="/61926AE2/6199BF77" Ref="R?"  Part="1"
 AR Path="/6199BF77" Ref="R?"  Part="1"
-AR Path="/61941831/6199BF77" Ref="R?"  Part="1"
-F 0 "R?" V 7950 3800 50  0000 L CNN
+AR Path="/61941831/6199BF77" Ref="R17"  Part="1"
+F 0 "R17" V 7950 3800 50  0000 L CNN
 F 1 "0" V 7868 3805 50  0000 L CNN
 F 2 "Resistor_SMD:R_0805_2012Metric_Pad1.20x1.40mm_HandSolder" V 7840 3840 50  0001 C CNN
@@
 AR Path="/61926AE2/619A0830" Ref="R?"  Part="1"
 AR Path="/619A0830" Ref="R?"  Part="1"
-AR Path="/61941831/619A0830" Ref="R?"  Part="1"
-F 0 "R?" V 3800 3700 50  0000 L CNN
+AR Path="/61941831/619A0830" Ref="R14"  Part="1"
+F 0 "R14" V 3800 3700 50  0000 L CNN
 F 1 "0" V 3718 3705 50  0000 L CNN
 F 2 "Resistor_SMD:R_0805_2012Metric_Pad1.20x1.40mm_HandSolder" V 3690 3740 50  0001 C CNN
@@
 Connection ~ 4150 3750
 $Comp
-L Connector:TestPoint TP?
+L Connector:TestPoint TP4
 U 1 1 619A27A4
 P 3950 3700
-F 0 "TP?" H 4008 3818 50  0000 L CNN
+F 0 "TP4" H 4008 3818 50  0000 L CNN
 F 1 "TestPoint" H 4008 3727 50  0000 L CNN
 F 2 "TestPoint:TestPoint_Pad_D2.0mm" H 4150 3700 50  0001 C CNN
@@
 	3950 3750 4150 3750
 $Comp
-L Connector:TestPoint TP?
+L Connector:TestPoint TP5
 U 1 1 619A4F8F
 P 7150 3800
-F 0 "TP?" H 7208 3918 50  0000 L CNN
+F 0 "TP5" H 7208 3918 50  0000 L CNN
 F 1 "TestPoint" H 7208 3827 50  0000 L CNN
 F 2 "TestPoint:TestPoint_Pad_D2.0mm" H 7350 3800 50  0001 C CNN

Commit message: k
Parts:
- added R15, R16: 0, Resistor_SMD:R_0805_2012Metric_Pad1.20x1.40mm_HandSolder, symbol Device:R_US
- renumbered C19 to C18, C20 to C19, C21 to C20, C22 to C21, C23 to C22, C24 to C23, R15 to R17, R16 to R18, R17 to R19
Connections:
- net GND: now also R16.2
- net at C18.1, C19.1, L2.1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: now also R15.1; no longer U5.6 (EN), U5.8 (PS)
- new net: R15.2, U5.6 (EN)
- new net: R16.1, U5.8 (PS)
Other:
- moved on the sheet: C18, C19, R14, TP4
