File: KiCad/batteryless_gaming_device/power_regulation.sch (KiCad schematic (older format))
At the start: 16 parts, among them U5 TPS61201DRC

Commit message: just kinda out here guys ya know what im saying
Parts:
- L500: renamed from L2; footprint (none) -> Inductor_SMD:L_Taiyo-Yuden_NR-30xx_HandSoldering; Digikey PN (none) -> 587-1648-1-ND
- R503: renamed from R17; footprint (none) -> Resistor_SMD:R_0603_1608Metric_Pad0.98x0.95mm_HandSolder; Digikey PN (none) -> 511-1820-1-ND
- R504: renamed from R18; footprint (none) -> Resistor_SMD:R_0603_1608Metric_Pad0.98x0.95mm_HandSolder; Digikey PN (none) -> RMCF0603FT180KCT-ND
- renumbered C18 to C500, C19 to C501, C20 to C502, C21 to C503, C22 to C504, C23 to C505, R14 to R500, R15 to R501, R16 to R502, R19 to R505, TP4 to TP500, TP5 to TP501, U5 to U500
Changed lines of the file:
@@
 P 5300 3950
 AR Path="/619505DB" Ref="U?"  Part="1"
-AR Path="/61941831/619505DB" Ref="U5"  Part="1"
-F 0 "U5" H 5300 4415 50  0000 C CNN
+AR Path="/61941831/619505DB" Ref="U500"  Part="1"
+F 0 "U500" H 5300 4415 50  0000 C CNN
 F 1 "TPS61201DRC" H 5300 4350 50  0000 C CNN
 F 2 "Package_SON:Texas_S-PVSON-N10_ThermalVias" H 5300 3500 50  0001 C CNN
@@
 P 5300 3400
 AR Path="/619505E1" Ref="L?"  Part="1"
-AR Path="/61941831/619505E1" Ref="L2"  Part="1"
-F 0 "L2" V 5490 3400 50  0000 C CNN
-F 1 "2.2u" V 5399 3400 50  0000 C CNN
-F 2 "" H 5300 3400 50  0001 C CNN
+AR Path="/61941831/619505E1" Ref="L500"  Part="1"
+F 0 "L500" V 5490 3420 50  0000 C CNN
+F 1 "2.2u" V 5418 3402 50  0000 C CNN
+F 2 "Inductor_SMD:L_Taiyo-Yuden_NR-30xx_HandSoldering" H 5300 3400 50  0001 C CNN
 F 3 "~" H 5300 3400 50  0001 C CNN
+F 4 "587-1648-1-ND" V 5350 3400 39  0000 C CNN "Digikey PN"
 	1    5300 3400
 	0    -1   -1   0
@@
 P 3100 3900
 AR Path="/619505E7" Ref="C?"  Part="1"
-AR Path="/61941831/619505E7" Ref="C18"  Part="1"
-F 0 "C18" H 3192 3946 50  0000 L CNN
+AR Path="/61941831/619505E7" Ref="C500"  Part="1"
+F 0 "C500" H 3192 3946 50  0000 L CNN
 F 1 "10uF" H 3192 3855 50  0000 L CNN
 F 2 "Capacitor_SMD:C_0805_2012Metric_Pad1.18x1.45mm_HandSolder" H 3100 3900 50  0001 C CNN
@@
 P 5300 4550
 AR Path="/619505ED" Ref="#PWR?"  Part="1"
-AR Path="/61941831/619505ED" Ref="#PWR027"  Part="1"
-F 0 "#PWR027" H 5300 4300 50  0001 C CNN
+AR Path="/61941831/619505ED" Ref="#PWR0502"  Part="1"
+F 0 "#PWR0502" H 5300 4300 50  0001 C CNN
 F 1 "GND" H 5305 4377 50  0000 C CNN
 F 2 "" H 5300 4550 50  0001 C CNN
@@
 P 6900 4000
 AR Path="/619505F3" Ref="C?"  Part="1"
-AR Path="/61941831/619505F3" Ref="C22"  Part="1"
-F 0 "C22" H 6992 4046 50  0000 L CNN
+AR Path="/61941831/619505F3" Ref="C504"  Part="1"
+F 0 "C504" H 6992 4046 50  0000 L CNN
 F 1 "10uF" H 6992 3955 50  0000 L CNN
 F 2 "Capacitor_SMD:C_0805_2012Metric_Pad1.18x1.45mm_HandSolder" H 6900 4000 50  0001 C CNN
@@
 P 5850 4050
 AR Path="/619505F9" Ref="C?"  Part="1"
-AR Path="/61941831/619505F9" Ref="C20"  Part="1"
-F 0 "C20" H 5942 4096 50  0000 L CNN
+AR Path="/61941831/619505F9" Ref="C502"  Part="1"
+F 0 "C502" H 5942 4096 50  0000 L CNN
 F 1 "1uF" H 5942 4005 50  0000 L CNN
 F 2 "Capacitor_SMD:C_0603_1608Metric_Pad1.08x0.95mm_HandSolder" H 5850 4050 50  0001 C CNN
@@
 P 5850 4200
 AR Path="/619505FF" Ref="#PWR?"  Part="1"
-AR Path="/61941831/619505FF" Ref="#PWR028"  Part="1"
-F 0 "#PWR028" H 5850 3950 50  0001 C CNN
+AR Path="/61941831/619505FF" Ref="#PWR0503"  Part="1"
+F 0 "#PWR0503" H 5850 3950 50  0001 C CNN
 F 1 "GND" H 5855 4027 50  0000 C CNN
 F 2 "" H 5850 4200 50  0001 C CNN
@@
 P 7300 4000
 AR Path="/61950607" Ref="C?"  Part="1"
-AR Path="/61941831/61950607" Ref="C23"  Part="1"
-F 0 "C23" H 7392 4046 50  0000 L CNN
+AR Path="/61941831/61950607" Ref="C505"  Part="1"
+F 0 "C505" H 7392 4046 50  0000 L CNN
 F 1 "10uF" H 7392 3955 50  0000 L CNN
 F 2 "Capacitor_SMD:C_0805_2012Metric_Pad1.18x1.45mm_HandSolder" H 7300 4000 50  0001 C CNN
@@
 P 3450 3900
 AR Path="/6195060D" Ref="C?"  Part="1"
-AR Path="/61941831/6195060D" Ref="C19"  Part="1"
-F 0 "C19" H 3542 3946 50  0000 L CNN
+AR Path="/61941831/6195060D" Ref="C501"  Part="1"
+F 0 "C501" H 3542 3946 50  0000 L CNN
 F 1 "0.1uF" H 3542 3855 50  0000 L CNN
 F 2 "Capacitor_SMD:C_0603_1608Metric_Pad1.08x0.95mm_HandSolder" H 3450 3900 50  0001 C CNN
@@
 P 6500 4000
 AR Path="/61950613" Ref="C?"  Part="1"
-AR Path="/61941831/61950613" Ref="C21"  Part="1"
-F 0 "C21" H 6592 4046 50  0000 L CNN
+AR Path="/61941831/61950613" Ref="C503"  Part="1"
+F 0 "C503" H 6592 4046 50  0000 L CNN
 F 1 "0.1uF" H 6592 3955 50  0000 L CNN
 F 2 "Capacitor_SMD:C_0603_1608Metric_Pad1.08x0.95mm_HandSolder" H 6500 4000 50  0001 C CNN
@@
 P 6150 4050
 AR Path="/61950619" Ref="R?"  Part="1"
-AR Path="/61941831/61950619" Ref="R17"  Part="1"
-F 0 "R17" H 6218 4096 50  0000 L CNN
+AR Path="/61941831/61950619" Ref="R503"  Part="1"
+F 0 "R503" H 6218 4096 50  0000 L CNN
 F 1 "1M" H 6218 4005 50  0000 L CNN
-F 2 "" V 6190 4040 50  0001 C CNN
+F 2 "Resistor_SMD:R_0603_1608Metric_Pad0.98x0.95mm_HandSolder" V 6190 4040 50  0001 C CNN
 F 3 "~" H 6150 4050 50  0001 C CNN
+F 4 "511-1820-1-ND" H 6200 4300 39  0000 C CNN "Digikey PN"
 	1    6150 4050
 	1    0    0    -1
@@
 P 6150 4400
 AR Path="/6195061F" Ref="R?"  Part="1"
-AR Path="/61941831/6195061F" Ref="R18"  Part="1"
-F 0 "R18" H 6218 4446 50  0000 L CNN
+AR Path="/61941831/6195061F" Ref="R504"  Part="1"
+F 0 "R504" H 6218 4446 50  0000 L CNN
 F 1 "180k" H 6218 4355 50  0000 L CNN
-F 2 "" V 6190 4390 50  0001 C CNN
+F 2 "Resistor_SMD:R_0603_1608Metric_Pad0.98x0.95mm_HandSolder" V 6190 4390 50  0001 C CNN
 F 3 "~" H 6150 4400 50  0001 C CNN
+F 4 "RMCF0603FT180KCT-ND" H 6550 4300 39  0000 C CNN "Digikey PN"
 	1    6150 4400
 	1    0    0    -1
@@
 P 3300 4150
 AR Path="/61950641" Ref="#PWR?"  Part="1"
-AR Path="/61941831/61950641" Ref="#PWR025"  Part="1"
-F 0 "#PWR025" H 3300 3900 50  0001 C CNN
+AR Path="/61941831/61950641" Ref="#PWR0500"  Part="1"
+F 0 "#PWR0500" H 3300 3900 50  0001 C CNN
 F 1 "GND" H 3305 3977 50  0000 C CNN
 F 2 "" H 3300 4150 50  0001 C CNN
@@
 P 6900 4200
 AR Path="/6195065B" Ref="#PWR?"  Part="1"
-AR Path="/61941831/6195065B" Ref="#PWR030"  Part="1"
-F 0 "#PWR030" H 6900 3950 50  0001 C CNN
+AR Path="/61941831/6195065B" Ref="#PWR0505"  Part="1"
+F 0 "#PWR0505" H 6900 3950 50  0001 C CNN
 F 1 "GND" H 6905 4027 50  0000 C CNN
 F 2 "" H 6900 4200 50  0001 C CNN
@@
 P 6150 4600
 AR Path="/61950666" Ref="#PWR?"  Part="1"
-AR Path="/61941831/61950666" Ref="#PWR029"  Part="1"
-F 0 "#PWR029" H 6150 4350 50  0001 C CNN
+AR Path="/61941831/61950666" Ref="#PWR0504"  Part="1"
+F 0 "#PWR0504" H 6150 4350 50  0001 C CNN
 F 1 "GND" H 6155 4427 50  0000 C CNN
 F 2 "" H 6150 4600 50  0001 C CNN
@@
 AR Path="/61926AE2/6199BF77" Ref="R?"  Part="1"
 AR Path="/6199BF77" Ref="R?"  Part="1"
-AR Path="/61941831/6199BF77" Ref="R19"  Part="1"
-F 0 "R19" V 7950 3800 50  0000 L CNN
+AR Path="/61941831/6199BF77" Ref="R505"  Part="1"
+F 0 "R505" V 7950 3800 50  0000 L CNN
 F 1 "0" V 7868 3805 50  0000 L CNN
 F 2 "Resistor_SMD:R_0805_2012Metric_Pad1.20x1.40mm_HandSolder" V 7840 3840 50  0001 C CNN
@@
 AR Path="/61926AE2/619A0830" Ref="R?"  Part="1"
 AR Path="/619A0830" Ref="R?"  Part="1"
-AR Path="/61941831/619A0830" Ref="R14"  Part="1"
-F 0 "R14" V 2750 3700 50  0000 L CNN
+AR Path="/61941831/619A0830" Ref="R500"  Part="1"
+F 0 "R500" V 2750 3700 50  0000 L CNN
 F 1 "0" V 2668 3705 50  0000 L CNN
 F 2 "Resistor_SMD:R_0805_2012Metric_Pad1.20x1.40mm_HandSolder" V 2640 3740 50  0001 C CNN
@@
 Connection ~ 3100 3750
 $Comp
-L Connector:TestPoint TP4
+L Connector:TestPoint TP500
 U 1 1 619A27A4
 P 2900 3700
-F 0 "TP4" H 2958 3818 50  0000 L CNN
+F 0 "TP500" H 2958 3818 50  0000 L CNN
 F 1 "TestPoint" H 2958 3727 50  0000 L CNN
 F 2 "TestPoint:TestPoint_Pad_D2.0mm" H 3100 3700 50  0001 C CNN
@@
 	2900 3750 3100 3750
 $Comp
-L Connector:TestPoint TP5
+L Connector:TestPoint TP501
 U 1 1 619A4F8F
 P 7150 3800
-F 0 "TP5" H 7208 3918 50  0000 L CNN
+F 0 "TP501" H 7208 3918 50  0000 L CNN
 F 1 "TestPoint" H 7208 3827 50  0000 L CNN
 F 2 "TestPoint:TestPoint_Pad_D2.0mm" H 7350 3800 50  0001 C CNN
@@
 AR Path="/61926AE2/61A2D45D" Ref="R?"  Part="1"
 AR Path="/61A2D45D" Ref="R?"  Part="1"
-AR Path="/61941831/61A2D45D" Ref="R16"  Part="1"
-F 0 "R16" V 4900 4250 50  0000 L CNN
+AR Path="/61941831/61A2D45D" Ref="R502"  Part="1"
+F 0 "R502" V 4900 4250 50  0000 L CNN
 F 1 "0" V 4818 4255 50  0000 L CNN
 F 2 "Resistor_SMD:R_0805_2012Metric_Pad1.20x1.40mm_HandSolder" V 4790 4290 50  0001 C CNN
@@
 	1    0    0    -1
 $EndComp
-Wire Wire Line
-	3450 3750 4200 3750
 Connection ~ 4750 3750
 $Comp
@@
 AR Path="/61926AE2/61A310EA" Ref="R?"  Part="1"
 AR Path="/61A310EA" Ref="R?"  Part="1"
-AR Path="/61941831/61A310EA" Ref="R15"  Part="1"
-F 0 "R15" V 4434 3934 50  0000 L CNN
+AR Path="/61941831/61A310EA" Ref="R501"  Part="1"
+F 0 "R501" V 4434 3934 50  0000 L CNN
 F 1 "0" V 4432 3724 50  0000 L CNN
 F 2 "Resistor_SMD:R_0805_2012Metric_Pad1.20x1.40mm_HandSolder" V 4440 3840 50  0001 C CNN
@@
 P 4750 4500
 AR Path="/61A391BB" Ref="#PWR?"  Part="1"
-AR Path="/61941831/61A391BB" Ref="#PWR026"  Part="1"
-F 0 "#PWR026" H 4750 4250 50  0001 C CNN
+AR Path="/61941831/61A391BB" Ref="#PWR0501"  Part="1"
+F 0 "#PWR0501" H 4750 4250 50  0001 C CNN
 F 1 "GND" H 4755 4327 50  0000 C CNN
 F 2 "" H 4750 4500 50  0001 C CNN
@@
 Wire Wire Line
 	4750 4450 4750 4500
+Wire Wire Line
+	3450 3750 3850 3750
+$Comp
+L power:PWR_FLAG #FLG0105
+U 1 1 61C1CBC2
+P 3850 3700
+F 0 "#FLG0105" H 3850 3775 50  0001 C CNN
+F 1 "PWR_FLAG" H 3850 3873 50  0000 C CNN
+F 2 "" H 3850 3700 50  0001 C CNN
+F 3 "~" H 3850 3700 50  0001 C CNN
+	1    3850 3700
+	1    0    0    -1
+$EndComp
+Wire Wire Line
+	3850 3700 3850 3750
+Connection ~ 3850 3750
+Wire Wire Line
+	3850 3750 4200 3750
 $EndSCHEMATC

Commit message: oh ya
Parts:
- C503: Digikey PN 296-21684-1-ND -> 311-1344-1-ND
Changed lines of the file:
@@
 F 2 "Capacitor_SMD:C_0603_1608Metric_Pad1.08x0.95mm_HandSolder" H 6500 4000 50  0001 C CNN
 F 3 "~" H 6500 4000 50  0001 C CNN
-F 4 "296-21684-1-ND" H 6590 3810 39  0000 C CNN "Digikey PN"
+F 4 "311-1344-1-ND" H 6590 3810 39  0000 C CNN "Digikey PN"
 	1    6500 4000
 	1    0    0    -1

Commit message: updated
Parts:
- R504: value 180k -> 2M; Digikey PN RMCF0603FT180KCT-ND -> (none)
Connections:
- net at R503.2, R504.1: now also U500.7 (UVLO); no longer U500.10 (FB)
- net at C503.1, C504.1, C505.1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: now also U500.10 (FB); no longer R503.1
- net at C500.1, C501.1, L500.1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: now also R503.1; no longer U500.7 (UVLO)
Other:
- note added: "Not correct resistor values for UVLO"
- note removed: "R1"
- note removed: "R1=R2*(Vout/Vfb-1)\nVout=3.3V,Vfb=0.5V,R2<200k\nR2=180k=>R1=1.00M"
- note removed: "R2"
Changed lines of the file:
@@
-	1    0    0    -1
-$EndComp
-$Comp
-L Device:R_US R?
-U 1 1 61950619
-P 6150 4050
-AR Path="/61950619" Ref="R?"  Part="1"
-AR Path="/61941831/61950619" Ref="R503"  Part="1"
-F 0 "R503" H 6218 4096 50  0000 L CNN
-F 1 "1M" H 6218 4005 50  0000 L CNN
-F 2 "Resistor_SMD:R_0603_1608Metric_Pad0.98x0.95mm_HandSolder" V 6190 4040 50  0001 C CNN
-F 3 "~" H 6150 4050 50  0001 C CNN
-F 4 "511-1820-1-ND" H 6200 4300 39  0000 C CNN "Digikey PN"
-	1    6150 4050
-	1    0    0    -1
-$EndComp
-$Comp
-L Device:R_US R?
-U 1 1 6195061F
-P 6150 4400
-AR Path="/6195061F" Ref="R?"  Part="1"
-AR Path="/61941831/6195061F" Ref="R504"  Part="1"
-F 0 "R504" H 6218 4446 50  0000 L CNN
-F 1 "180k" H 6218 4355 50  0000 L CNN
-F 2 "Resistor_SMD:R_0603_1608Metric_Pad0.98x0.95mm_HandSolder" V 6190 4390 50  0001 C CNN
-F 3 "~" H 6150 4400 50  0001 C CNN
-F 4 "RMCF0603FT180KCT-ND" H 6550 4300 39  0000 C CNN "Digikey PN"
-	1    6150 4400
 	1    0    0    -1
 $EndComp
@@
 	1    0    0    -1
 $EndComp
-Wire Wire Line
-	5700 3850 6150 3850
-Wire Wire Line
-	6150 3900 6150 3850
-Connection ~ 6150 3850
-Wire Wire Line
-	6150 3850 6500 3850
-Wire Wire Line
-	6150 4200 6150 4250
-$Comp
-L power:GND #PWR?
-U 1 1 61950666
-P 6150 4600
-AR Path="/61950666" Ref="#PWR?"  Part="1"
-AR Path="/61941831/61950666" Ref="#PWR0504"  Part="1"
-F 0 "#PWR0504" H 6150 4350 50  0001 C CNN
-F 1 "GND" H 6155 4427 50  0000 C CNN
-F 2 "" H 6150 4600 50  0001 C CNN
-F 3 "" H 6150 4600 50  0001 C CNN
-	1    6150 4600
-	1    0    0    -1
-$EndComp
-Wire Wire Line
-	6150 4600 6150 4550
-Wire Wire Line
-	6150 4200 6050 4200
-Wire Wire Line
-	6050 4200 6050 4500
-Wire Wire Line
-	6050 4500 5700 4500
-Wire Wire Line
-	5700 4500 5700 4150
-Connection ~ 6150 4200
-Text Notes 6250 4800 0    50   ~ 0
-R1=R2*(Vout/Vfb-1)\nVout=3.3V,Vfb=0.5V,R2<200k\nR2=180k=>R1=1.00M
-Text Notes 6200 3950 0    50   ~ 0
-R1
-Text Notes 6200 4300 0    50   ~ 0
-R2
 Wire Wire Line
 	2300 3750 2450 3750
@@
 F 2 "Resistor_SMD:R_0805_2012Metric_Pad1.20x1.40mm_HandSolder" V 4790 4290 50  0001 C CNN
 F 3 "~" H 4750 4300 50  0001 C CNN
-F 4 "YAG3755CT-ND" H 4450 4300 39  0000 C CNN "Digikey PN"
+F 4 "YAG3755CT-ND" H 4850 4150 39  0000 C CNN "Digikey PN"
 	1    4750 4300
 	1    0    0    -1
@@
 	4200 3850 4250 3850
 Wire Wire Line
-	4200 4050 4900 4050
-Wire Wire Line
 	4200 3850 4200 3750
 Connection ~ 4200 3850
@@
 Wire Wire Line
 	3850 3750 4200 3750
+$Comp
+L Device:R_US R?
+U 1 1 61B125C6
+P 4200 4200
+AR Path="/61B125C6" Ref="R?"  Part="1"
+AR Path="/61941831/61B125C6" Ref="R503"  Part="1"
+F 0 "R503" H 4268 4246 50  0000 L CNN
+F 1 "1M" H 4268 4155 50  0000 L CNN
+F 2 "Resistor_SMD:R_0603_1608Metric_Pad0.98x0.95mm_HandSolder" V 4240 4190 50  0001 C CNN
+F 3 "~" H 4200 4200 50  0001 C CNN
+F 4 "511-1820-1-ND" H 4250 4350 39  0000 C CNN "Digikey PN"
+	1    4200 4200
+	1    0    0    -1
+$EndComp
+Wire Wire Line
+	5700 3850 6250 3850
+$Comp
+L Device:R_US R?
+U 1 1 61B1718F
+P 4200 4600
+AR Path="/61B1718F" Ref="R?"  Part="1"
+AR Path="/61941831/61B1718F" Ref="R504"  Part="1"
+F 0 "R504" H 4268 4646 50  0000 L CNN
+F 1 "2M" H 4268 4555 50  0000 L CNN
+F 2 "Resistor_SMD:R_0603_1608Metric_Pad0.98x0.95mm_HandSolder" V 4240 4590 50  0001 C CNN
+F 3 "~" H 4200 4600 50  0001 C CNN
+F 4 "" H 3950 4750 39  0000 C CNN "Digikey PN"
+	1    4200 4600
+	1    0    0    -1
+$EndComp
+$Comp
+L power:GND #PWR?
+U 1 1 61B17DBB
+P 4200 4750
+AR Path="/61B17DBB" Ref="#PWR?"  Part="1"
+AR Path="/61941831/61B17DBB" Ref="#PWR0115"  Part="1"
+F 0 "#PWR0115" H 4200 4500 50  0001 C CNN
+F 1 "GND" H 4205 4577 50  0000 C CNN
+F 2 "" H 4200 4750 50  0001 C CNN
+F 3 "" H 4200 4750 50  0001 C CNN
+	1    4200 4750
+	1    0    0    -1
+$EndComp
+Wire Wire Line
+	4200 4450 4200 4400
+Wire Wire Line
+	4200 4400 4600 4400
+Wire Wire Line
+	4600 4400 4600 4050
+Wire Wire Line
+	4600 4050 4900 4050
+Connection ~ 4200 4400
+Wire Wire Line
+	4200 4400 4200 4350
+Wire Wire Line
+	5700 4150 5700 4450
+Wire Wire Line
+	5700 4450 6250 4450
+Wire Wire Line
+	6250 4450 6250 3850
+Connection ~ 6250 3850
+Wire Wire Line
+	6250 3850 6500 3850
+Text Notes 4050 4650 2    50   ~ 0
+Not correct resistor values for UVLO
 $EndSCHEMATC
