File: KiCad/batteryless_gaming_device/power_storage.sch (KiCad schematic (older format))
At the start: 18 parts

Commit message: updated schematic
Parts:
- C?: value 220m -> 220mF
- C?: value 0.1u -> 0.1uF
- C?: value 10u -> 10uF
- C?: value 0.01u -> 0.01uF
- R?: value 4.32M -> 5.62M
- R?: value 1.67M -> 0.39M
- R?: value 1.3M -> 1.69M
- R?: value 6.2M -> 6.98M
- R?: value 2.7M -> 1.4M
- R?: value 8.25M -> 9.76M
- R?: value 5.6M -> 4.53M
Connections:
- net labels added: VBAT_OK, Vin, Vout
- net labels removed: +3.3V
- no-connect marks 1 -> 0
Other:
- note added: "VBAT_OV=4.2V\nVBAT_UV=1.3V\n\nVBAT_OK=1.5V\nVBAT_OK_HYST=1.8V\n"

Commit message: k
Parts:
- added C? (x4): 10uF, symbol Device:C_Small
- added TP? (x3): TestPoint, TestPoint:TestPoint_Pad_D2.0mm, symbol Connector:TestPoint
- C?: value 4.7u -> 4.7uF
- C?: Digikey PN (none) -> 311-1344-1-ND
- C?: Digikey PN (none) -> 399-11939-1-ND
- C?: value 47u -> 47uF
- C?: Digikey PN (none) -> 1276-CL10B103KB8WPJCCT-ND
- D?: value Zener -> 4V
Connections:
- wire segments 82 -> 99
Other:
- moved on the sheet: C?
Changed lines of the file:
@@
 	7400 2450 7400 2500
 Wire Wire Line
-	7100 2450 7400 2450
+	7100 2450 7150 2450
 Wire Wire Line
 	7100 2700 7100 2450
@@
 	1    0    0    -1
 $EndComp
-Connection ~ 5100 2650
-Wire Wire Line
-	4750 2950 5100 2950
-Connection ~ 4750 2950
-Wire Wire Line
-	4350 2950 4750 2950
-Wire Wire Line
-	4750 2650 4750 2700
-Wire Wire Line
-	4750 2950 4750 2900
-Wire Wire Line
-	4750 2650 5100 2650
-Connection ~ 4750 2650
 Connection ~ 4850 3950
 Connection ~ 4500 3950
@@
 	6100 4450 6500 4450
 Connection ~ 6500 4450
-$Comp
-L Diode:ZMMxx D?
-U 1 1 619D7F03
-P 3800 2850
-AR Path="/619D7F03" Ref="D?"  Part="1"
-AR Path="/61991596/619D7F03" Ref="D?"  Part="1"
-F 0 "D?" V 3754 2930 50  0000 L CNN
-F 1 "Zener" V 3845 2930 50  0000 L CNN
-F 2 "Diode_SMD:D_MiniMELF" H 3800 2675 50  0001 C CNN
-F 3 "https://diotec.com/tl_files/diotec/files/pdf/datasheets/zmm1.pdf" H 3800 2850 50  0001 C CNN
-	1    3800 2850
-	0    1    1    0
-$EndComp
-Wire Wire Line
-	3800 2700 3800 2650
-Wire Wire Line
-	3800 2650 4750 2650
-Wire Wire Line
-	3800 3000 4350 3000
-Wire Wire Line
-	4350 3000 4350 2950
-Wire Wire Line
-	3800 2650 3300 2650
-Connection ~ 3800 2650
-Wire Wire Line
-	3800 3000 3300 3000
-Wire Wire Line
-	3300 3000 3300 2950
-Connection ~ 3800 3000
 Wire Wire Line
 	6700 4300 6700 4450
-Text HLabel 2550 2650 0    50   Input ~ 0
-Vin
-Text HLabel 8400 3800 2    50   Output ~ 0
-Vout
-Wire Wire Line
-	7850 3800 8400 3800
+Wire Wire Line
+	7850 3800 8000 3800
 Connection ~ 7850 3800
 $Comp
@@
 F 2 "" H 5750 4200 50  0001 C CNN
 F 3 "~" H 5750 4200 50  0001 C CNN
+F 4 "1276-CL10B103KB8WPJCCT-ND" V 5850 3600 39  0000 C CNN "Digikey PN"
 	1    5750 4200
 	1    0    0    -1
@@
 F 2 "" H 7850 3950 50  0001 C CNN
 F 3 "~" H 7850 3950 50  0001 C CNN
+F 4 "311-1344-1-ND" H 8150 3850 39  0000 C CNN "Digikey PN"
 	1    7850 3950
 	1    0    0    -1
@@
 F 2 "" H 7450 3950 50  0001 C CNN
 F 3 "~" H 7450 3950 50  0001 C CNN
+F 4 "399-11939-1-ND" H 7500 3850 39  0000 C CNN "Digikey PN"
 	1    7450 3950
 	1    0    0    -1
@@
 P 5100 2800
 F 0 "C?" H 5192 2846 50  0000 L CNN
-F 1 "4.7u" H 5192 2755 50  0000 L CNN
+F 1 "4.7uF" H 5192 2755 50  0000 L CNN
 F 2 "" H 5100 2800 50  0001 C CNN
 F 3 "~" H 5100 2800 50  0001 C CNN
@@
 	1    0    0    -1
 $EndComp
+Text Notes 3550 4000 0    50   ~ 0
+VBAT_OV=4.2V\nVBAT_UV=1.3V\n\nVBAT_OK=1.5V\nVBAT_OK_HYST=1.8V\n
+Wire Wire Line
+	7300 3200 7700 3200
+Text HLabel 7700 3200 2    50   Output ~ 0
+VBAT_OK
+Text HLabel 8400 3800 2    50   Output ~ 0
+Vout
+$Comp
+L Connector:TestPoint TP?
+U 1 1 619CF02B
+P 7150 2400
+AR Path="/61941831/619CF02B" Ref="TP?"  Part="1"
+AR Path="/61991596/619CF02B" Ref="TP?"  Part="1"
+F 0 "TP?" H 7208 2518 50  0000 L CNN
+F 1 "TestPoint" H 7208 2427 50  0000 L CNN
+F 2 "TestPoint:TestPoint_Pad_D2.0mm" H 7350 2400 50  0001 C CNN
+F 3 "~" H 7350 2400 50  0001 C CNN
+	1    7150 2400
+	1    0    0    -1
+$EndComp
+Wire Wire Line
+	7150 2400 7150 2450
+Connection ~ 7150 2450
+Wire Wire Line
+	7150 2450 7400 2450
+$Comp
+L Connector:TestPoint TP?
+U 1 1 619D3EDF
+P 8000 3750
+AR Path="/61941831/619D3EDF" Ref="TP?"  Part="1"
+AR Path="/61991596/619D3EDF" Ref="TP?"  Part="1"
+F 0 "TP?" H 8058 3868 50  0000 L CNN
+F 1 "TestPoint" H 8058 3777 50  0000 L CNN
+F 2 "TestPoint:TestPoint_Pad_D2.0mm" H 8200 3750 50  0001 C CNN
+F 3 "~" H 8200 3750 50  0001 C CNN
+	1    8000 3750
+	1    0    0    -1
+$EndComp
+Wire Wire Line
+	8000 3750 8000 3800
+Connection ~ 8000 3800
+Wire Wire Line
+	8000 3800 8400 3800
+Wire Wire Line
+	3100 2950 3450 2950
+Wire Wire Line
+	3100 2650 3100 2700
+Wire Wire Line
+	3100 2950 3100 2900
+Wire Wire Line
+	3100 2650 3250 2650
+Connection ~ 3100 2650
 $Comp
 L Device:CP1_Small C?
 U 1 1 6199CFFF
-P 4750 2800
+P 3100 2800
 AR Path="/6199CFFF" Ref="C?"  Part="1"
 AR Path="/61991596/6199CFFF" Ref="C?"  Part="1"
-F 0 "C?" H 4841 2846 50  0000 L CNN
-F 1 "47u" H 4841 2755 50  0000 L CNN
-F 2 "" H 4750 2800 50  0001 C CNN
-F 3 "~" H 4750 2800 50  0001 C CNN
-	1    4750 2800
-	1    0    0    -1
-$EndComp
-Text Notes 3550 4000 0    50   ~ 0
-VBAT_OV=4.2V\nVBAT_UV=1.3V\n\nVBAT_OK=1.5V\nVBAT_OK_HYST=1.8V\n
-Text HLabel 7700 3200 2    50   Output ~ 0
-VBAT_OK
-Wire Wire Line
-	7300 3200 7700 3200
+F 0 "C?" H 3191 2846 50  0000 L CNN
+F 1 "47uF" H 3191 2755 50  0000 L CNN
+F 2 "" H 3100 2800 50  0001 C CNN
+F 3 "~" H 3100 2800 50  0001 C CNN
+	1    3100 2800
+	1    0    0    -1
+$EndComp
+$Comp
+L Diode:ZMMxx D?
+U 1 1 619D7F03
+P 2750 2800
+AR Path="/619D7F03" Ref="D?"  Part="1"
+AR Path="/61991596/619D7F03" Ref="D?"  Part="1"
+F 0 "D?" V 2704 2880 50  0000 L CNN
+F 1 "4V" V 2795 2880 50  0000 L CNN
+F 2 "Diode_SMD:D_MiniMELF" H 2750 2625 50  0001 C CNN
+F 3 "https://diotec.com/tl_files/diotec/files/pdf/datasheets/zmm1.pdf" H 2750 2800 50  0001 C CNN
+	1    2750 2800
+	0    1    1    0
+$EndComp
+Wire Wire Line
+	2750 2650 3100 2650
+Wire Wire Line
+	2750 2950 3100 2950
+Connection ~ 3100 2950
+Connection ~ 2750 2650
+Wire Wire Line
+	2450 2650 2750 2650
+Text HLabel 2450 2650 0    50   Input ~ 0
+Vin
+$Comp
+L Connector:TestPoint TP?
+U 1 1 619D814E
+P 3250 2600
+AR Path="/61941831/619D814E" Ref="TP?"  Part="1"
+AR Path="/61991596/619D814E" Ref="TP?"  Part="1"
+F 0 "TP?" H 3308 2718 50  0000 L CNN
+F 1 "TestPoint" H 3308 2627 50  0000 L CNN
+F 2 "TestPoint:TestPoint_Pad_D2.0mm" H 3450 2600 50  0001 C CNN
+F 3 "~" H 3450 2600 50  0001 C CNN
+	1    3250 2600
+	1    0    0    -1
+$EndComp
+Wire Wire Line
+	3250 2600 3250 2650
+Connection ~ 3250 2650
+$Comp
+L Device:C_Small C?
+U 1 1 619F0CC5
+P 3450 2800
+F 0 "C?" H 3480 2870 50  0000 L CNN
+F 1 "10uF" H 3520 2805 50  0000 L CNN
+F 2 "" H 3450 2800 50  0001 C CNN
+F 3 "~" H 3450 2800 50  0001 C CNN
+F 4 "DNU" H 3545 2735 50  0000 C CNN "Digikey PN"
+	1    3450 2800
+	1    0    0    -1
+$EndComp
+$Comp
+L Device:C_Small C?
+U 1 1 619F1106
+P 3800 2800
+F 0 "C?" H 3825 2860 50  0000 L CNN
+F 1 "10uF" H 3875 2800 50  0000 L CNN
+F 2 "" H 3800 2800 50  0001 C CNN
+F 3 "~" H 3800 2800 50  0001 C CNN
+F 4 "DNU" H 3920 2740 50  0000 C CNN "Digikey PN"
+	1    3800 2800
+	1    0    0    -1
+$EndComp
+$Comp
+L Device:C_Small C?
+U 1 1 619F556E
+P 4200 2800
+F 0 "C?" H 4235 2865 50  0000 L CNN
+F 1 "10uF" H 4275 2805 50  0000 L CNN
+F 2 "" H 4200 2800 50  0001 C CNN
+F 3 "~" H 4200 2800 50  0001 C CNN
+F 4 "DNU" H 4315 2740 50  0000 C CNN "Digikey PN"
+	1    4200 2800
+	1    0    0    -1
+$EndComp
+$Comp
+L Device:C_Small C?
+U 1 1 619F58AB
+P 4600 2800
+F 0 "C?" H 4620 2865 50  0000 L CNN
+F 1 "10uF" H 4660 2800 50  0000 L CNN
+F 2 "" H 4600 2800 50  0001 C CNN
+F 3 "~" H 4600 2800 50  0001 C CNN
+F 4 "DNU" H 4705 2740 50  0000 C CNN "Digikey PN"
+	1    4600 2800
+	1    0    0    -1
+$EndComp
+Wire Wire Line
+	3450 2900 3450 2950
+Wire Wire Line
+	3800 2900 3800 2950
+Wire Wire Line
+	3800 2950 3450 2950
+Connection ~ 3450 2950
+Wire Wire Line
+	3800 2950 4200 2950
+Wire Wire Line
+	4200 2950 4200 2900
+Connection ~ 3800 2950
+Wire Wire Line
+	4200 2950 4600 2950
+Wire Wire Line
+	4600 2950 4600 2900
+Connection ~ 4200 2950
+Wire Wire Line
+	4600 2950 5100 2950
+Connection ~ 4600 2950
+Wire Wire Line
+	3250 2650 3450 2650
+Connection ~ 5100 2650
+Wire Wire Line
+	3450 2700 3450 2650
+Connection ~ 3450 2650
+Wire Wire Line
+	3450 2650 3800 2650
+Wire Wire Line
+	3800 2700 3800 2650
+Connection ~ 3800 2650
+Wire Wire Line
+	3800 2650 4200 2650
+Wire Wire Line
+	4200 2700 4200 2650
+Connection ~ 4200 2650
+Wire Wire Line
+	4200 2650 4600 2650
+Wire Wire Line
+	4600 2700 4600 2650
+Connection ~ 4600 2650
+Wire Wire Line
+	4600 2650 5100 2650
 $EndSCHEMATC

Commit message: k
Parts:
- C1: renamed from C?; footprint (none) -> Capacitor_THT:CP_Radial_D5.0mm_P2.00mm; Digikey PN (none) -> 732-8700-1-ND
- C10, C7: renamed from C?; footprint (none) -> Capacitor_SMD:C_0603_1608Metric_Pad1.08x0.95mm_HandSolder
- C2, C3, C4, C5, C9: renamed from C?; footprint (none) -> Capacitor_SMD:C_0805_2012Metric_Pad1.18x1.45mm_HandSolder
- C6: renamed from C?; footprint (none) -> Capacitor_SMD:C_0603_1608Metric_Pad1.08x0.95mm_HandSolder; Digikey PN (none) -> 1276-1902-1-ND
- gave numbers to parts that had none: 16

Commit message: k
Parts:
- removed C1: 47uF, Capacitor_THT:CP_Radial_D5.0mm_P2.00mm, symbol Device:CP1_Small
- L1: Digikey PN (none) -> 732-1012-1-ND
- R1: footprint (none) -> Resistor_SMD:R_0603_1608Metric_Pad0.98x0.95mm_HandSolder; Digikey PN (none) -> RMCF0603FT5M62CT-ND
- R2: footprint (none) -> Resistor_SMD:R_0603_1608Metric_Pad0.98x0.95mm_HandSolder; Digikey PN (none) -> RMCF0603FT4M53CT-ND
- R3: footprint (none) -> Resistor_SMD:R_0603_1608Metric_Pad0.98x0.95mm_HandSolder; Digikey PN (none) -> RMCF0603FT390KCT-ND
- R4: footprint (none) -> Resistor_SMD:R_0603_1608Metric_Pad0.98x0.95mm_HandSolder; Digikey PN (none) -> 541-9.76MHCT-ND
- R5: footprint (none) -> Resistor_SMD:R_0603_1608Metric_Pad0.98x0.95mm_HandSolder; Digikey PN (none) -> 541-1.69MHCT-ND
- R6: footprint (none) -> Resistor_SMD:R_0603_1608Metric_Pad0.98x0.95mm_HandSolder; Digikey PN (none) -> RMCF0603FT1M40CT-ND
- R7: footprint (none) -> Resistor_SMD:R_0603_1608Metric_Pad0.98x0.95mm_HandSolder; Digikey PN (none) -> RMCF0603FT6M98CT-ND
- R8, R9: footprint (none) -> Resistor_SMD:R_0603_1608Metric_Pad0.98x0.95mm_HandSolder; Digikey PN (none) -> 541-2804-1-ND
- renumbered C2 to C1, C3 to C2, C4 to C3, C5 to C4, C6 to C5, C7 to C6, C8 to C7, C9 to C8, C10 to C9
Connections:
- wire segments 99 -> 95
Other:
- moved on the sheet: R1, R2

Commit message: just kinda out here guys ya know what im saying
Parts:
- removed D1: 4V, Diode_SMD:D_MiniMELF, symbol Diode:ZMMxx
- added D200: BZX84Cxx, batteryless_gaming_device:D_SOT-23_ANK_HandSoldering, symbol Diode:BZX84Cxx
- C206: renamed from C7; footprint (none) -> Capacitor_THT:CP_Radial_D14.0mm_P5.00mm
- L200: renamed from L1; footprint (none) -> batteryless_gaming_device:L_Wuerth-3816_6.3x6.3mm
- U200: renamed from U2; footprint Package_DFN_QFN:QFN-16-1EP_3x3mm_P0.5mm_EP1.8x1.8mm -> Package_DFN_QFN:VQFN-16-1EP_3x3mm_P0.5mm_EP1.8x1.8mm
- renumbered C1 to C200, C2 to C201, C3 to C202, C4 to C203, C5 to C204, C6 to C205, C8 to C207, C9 to C208, R1 to R200, R2 to R201, R3 to R202, R4 to R203, R5 to R204, R6 to R205, R7 to R206, R8 to R207, R9 to R208, TP1 to TP200, TP2 to TP201, TP3 to TP202

Commit message: oh ya
Parts:
- removed C203: 10uF, Capacitor_SMD:C_0805_2012Metric_Pad1.18x1.45mm_HandSolder, symbol Device:C_Small
- U200: Digikey PN (none) -> 296-48495-1-ND
Changed lines of the file:
@@
-	1    0    0    -1
-$EndComp
-$Comp
-L Device:C_Small C203
-U 1 1 619F58AB
-P 4600 2800
-F 0 "C203" H 4620 2865 50  0000 L CNN
-F 1 "10uF" H 4660 2800 50  0000 L CNN
-F 2 "Capacitor_SMD:C_0805_2012Metric_Pad1.18x1.45mm_HandSolder" H 4600 2800 50  0001 C CNN
-F 3 "~" H 4600 2800 50  0001 C CNN
-F 4 "DNU" H 4705 2740 50  0000 C CNN "Digikey PN"
-	1    4600 2800
 	1    0    0    -1
 $EndComp
@@
 	4200 2950 4200 2900
 Connection ~ 3800 2950
-Wire Wire Line
-	4200 2950 4600 2950
-Wire Wire Line
-	4600 2950 4600 2900
 Connection ~ 4200 2950
-Wire Wire Line
-	4600 2950 5100 2950
-Connection ~ 4600 2950
 Wire Wire Line
 	3250 2650 3450 2650
@@
 	4200 2700 4200 2650
 Connection ~ 4200 2650
-Wire Wire Line
-	4200 2650 4600 2650
-Wire Wire Line
-	4600 2700 4600 2650
-Connection ~ 4600 2650
-Wire Wire Line
-	4600 2650 5100 2650
 Wire Wire Line
 	2750 2950 3450 2950
@@
 F 2 "Package_DFN_QFN:VQFN-16-1EP_3x3mm_P0.5mm_EP1.8x1.8mm" H 6700 3500 50  0001 C CNN
 F 3 "http://www.ti.com/lit/ds/symlink/bq25504.pdf" H 6400 4300 50  0001 C CNN
+F 4 "296-48495-1-ND" H 7650 3350 39  0000 C CNN "Digikey PN"
 	1    6700 3500
 	1    0    0    -1
@@
 Wire Wire Line
 	2750 2650 3250 2650
+Wire Wire Line
+	4200 2950 5100 2950
+Wire Wire Line
+	4200 2650 5100 2650
 $EndSCHEMATC

Commit message: updated
Parts:
- added C203, C209: 100uF, Capacitor_THT:CP_Radial_D14.0mm_P5.00mm, symbol Device:CP1_Small
- added R209: 1.1M, Resistor_SMD:R_0603_1608Metric_Pad0.98x0.95mm_HandSolder, symbol Device:R_US
- added R210: 1M, Resistor_SMD:R_0603_1608Metric_Pad0.98x0.95mm_HandSolder, symbol Device:R_US
- C206: value 220mF -> 100mF
Connections:
- net GND: now also C203.2, C209.2, R210.1
- net Vout: now also C209.1
- net at C206.1, TP201.1, U200.14 (VBAT): now also C203.1, R209.2
- new net Vsupercap: R209.1, R210.2
Other:
- note added: "Not correct resistor values for charactistics stated above"
- note added: "WANTED CHARACTERISTICS\nVBAT_OV=4.2V\nVBAT_UV=2.2V\n\nVBAT_OK=2.6V\nVBAT_OK_HYST=2.8V\n"
- note removed: "VBAT_OV=4.2V\nVBAT_UV=1.3V\n\nVBAT_OK=1.5V\nVBAT_OK_HYST=1.8V\n"
Changed lines of the file:
@@
 P 7400 2600
 F 0 "C206" H 7491 2646 50  0000 L CNN
-F 1 "220mF" H 7491 2555 50  0000 L CNN
+F 1 "100mF" H 7491 2555 50  0000 L CNN
 F 2 "Capacitor_THT:CP_Radial_D14.0mm_P5.00mm" H 7400 2600 50  0001 C CNN
 F 3 "~" H 7400 2600 50  0001 C CNN
@@
 	1    0    0    -1
 $EndComp
-Text Notes 2600 3950 0    50   ~ 0
-VBAT_OV=4.2V\nVBAT_UV=1.3V\n\nVBAT_OK=1.5V\nVBAT_OK_HYST=1.8V\n
-Wire Wire Line
-	7300 3200 7700 3200
-Text HLabel 7700 3200 2    50   Output ~ 0
-VBAT_OK
-Text HLabel 8400 3800 2    50   Output ~ 0
+Text Notes 2500 3950 0    50   ~ 0
+WANTED CHARACTERISTICS\nVBAT_OV=4.2V\nVBAT_UV=2.2V\n\nVBAT_OK=2.6V\nVBAT_OK_HYST=2.8V\n
+Text HLabel 8900 3800 2    50   Output ~ 0
 Vout
 $Comp
@@
 Connection ~ 8000 3800
 Wire Wire Line
-	8000 3800 8400 3800
+	8000 3800 8600 3800
 Text HLabel 2450 2650 0    50   Input ~ 0
 Vin
@@
 Wire Wire Line
 	4200 2650 5100 2650
+$Comp
+L Device:CP1_Small C203
+U 1 1 61B2CBD0
+P 7900 2600
+F 0 "C203" H 7991 2646 50  0000 L CNN
+F 1 "100uF" H 7991 2555 50  0000 L CNN
+F 2 "Capacitor_THT:CP_Radial_D14.0mm_P5.00mm" H 7900 2600 50  0001 C CNN
+F 3 "~" H 7900 2600 50  0001 C CNN
+	1    7900 2600
+	1    0    0    -1
+$EndComp
+Wire Wire Line
+	7400 2700 7900 2700
+Connection ~ 7400 2700
+Wire Wire Line
+	7900 2500 7900 2450
+Wire Wire Line
+	7900 2450 7400 2450
+Connection ~ 7400 2450
+Text HLabel 7700 3200 2    50   Output ~ 0
+VBAT_OK
+Wire Wire Line
+	7300 3200 7700 3200
+Text HLabel 8900 2450 2    50   Output ~ 0
+Vsupercap
+$Comp
+L Device:R_US R?
+U 1 1 61BF204D
+P 8300 2450
+AR Path="/619A7303/61BF204D" Ref="R?"  Part="1"
+AR Path="/61991596/61BF204D" Ref="R209"  Part="1"
+F 0 "R209" V 8095 2450 50  0000 C CNN
+F 1 "1.1M" V 8186 2450 50  0000 C CNN
+F 2 "Resistor_SMD:R_0603_1608Metric_Pad0.98x0.95mm_HandSolder" V 8340 2440 50  0001 C CNN
+F 3 "~" H 8300 2450 50  0001 C CNN
+F 4 "" V 8400 2450 39  0000 C CNN "Digikey PN"
+	1    8300 2450
+	0    1    1    0
+$EndComp
+Wire Wire Line
+	8650 2450 8450 2450
+Wire Wire Line
+	7900 2450 8150 2450
+$Comp
+L Device:R_US R?
+U 1 1 61BF2059
+P 8650 2750
+AR Path="/619A7303/61BF2059" Ref="R?"  Part="1"
+AR Path="/61991596/61BF2059" Ref="R210"  Part="1"
+F 0 "R210" H 8550 2650 50  0000 C CNN
+F 1 "1M" H 8536 2750 50  0000 C CNN
+F 2 "Resistor_SMD:R_0603_1608Metric_Pad0.98x0.95mm_HandSolder" V 8690 2740 50  0001 C CNN
+F 3 "~" H 8650 2750 50  0001 C CNN
+F 4 "511-1820-1-ND" H 8300 2850 39  0000 C CNN "Digikey PN"
+	1    8650 2750
+	-1   0    0    1
+$EndComp
+Wire Wire Line
+	8650 2450 8650 2600
+$Comp
+L power:GND #PWR?
+U 1 1 61BF2060
+P 8650 2950
+AR Path="/619A7303/61BF2060" Ref="#PWR?"  Part="1"
+AR Path="/61991596/61BF2060" Ref="#PWR0114"  Part="1"
+F 0 "#PWR0114" H 8650 2700 50  0001 C CNN
+F 1 "GND" H 8655 2777 50  0000 C CNN
+F 2 "" H 8650 2950 50  0001 C CNN
+F 3 "" H 8650 2950 50  0001 C CNN
+	1    8650 2950
+	1    0    0    -1
+$EndComp
+Wire Wire Line
+	8650 2900 8650 2950
+Connection ~ 7900 2450
+Wire Wire Line
+	8650 2450 8900 2450
+Connection ~ 8650 2450
+$Comp
+L Device:CP1_Small C209
+U 1 1 61C35FE5
+P 8600 4000
+F 0 "C209" H 8691 4046 50  0000 L CNN
+F 1 "100uF" H 8691 3955 50  0000 L CNN
+F 2 "Capacitor_THT:CP_Radial_D14.0mm_P5.00mm" H 8600 4000 50  0001 C CNN
+F 3 "~" H 8600 4000 50  0001 C CNN
+	1    8600 4000
+	1    0    0    -1
+$EndComp
+Wire Wire Line
+	8600 3800 8600 3900
+Connection ~ 8600 3800
+Wire Wire Line
+	8600 3800 8900 3800
+Wire Wire Line
+	8600 4100 8600 4150
+Wire Wire Line
+	8600 4150 7850 4150
+Connection ~ 7850 4150
+Text Notes 3500 4150 2    50   ~ 0
+Not correct resistor values for charactistics stated above
 $EndSCHEMATC
